Commit message: feat(ros2_control): moved urdf to xacro architecture, implemented ros2_control

File: InMoov/robot_description/urdf/robot_description.urdf.xacro (robot description, xacro)
@@ -1,3 +1,4 @@
-<robot name="InMoov" version="1.0">
+<?xml version="1.0"?>
+<robot xmlns:xacro="http://www.ros.org/wiki/xacro" name="InMoov" version="1.0">
   <joint name="Empty.001_link_joint" type="fixed">
     <origin rpy="0.00000 0.00000 0.00000" xyz="-0.00394 0.00025 -0.19163"/>

File: hardware_config/inmoov_actuators_config.xacro (robot description, xacro)
@@ -15,6 +15,7 @@
 <!-- Servo Motor Configuration Macro -->
 <!-- Defines a standard template for servo motor configuration with parameters for name, joint, board, pin, type, limits, and default position -->
-<xacro:macro name="servo_motor"params="name joint_name board pin type min_limit max_limit default_pos enabled:=false">
-    <actuator name="${name}"enabled="${enabled}">
+<robot xmlns:xacro="http://www.ros.org/wiki/xacro">
+<xacro:macro name="servo_motor" params="name joint_name board pin type min_limit max_limit default_pos enabled:=false">
+    <actuator name="${name}" enabled="${enabled}">
         <joint name="${joint_name}"/>
         <hardware>
@@ -486,2 +487,3 @@
                    default_pos="null"
                    enabled="false"/>
+</robot>

File: hardware_config/inmoov_hardware_config.xacro (robot description, xacro)
@@ -1,18 +1,4 @@
 <?xml version="1.0"?>
 <robot name="inmoov-i2" xmlns:xacro="http://www.ros.org/wiki/xacro">
-    <!-- =============================================== -->
-    <!-- Inmoov Humanoid Robot Hardware Configuration    -->
-    <!-- =============================================== -->
-    <!--
-        This file contains the complete hardware specifications for the Inmoov robot:
-        - Servo motors (through inmoov_actuators_config.xacro)
-        - Pressure sensors (through inmoov_sensors_config.xacro)
-        This is the main entry point for hardware configuration that imports
-        the separated configuration files.
-    -->
-    <!-- =============================================== -->
-    <!-- Import Configuration Files                      -->
-    <!-- =============================================== -->
-    <!-- Import Actuators Configuration -->
     <xacro:include filename="inmoov_actuators_config.xacro"/>
     <!-- Import ROS2 Control Configuration -->

File: hardware_config/inmoov_sensors_config.xacro (robot description, xacro)
@@ -15,4 +15,5 @@
 <!-- Pressure Sensor Configuration Macro -->
 <!-- Defines a standard template for pressure sensors with parameters for name, associated finger, board, pin, and resistance range -->
+<robot xmlns:xacro="http://www.ros.org/wiki/xacro">
 <xacro:macro name="pressure_sensor" params="name finger_name board pin min_resistance max_resistance enabled:=false">
     <sensor name="${name}" enabled="${enabled}">
@@ -113,2 +114,3 @@
                       max_resistance="null"
                       enabled="false"/>
+</robot>

Commit message: fix(xacro): fixed the paths of meshes to be absolute path instead of relative (../)

File: InMoov/robot_description/urdf/robot_description.urdf.xacro (robot description, xacro)
@@ -1,4 +1,5 @@
 <?xml version="1.0"?>
 <robot xmlns:xacro="http://www.ros.org/wiki/xacro" name="InMoov" version="1.0">
+  <xacro:property name="mesh_dir" value="/home/dev/thais_urdf/InMoov/robot_description/meshes/stl"/>
   <joint name="Empty.001_link_joint" type="fixed">
     <origin rpy="0.00000 0.00000 0.00000" xyz="-0.00394 0.00025 -0.19163"/>
@@ -409,5 +410,5 @@
       <origin rpy="3.14159 -0.00000 3.14159" xyz="-0.00394 -0.00730 9.35280"/>
       <geometry>
-        <mesh filename="../meshes/stl/stand.stl" scale="1.00000 1.00000 1.00000"/>
+        <mesh filename="${mesh_dir}/stand.stl" scale="1.00000 1.00000 1.00000"/>
       </geometry>
     </visual>
@@ -419,5 +420,5 @@
       <material name="Material.035"/>
       <geometry>
-        <mesh filename="../meshes/stl/Texture.011.stl" scale="1.00000 1.00000 1.00000"/>
+        <mesh filename="${mesh_dir}/Texture.011.stl" scale="1.00000 1.00000 1.00000"/>
       </geometry>
     </visual>
@@ -429,5 +430,5 @@
       <material name="Material.038"/>
       <geometry>
-        <mesh filename="../meshes/stl/Texture.012.stl" scale="1.00000 1.00000 1.00000"/>
+        <mesh filename="${mesh_dir}/Texture.012.stl" scale="1.00000 1.00000 1.00000"/>
       </geometry>
     </visual>
@@ -438,5 +439,5 @@
       <material name="Material.046"/>
       <geometry>
-        <mesh filename="../meshes/stl/Texture.014.stl" scale="1.00000 1.00000 1.00000"/>
+        <mesh filename="${mesh_dir}/Texture.014.stl" scale="1.00000 1.00000 1.00000"/>
       </geometry>
     </visual>
@@ -445,5 +446,5 @@
       <material name="Material.046"/>
       <geometry>
-        <mesh filename="../meshes/stl/Texture.086.stl" scale="1.00000 1.00000 1.00000"/>
+        <mesh filename="${mesh_dir}/Texture.086.stl" scale="1.00000 1.00000 1.00000"/>
       </geometry>
     </visual>
@@ -452,5 +453,5 @@
       <material name="Material.046"/>
       <geometry>
-        <mesh filename="../meshes/stl/Texture.087.stl" scale="1.00000 1.00000 1.00000"/>
+        <mesh filename="${mesh_dir}/Texture.087.stl" scale="1.00000 1.00000 1.00000"/>
       </geometry>
     </visual>
@@ -462,5 +463,5 @@
       <material name="Material.044"/>
       <geometry>
-        <mesh filename="../meshes/stl/Texture.013.stl" scale="1.00000 1.00000 1.00000"/>
+        <mesh filename="${mesh_dir}/Texture.013.stl" scale="1.00000 1.00000 1.00000"/>
       </geometry>
     </visual>
@@ -469,5 +470,5 @@
       <material name="Material.044"/>
       <geometry>
-        <mesh filename="../meshes/stl/Texture.068.stl" scale="1.00000 1.00000 1.00000"/>
+        <mesh filename="${mesh_dir}/Texture.068.stl" scale="1.00000 1.00000 1.00000"/>
       </geometry>
     </visual>
@@ -476,5 +477,5 @@
       <material name="Material.044"/>
       <geometry>
-        <mesh filename="../meshes/stl/Texture.069.stl" scale="1.00000 1.00000 1.00000"/>
+        <mesh filename="${mesh_dir}/Texture.069.stl" scale="1.00000 1.00000 1.00000"/>
       </geometry>
     </visual>
@@ -483,5 +484,5 @@
       <material name="Material.044"/>
       <geometry>
-        <mesh filename="../meshes/stl/Texture.070.stl" scale="1.00000 1.00000 1.00000"/>
+        <mesh filename="${mesh_dir}/Texture.070.stl" scale="1.00000 1.00000 1.00000"/>
       </geometry>
     </visual>
@@ -490,5 +491,5 @@
       <material name="Material.044"/>
       <geometry>
-        <mesh filename="../meshes/stl/Texture.071.stl" scale="1.00000 1.00000 1.00000"/>
+        <mesh filename="${mesh_dir}/Texture.071.stl" scale="1.00000 1.00000 1.00000"/>
       </geometry>
     </visual>
@@ -497,5 +498,5 @@
       <material name="Material.044"/>
       <geometry>
-        <mesh filename="../meshes/stl/Texture.072.stl" scale="1.00000 1.00000 1.00000"/>
+        <mesh filename="${mesh_dir}/Texture.072.stl" scale="1.00000 1.00000 1.00000"/>
       </geometry>
     </visual>
@@ -504,5 +505,5 @@
       <material name="Material.044"/>
       <geometry>
-        <mesh filename="../meshes/stl/Texture.073.stl" scale="1.00000 1.00000 1.00000"/>
+        <mesh filename="${mesh_dir}/Texture.073.stl" scale="1.00000 1.00000 1.00000"/>
       </geometry>
     </visual>
@@ -511,5 +512,5 @@
       <material name="Material.044"/>
       <geometry>
-        <mesh filename="../meshes/stl/Texture.074.stl" scale="1.00000 1.00000 1.00000"/>
+        <mesh filename="${mesh_dir}/Texture.074.stl" scale="1.00000 1.00000 1.00000"/>
       </geometry>
     </visual>
@@ -518,5 +519,5 @@
       <material name="Material.044"/>
       <geometry>
-        <mesh filename="../meshes/stl/Texture.075.stl" scale="1.00000 1.00000 1.00000"/>
+        <mesh filename="${mesh_dir}/Texture.075.stl" scale="1.00000 1.00000 1.00000"/>
       </geometry>
     </visual>
@@ -525,5 +526,5 @@
       <material name="Material.044"/>
       <geometry>
-        <mesh filename="../meshes/stl/Texture.076.stl" scale="1.00000 1.00000 1.00000"/>
+        <mesh filename="${mesh_dir}/Texture.076.stl" scale="1.00000 1.00000 1.00000"/>
       </geometry>
     </visual>
@@ -532,5 +533,5 @@
       <material name="Material.044"/>
       <geometry>
-        <mesh filename="../meshes/stl/Texture.077.stl" scale="1.00000 1.00000 1.00000"/>
+        <mesh filename="${mesh_dir}/Texture.077.stl" scale="1.00000 1.00000 1.00000"/>
       </geometry>
     </visual>
@@ -539,5 +540,5 @@
       <material name="Material.044"/>
       <geometry>
-        <mesh filename="../meshes/stl/Texture.078.stl" scale="1.00000 1.00000 1.00000"/>
+        <mesh filename="${mesh_dir}/Texture.078.stl" scale="1.00000 1.00000 1.00000"/>
       </geometry>
     </visual>
@@ -546,5 +547,5 @@
       <material name="Material.044"/>
       <geometry>
-        <mesh filename="../meshes/stl/Texture.079.stl" scale="1.00000 1.00000 1.00000"/>
+        <mesh filename="${mesh_dir}/Texture.079.stl" scale="1.00000 1.00000 1.00000"/>
       </geometry>
     </visual>
@@ -553,5 +554,5 @@
       <material name="Material.044"/>
       <geometry>
-        <mesh filename="../meshes/stl/Texture.080.stl" scale="1.00000 1.00000 1.00000"/>
+        <mesh filename="${mesh_dir}/Texture.080.stl" scale="1.00000 1.00000 1.00000"/>
       </geometry>
     </visual>
@@ -560,5 +561,5 @@
       <material name="Material.044"/>
       <geometry>
-        <mesh filename="../meshes/stl/Texture.081.stl" scale="1.00000 1.00000 1.00000"/>
+        <mesh filename="${mesh_dir}/Texture.081.stl" scale="1.00000 1.00000 1.00000"/>
       </geometry>
     </visual>
@@ -567,5 +568,5 @@
       <material name="Material.044"/>
       <geometry>
-        <mesh filename="../meshes/stl/Texture.082.stl" scale="1.00000 1.00000 1.00000"/>
+        <mesh filename="${mesh_dir}/Texture.082.stl" scale="1.00000 1.00000 1.00000"/>
       </geometry>
     </visual>
@@ -576,5 +577,5 @@
       <material name="Material.614"/>
       <geometry>
-        <mesh filename="../meshes/stl/Texture.019.stl" scale="1.00000 1.00000 1.00000"/>
+        <mesh filename="${mesh_dir}/Texture.019.stl" scale="1.00000 1.00000 1.00000"/>
       </geometry>
     </visual>
@@ -585,5 +586,5 @@
       <material name="Material.618"/>
       <geometry>
-        <mesh filename="../meshes/stl/Texture.020.stl" scale="1.00000 1.00000 1.00000"/>
+        <mesh filename="${mesh_dir}/Texture.020.stl" scale="1.00000 1.00000 1.00000"/>
       </geometry>
     </visual>
@@ -594,5 +595,5 @@
       <material name="Material.610"/>
       <geometry>
-        <mesh filename="../meshes/stl/Texture.018.stl" scale="1.00000 1.00000 1.00000"/>
+        <mesh filename="${mesh_dir}/Texture.018.stl" scale="1.00000 1.00000 1.00000"/>
       </geometry>
     </visual>
@@ -603,5 +604,5 @@
       <material name="Material.613"/>
       <geometry>
-        <mesh filename="../meshes/stl/Texture.023.stl" scale="1.00000 1.00000 1.00000"/>
+        <mesh filename="${mesh_dir}/Texture.023.stl" scale="1.00000 1.00000 1.00000"/>
       </geometry>
     </visual>
@@ -612,5 +613,5 @@
       <material name="Material.617"/>
       <geometry>
-        <mesh filename="../meshes/stl/Texture.024.stl" scale="1.00000 1.00000 1.00000"/>
+        <mesh filename="${mesh_dir}/Texture.024.stl" scale="1.00000 1.00000 1.00000"/>
       </geometry>
     </visual>
@@ -621,5 +622,5 @@
       <material name="Material.609"/>
       <geometry>
-        <mesh filename="../meshes/stl/Texture.022.stl" scale="1.00000 1.00000 1.00000"/>
+        <mesh filename="${mesh_dir}/Texture.022.stl" scale="1.00000 1.00000 1.00000"/>
       </geometry>
     </visual>
@@ -630,5 +631,5 @@
       <material name="Material.601"/>
       <geometry>
-        <mesh filename="../meshes/stl/Texture.041.stl" scale="1.00000 1.00000 1.00000"/>
+        <mesh filename="${mesh_dir}/Texture.041.stl" scale="1.00000 1.00000 1.00000"/>
       </geometry>
     </visual>
@@ -639,5 +640,5 @@
       <material name="Material.611"/>
       <geometry>
-        <mesh filename="../meshes/stl/Texture.028.stl" scale="1.00000 1.00000 1.00000"/>
+        <mesh filename="${mesh_dir}/Texture.028.stl" scale="1.00000 1.00000 1.00000"/>
       </geometry>
     </visual>
@@ -648,5 +649,5 @@
       <material name="Material.615"/>
       <geometry>
-        <mesh filename="../meshes/stl/Texture.029.stl" scale="1.00000 1.00000 1.00000"/>
+        <mesh filename="${mesh_dir}/Texture.029.stl" scale="1.00000 1.00000 1.00000"/>
       </geometry>
     </visual>
@@ -657,5 +658,5 @@
       <material name="Material.607"/>
       <geometry>
-        <mesh filename="../meshes/stl/Texture.027.stl" scale="1.00000 1.00000 1.00000"/>
+        <mesh filename="${mesh_dir}/Texture.027.stl" scale="1.00000 1.00000 1.00000"/>
       </geometry>
     </visual>
@@ -666,5 +667,5 @@
       <material name="Material.608"/>
       <geometry>
-        <mesh filename="../meshes/stl/Texture.032.stl" scale="1.00000 1.00000 1.00000"/>
+        <mesh filename="${mesh_dir}/Texture.032.stl" scale="1.00000 1.00000 1.00000"/>
       </geometry>
     </visual>
@@ -675,5 +676,5 @@
       <material name="Material.606"/>
       <geometry>
-        <mesh filename="../meshes/stl/Texture.040.stl" scale="1.00000 1.00000 1.00000"/>
+        <mesh filename="${mesh_dir}/Texture.040.stl" scale="1.00000 1.00000 1.00000"/>
       </geometry>
     </visual>
@@ -684,5 +685,5 @@
       <material name="Material.612"/>
       <geometry>
-        <mesh filename="../meshes/stl/Texture.033.stl" scale="1.00000 1.00000 1.00000"/>
+        <mesh filename="${mesh_dir}/Texture.033.stl" scale="1.00000 1.00000 1.00000"/>
       </geometry>
     </visual>
@@ -693,5 +694,5 @@
       <material name="Material.616"/>
       <geometry>
-        <mesh filename="../meshes/stl/Texture.034.stl" scale="1.00000 1.00000 1.00000"/>
+        <mesh filename="${mesh_dir}/Texture.034.stl" scale="1.00000 1.00000 1.00000"/>
       </geometry>
     </visual>
@@ -702,5 +703,5 @@
       <material name="Material.603"/>
       <geometry>
-        <mesh filename="../meshes/stl/Texture.035.stl" scale="1.00000 1.00000 1.00000"/>
+        <mesh filename="${mesh_dir}/Texture.035.stl" scale="1.00000 1.00000 1.00000"/>
       </geometry>
     </visual>
@@ -711,5 +712,5 @@
       <material name="Material.605"/>
       <geometry>
-        <mesh filename="../meshes/stl/Texture.038.stl" scale="1.00000 1.00000 1.00000"/>
+        <mesh filename="${mesh_dir}/Texture.038.stl" scale="1.00000 1.00000 1.00000"/>
       </geometry>
     </visual>
@@ -720,5 +721,5 @@
       <material name="Material.604"/>
       <geometry>
-        <mesh filename="../meshes/stl/Texture.037.stl" scale="1.00000 1.00000 1.00000"/>
+        <mesh filename="${mesh_dir}/Texture.037.stl" scale="1.00000 1.00000 1.00000"/>
       </geometry>
     </visual>
@@ -729,5 +730,5 @@
       <material name="Material.602"/>
       <geometry>
-        <mesh filename="../meshes/stl/Texture.235.stl" scale="1.00000 1.00000 1.00000"/>
+        <mesh filename="${mesh_dir}/Texture.235.stl" scale="1.00000 1.00000 1.00000"/>
       </geometry>
     </visual>
@@ -738,5 +739,5 @@
       <material name="Material.636"/>
       <geometry>
-        <mesh filename="../meshes/stl/Texture.045.stl" scale="1.00000 1.00000 1.00000"/>
+        <mesh filename="${mesh_dir}/Texture.045.stl" scale="1.00000 1.00000 1.00000"/>
       </geometry>
     </visual>
@@ -747,5 +748,5 @@
       <material name="Material.640"/>
       <geometry>
-        <mesh filename="../meshes/stl/Texture.046.stl" scale="1.00000 1.00000 1.00000"/>
+        <mesh filename="${mesh_dir}/Texture.046.stl" scale="1.00000 1.00000 1.00000"/>
       </geometry>
     </visual>
@@ -756,5 +757,5 @@
       <material name="Material.632"/>
       <geometry>
-        <mesh filename="../meshes/stl/Texture.044.stl" scale="1.00000 1.00000 1.00000"/>
+        <mesh filename="${mesh_dir}/Texture.044.stl" scale="1.00000 1.00000 1.00000"/>
       </geometry>
     </visual>
@@ -765,5 +766,5 @@
       <material name="Material.637"/>
       <geometry>
-        <mesh filename="../meshes/stl/Texture.049.stl" scale="1.00000 1.00000 1.00000"/>
+        <mesh filename="${mesh_dir}/Texture.049.stl" scale="1.00000 1.00000 1.00000"/>
       </geometry>
     </visual>
@@ -774,5 +775,5 @@
       <material name="Material.641"/>
       <geometry>
-        <mesh filename="../meshes/stl/Texture.050.stl" scale="1.00000 1.00000 1.00000"/>
+        <mesh filename="${mesh_dir}/Texture.050.stl" scale="1.00000 1.00000 1.00000"/>
       </geometry>
     </visual>
@@ -783,5 +784,5 @@
       <material name="Material.633"/>
       <geometry>
-        <mesh filename="../meshes/stl/Texture.048.stl" scale="1.00000 1.00000 1.00000"/>
+        <mesh filename="${mesh_dir}/Texture.048.stl" scale="1.00000 1.00000 1.00000"/>
       </geometry>
     </visual>
@@ -792,5 +793,5 @@
       <material name="Material.630"/>
       <geometry>
-        <mesh filename="../meshes/stl/Texture.067.stl" scale="1.00000 1.00000 1.00000"/>
+        <mesh filename="${mesh_dir}/Texture.067.stl" scale="1.00000 1.00000 1.00000"/>
       </geometry>
     </visual>
@@ -801,5 +802,5 @@
       <material name="Material.639"/>
       <geometry>
-        <mesh filename="../meshes/stl/Texture.054.stl" scale="1.00000 1.00000 1.00000"/>
+        <mesh filename="${mesh_dir}/Texture.054.stl" scale="1.00000 1.00000 1.00000"/>
       </geometry>
     </visual>
@@ -810,5 +811,5 @@
       <material name="Material.643"/>
       <geometry>
-        <mesh filename="../meshes/stl/Texture.055.stl" scale="1.00000 1.00000 1.00000"/>
+        <mesh filename="${mesh_dir}/Texture.055.stl" scale="1.00000 1.00000 1.00000"/>
       </geometry>
     </visual>
@@ -819,5 +820,5 @@
       <material name="Material.635"/>
       <geometry>
-        <mesh filename="../meshes/stl/Texture.053.stl" scale="1.00000 1.00000 1.00000"/>
+        <mesh filename="${mesh_dir}/Texture.053.stl" scale="1.00000 1.00000 1.00000"/>
       </geometry>
     </visual>
@@ -828,5 +829,5 @@
       <material name="Material.634"/>
       <geometry>
-        <mesh filename="../meshes/stl/Texture.058.stl" scale="1.00000 1.00000 1.00000"/>
+        <mesh filename="${mesh_dir}/Texture.058.stl" scale="1.00000 1.00000 1.00000"/>
       </geometry>
     </visual>
@@ -837,5 +838,5 @@
       <material name="Material.631"/>
       <geometry>
-        <mesh filename="../meshes/stl/Texture.066.stl" scale="1.00000 1.00000 1.00000"/>
+        <mesh filename="${mesh_dir}/Texture.066.stl" scale="1.00000 1.00000 1.00000"/>
       </geometry>
     </visual>
@@ -846,5 +847,5 @@
       <material name="Material.638"/>
       <geometry>
-        <mesh filename="../meshes/stl/Texture.059.stl" scale="1.00000 1.00000 1.00000"/>
+        <mesh filename="${mesh_dir}/Texture.059.stl" scale="1.00000 1.00000 1.00000"/>
       </geometry>
     </visual>
@@ -855,5 +856,5 @@
       <material name="Material.642"/>
       <geometry>
-        <mesh filename="../meshes/stl/Texture.060.stl" scale="1.00000 1.00000 1.00000"/>
+        <mesh filename="${mesh_dir}/Texture.060.stl" scale="1.00000 1.00000 1.00000"/>
       </geometry>
     </visual>
@@ -864,5 +865,5 @@
       <material name="Material.628"/>
       <geometry>
-        <mesh filename="../meshes/stl/Texture.063.stl" scale="1.00000 1.00000 1.00000"/>
+        <mesh filename="${mesh_dir}/Texture.063.stl" scale="1.00000 1.00000 1.00000"/>
       </geometry>
     </visual>
@@ -873,5 +874,5 @@
       <material name="Material.626"/>
       <geometry>
-        <mesh filename="../meshes/stl/Texture.062.stl" scale="1.00000 1.00000 1.00000"/>
+        <mesh filename="${mesh_dir}/Texture.062.stl" scale="1.00000 1.00000 1.00000"/>
       </geometry>
     </visual>
@@ -882,5 +883,5 @@
       <material name="Material.627"/>
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