Commit message: feat(left arm): added configuration ros2 control for left arm joints

File: InMoov/ros2_control/inmoov_ros2_control.xacro (robot description, xacro)
@@ -8,9 +8,41 @@
           <param name="node_name">lucy_hardware_interface_left_arm</param>
       </hardware>
-      <joint name="left_thumb_joint">
+      <joint name="left_shoulder_yaw">
+          <command_interface name="position">
+          </command_interface>
+          <state_interface name="position" />
+      </joint>
+      <joint name="left_shoulder_roll">
           <command_interface name="position" />
           <state_interface name="position" />
       </joint>
-      <joint name="left_index_joint">
+      <joint name="left_elbow">
+          <command_interface name="position" />
+          <state_interface name="position" />
+      </joint>
+      <joint name="left_wrist">
+          <command_interface name="position" />
+          <state_interface name="position" />
+      </joint>
+      <joint name="left_thumb">
+          <command_interface name="position" />
+          <state_interface name="position" />
+      </joint>
+      <joint name="left_index">
+          <command_interface name="position">
+          <param name="min">0</param>
+          <param name="max">1</param>
+          </command_interface>
+          <state_interface name="position" />
+      </joint>
+      <joint name="left_middle">
+          <command_interface name="position" />
+          <state_interface name="position" />
+      </joint>
+      <joint name="left_ring">
+          <command_interface name="position" />
+          <state_interface name="position" />
+      </joint>
+      <joint name="left_pinky">
           <command_interface name="position" />
           <state_interface name="position" />
