Commit message: feat(urdf): updated mesh_dir variable for rviz path

File: inmoov/3dmodel/robot_description.urdf.xacro (robot description, xacro)
@@ -1,3 +1,5 @@
-<robot name="inmoov" version="1.0">
+<?xml version="1.0"?>
+<robot xmlns:xacro="http://www.ros.org/wiki/xacro" name="inmoov" version="1.0">
+  <xacro:property name="mesh_dir" value="file:///home/samuel/sentience/local_ws/src/thais_urdf/inmoov/meshes/dae"/>
   <joint name="Empty.001_link_joint" type="fixed">
     <origin rpy="0.00000 0.00000 0.00000" xyz="-0.00394 0.00025 -0.19163"/>
@@ -222,5 +224,5 @@
     <axis xyz="0.00000 0.00000 1.00000"/>
   </joint>
-  <joint name="right_elbow_x_link_joint" type="revolute">
+  <joint name="right_elbow" type="revolute">
     <limit lower="0.00000" upper="1.57080" effort="0.00000" velocity="0.78540"/>
     <origin rpy="0.06567 0.00000 0.00000" xyz="0.00858 0.29228 -2.11577"/>
@@ -409,5 +411,5 @@
       <origin rpy="3.14159 -0.00000 3.14159" xyz="-0.00394 -0.00730 9.35280"/>
       <geometry>
-        <mesh filename="../meshes/dae/stand.dae" scale="1.00000 1.00000 1.00000"/>
+        <mesh filename="${mesh_dir}/stand.dae" scale="1.00000 1.00000 1.00000"/>
       </geometry>
     </visual>
@@ -420,5 +422,5 @@
       <origin rpy="-0.00000 0.00000 0.00000" xyz="0.29460 0.89123 -16.02297"/>
       <geometry>
-        <mesh filename="../meshes/dae/Texture.012.dae" scale="1.00000 1.00000 1.00000"/>
+        <mesh filename="${mesh_dir}/Texture.012.dae" scale="1.00000 1.00000 1.00000"/>
       </geometry>
     </visual>
@@ -429,5 +431,5 @@
       <origin rpy="0.00000 0.00000 -0.00000" xyz="0.00732 0.15065 -15.97164"/>
       <geometry>
-        <mesh filename="../meshes/dae/Texture.014.dae" scale="1.00000 1.00000 1.00000"/>
+        <mesh filename="${mesh_dir}/Texture.014.dae" scale="1.00000 1.00000 1.00000"/>
       </geometry>
     </visual>
@@ -436,5 +438,5 @@
       <origin rpy="0.00000 0.00000 -0.00000" xyz="0.00732 0.15065 -15.97164"/>
       <geometry>
-        <mesh filename="../meshes/dae/Texture.086.dae" scale="1.00000 1.00000 1.00000"/>
+        <mesh filename="${mesh_dir}/Texture.086.dae" scale="1.00000 1.00000 1.00000"/>
       </geometry>
     </visual>
@@ -443,5 +445,5 @@
       <origin rpy="0.00000 0.00000 -0.00000" xyz="0.00732 0.15065 -15.97164"/>
       <geometry>
-        <mesh filename="../meshes/dae/Texture.087.dae" scale="1.00000 1.00000 1.00000"/>
+        <mesh filename="${mesh_dir}/Texture.087.dae" scale="1.00000 1.00000 1.00000"/>
       </geometry>
     </visual>
@@ -452,5 +454,5 @@
       <origin rpy="0.06568 0.00000 0.00000" xyz="-1.35226 1.11649 -13.89027"/>
       <geometry>
-        <mesh filename="../meshes/dae/Texture.004.dae" scale="1.00000 1.00000 1.00000"/>
+        <mesh filename="${mesh_dir}/Texture.004.dae" scale="1.00000 1.00000 1.00000"/>
       </geometry>
     </visual>
@@ -459,5 +461,5 @@
       <origin rpy="0.06568 0.00000 0.00000" xyz="-1.35226 1.11649 -13.89027"/>
       <geometry>
-        <mesh filename="../meshes/dae/Texture.248.dae" scale="1.00000 1.00000 1.00000"/>
+        <mesh filename="${mesh_dir}/Texture.248.dae" scale="1.00000 1.00000 1.00000"/>
       </geometry>
     </visual>
@@ -466,5 +468,5 @@
       <origin rpy="0.06568 0.00000 0.00000" xyz="-1.35226 1.11649 -13.89027"/>
       <geometry>
-        <mesh filename="../meshes/dae/Texture.249.dae" scale="1.00000 1.00000 1.00000"/>
+        <mesh filename="${mesh_dir}/Texture.249.dae" scale="1.00000 1.00000 1.00000"/>
       </geometry>
     </visual>
@@ -473,5 +475,5 @@
       <origin rpy="0.06568 0.00000 0.00000" xyz="-1.35226 1.11649 -13.89027"/>
       <geometry>
-        <mesh filename="../meshes/dae/Texture.250.dae" scale="1.00000 1.00000 1.00000"/>
+        <mesh filename="${mesh_dir}/Texture.250.dae" scale="1.00000 1.00000 1.00000"/>
       </geometry>
     </visual>
@@ -480,5 +482,5 @@
       <origin rpy="0.06568 0.00000 0.00000" xyz="-1.35226 1.11649 -13.89027"/>
       <geometry>
-        <mesh filename="../meshes/dae/Texture.251.dae" scale="1.00000 1.00000 1.00000"/>
+        <mesh filename="${mesh_dir}/Texture.251.dae" scale="1.00000 1.00000 1.00000"/>
       </geometry>
     </visual>
@@ -487,5 +489,5 @@
       <origin rpy="0.06568 0.00000 0.00000" xyz="-1.35226 1.11649 -13.89027"/>
       <geometry>
-        <mesh filename="../meshes/dae/Texture.252.dae" scale="1.00000 1.00000 1.00000"/>
+        <mesh filename="${mesh_dir}/Texture.252.dae" scale="1.00000 1.00000 1.00000"/>
       </geometry>
     </visual>
@@ -494,5 +496,5 @@
       <origin rpy="0.06568 0.00000 0.00000" xyz="-1.35226 1.11649 -13.89027"/>
       <geometry>
-        <mesh filename="../meshes/dae/Texture.253.dae" scale="1.00000 1.00000 1.00000"/>
+        <mesh filename="${mesh_dir}/Texture.253.dae" scale="1.00000 1.00000 1.00000"/>
       </geometry>
     </visual>
@@ -503,5 +505,5 @@
       <origin rpy="0.06568 0.00000 0.00000" xyz="-1.46578 1.11459 -13.51522"/>
       <geometry>
-        <mesh filename="../meshes/dae/Texture.003.dae" scale="1.00000 1.00000 1.00000"/>
+        <mesh filename="${mesh_dir}/Texture.003.dae" scale="1.00000 1.00000 1.00000"/>
       </geometry>
     </visual>
@@ -510,5 +512,5 @@
       <origin rpy="0.06568 0.00000 0.00000" xyz="-1.46578 1.11459 -13.51522"/>
       <geometry>
-        <mesh filename="../meshes/dae/Texture.254.dae" scale="1.00000 1.00000 1.00000"/>
+        <mesh filename="${mesh_dir}/Texture.254.dae" scale="1.00000 1.00000 1.00000"/>
       </geometry>
     </visual>
@@ -517,5 +519,5 @@
       <origin rpy="0.06568 0.00000 0.00000" xyz="-1.46578 1.11459 -13.51522"/>
       <geometry>
-        <mesh filename="../meshes/dae/Texture.255.dae" scale="1.00000 1.00000 1.00000"/>
+        <mesh filename="${mesh_dir}/Texture.255.dae" scale="1.00000 1.00000 1.00000"/>
       </geometry>
     </visual>
@@ -524,5 +526,5 @@
       <origin rpy="0.06568 0.00000 0.00000" xyz="-1.46578 1.11459 -13.51522"/>
       <geometry>
-        <mesh filename="../meshes/dae/Texture.256.dae" scale="1.00000 1.00000 1.00000"/>
+        <mesh filename="${mesh_dir}/Texture.256.dae" scale="1.00000 1.00000 1.00000"/>
       </geometry>
     </visual>
@@ -531,5 +533,5 @@
       <origin rpy="0.06568 0.00000 0.00000" xyz="-1.46578 1.11459 -13.51522"/>
       <geometry>
-        <mesh filename="../meshes/dae/Texture.257.dae" scale="1.00000 1.00000 1.00000"/>
+        <mesh filename="${mesh_dir}/Texture.257.dae" scale="1.00000 1.00000 1.00000"/>
       </geometry>
     </visual>
@@ -538,5 +540,5 @@
       <origin rpy="0.06568 0.00000 0.00000" xyz="-1.46578 1.11459 -13.51522"/>
       <geometry>
-        <mesh filename="../meshes/dae/Texture.258.dae" scale="1.00000 1.00000 1.00000"/>
+        <mesh filename="${mesh_dir}/Texture.258.dae" scale="1.00000 1.00000 1.00000"/>
       </geometry>
     </visual>
@@ -545,5 +547,5 @@
       <origin rpy="0.06568 0.00000 0.00000" xyz="-1.46578 1.11459 -13.51522"/>
       <geometry>
-        <mesh filename="../meshes/dae/Texture.259.dae" scale="1.00000 1.00000 1.00000"/>
+        <mesh filename="${mesh_dir}/Texture.259.dae" scale="1.00000 1.00000 1.00000"/>
       </geometry>
     </visual>
@@ -552,5 +554,5 @@
       <origin rpy="0.06568 0.00000 0.00000" xyz="-1.46578 1.11459 -13.51522"/>
       <geometry>
-        <mesh filename="../meshes/dae/Texture.260.dae" scale="1.00000 1.00000 1.00000"/>
+        <mesh filename="${mesh_dir}/Texture.260.dae" scale="1.00000 1.00000 1.00000"/>
       </geometry>
     </visual>
@@ -559,5 +561,5 @@
       <origin rpy="0.06568 0.00000 0.00000" xyz="-1.46578 1.11459 -13.51522"/>
       <geometry>
-        <mesh filename="../meshes/dae/Texture.261.dae" scale="1.00000 1.00000 1.00000"/>
+        <mesh filename="${mesh_dir}/Texture.261.dae" scale="1.00000 1.00000 1.00000"/>
       </geometry>
     </visual>
@@ -566,5 +568,5 @@
       <origin rpy="0.06568 0.00000 0.00000" xyz="-1.46578 1.11459 -13.51522"/>
       <geometry>
-        <mesh filename="../meshes/dae/Texture.262.dae" scale="1.00000 1.00000 1.00000"/>
+        <mesh filename="${mesh_dir}/Texture.262.dae" scale="1.00000 1.00000 1.00000"/>
       </geometry>
     </visual>
@@ -573,5 +575,5 @@
       <origin rpy="0.06568 0.00000 0.00000" xyz="-1.46578 1.11459 -13.51522"/>
       <geometry>
-        <mesh filename="../meshes/dae/Texture.263.dae" scale="1.00000 1.00000 1.00000"/>
+        <mesh filename="${mesh_dir}/Texture.263.dae" scale="1.00000 1.00000 1.00000"/>
       </geometry>
     </visual>
@@ -580,5 +582,5 @@
       <origin rpy="0.06568 0.00000 0.00000" xyz="-1.46578 1.11459 -13.51522"/>
       <geometry>
-        <mesh filename="../meshes/dae/Texture.264.dae" scale="1.00000 1.00000 1.00000"/>
+        <mesh filename="${mesh_dir}/Texture.264.dae" scale="1.00000 1.00000 1.00000"/>
       </geometry>
     </visual>
@@ -587,5 +589,5 @@
       <origin rpy="0.06568 0.00000 0.00000" xyz="-1.46578 1.11459 -13.51522"/>
       <geometry>
-        <mesh filename="../meshes/dae/Texture.265.dae" scale="1.00000 1.00000 1.00000"/>
+        <mesh filename="${mesh_dir}/Texture.265.dae" scale="1.00000 1.00000 1.00000"/>
       </geometry>
     </visual>
@@ -594,5 +596,5 @@
       <origin rpy="0.06568 0.00000 0.00000" xyz="-1.46578 1.11459 -13.51522"/>
       <geometry>
-        <mesh filename="../meshes/dae/Texture.266.dae" scale="1.00000 1.00000 1.00000"/>
+        <mesh filename="${mesh_dir}/Texture.266.dae" scale="1.00000 1.00000 1.00000"/>
       </geometry>
     </visual>
@@ -601,5 +603,5 @@
       <origin rpy="0.06568 0.00000 0.00000" xyz="-1.46578 1.11459 -13.51522"/>
       <geometry>
-        <mesh filename="../meshes/dae/Texture.267.dae" scale="1.00000 1.00000 1.00000"/>
+        <mesh filename="${mesh_dir}/Texture.267.dae" scale="1.00000 1.00000 1.00000"/>
       </geometry>
     </visual>
@@ -608,5 +610,5 @@
       <origin rpy="0.06568 0.00000 0.00000" xyz="-1.46578 1.11459 -13.51522"/>
       <geometry>
-        <mesh filename="../meshes/dae/Texture.268.dae" scale="1.00000 1.00000 1.00000"/>
+        <mesh filename="${mesh_dir}/Texture.268.dae" scale="1.00000 1.00000 1.00000"/>
       </geometry>
     </visual>
@@ -615,5 +617,5 @@
       <origin rpy="0.06568 0.00000 0.00000" xyz="-1.46578 1.11459 -13.51522"/>
       <geometry>
-        <mesh filename="../meshes/dae/Texture.269.dae" scale="1.00000 1.00000 1.00000"/>
+        <mesh filename="${mesh_dir}/Texture.269.dae" scale="1.00000 1.00000 1.00000"/>
       </geometry>
     </visual>
@@ -622,5 +624,5 @@
       <origin rpy="0.06568 0.00000 0.00000" xyz="-1.46578 1.11459 -13.51522"/>
       <geometry>
-        <mesh filename="../meshes/dae/Texture.270.dae" scale="1.00000 1.00000 1.00000"/>
+        <mesh filename="${mesh_dir}/Texture.270.dae" scale="1.00000 1.00000 1.00000"/>
       </geometry>
     </visual>
@@ -631,5 +633,5 @@
       <origin rpy="-0.00792 -0.00000 -0.00000" xyz="-2.08983 1.12391 -12.92101"/>
       <geometry>
-        <mesh filename="../meshes/dae/G-__564753.dae" scale="1.00000 1.00000 1.00000"/>
+        <mesh filename="${mesh_dir}/G-__564753.dae" scale="1.00000 1.00000 1.00000"/>
       </geometry>
     </visual>
@@ -638,5 +640,5 @@
       <origin rpy="-0.00792 -0.00000 -0.00000" xyz="-2.08983 1.12391 -12.92101"/>
       <geometry>
-        <mesh filename="../meshes/dae/G-__564753.001.dae" scale="1.00000 1.00000 1.00000"/>
+        <mesh filename="${mesh_dir}/G-__564753.001.dae" scale="1.00000 1.00000 1.00000"/>
       </geometry>
     </visual>
@@ -645,5 +647,5 @@
       <origin rpy="-0.00792 -0.00000 -0.00000" xyz="-2.08983 1.12391 -12.92101"/>
       <geometry>
-        <mesh filename="../meshes/dae/G-__564753.002.dae" scale="1.00000 1.00000 1.00000"/>
+        <mesh filename="${mesh_dir}/G-__564753.002.dae" scale="1.00000 1.00000 1.00000"/>
       </geometry>
     </visual>
@@ -652,5 +654,5 @@
       <origin rpy="-0.00792 -0.00000 -0.00000" xyz="-2.08983 1.12391 -12.92101"/>
       <geometry>
-        <mesh filename="../meshes/dae/G-__564753.003.dae" scale="1.00000 1.00000 1.00000"/>
+        <mesh filename="${mesh_dir}/G-__564753.003.dae" scale="1.00000 1.00000 1.00000"/>
       </geometry>
     </visual>
@@ -659,5 +661,5 @@
       <origin rpy="-0.00792 -0.00000 -0.00000" xyz="-2.08983 1.12391 -12.92101"/>
       <geometry>
-        <mesh filename="../meshes/dae/G-__564753.004.dae" scale="1.00000 1.00000 1.00000"/>
+        <mesh filename="${mesh_dir}/G-__564753.004.dae" scale="1.00000 1.00000 1.00000"/>
       </geometry>
     </visual>
@@ -666,5 +668,5 @@
       <origin rpy="-0.00792 -0.00000 -0.00000" xyz="-2.08983 1.12391 -12.92101"/>
       <geometry>
-        <mesh filename="../meshes/dae/G-__564753.005.dae" scale="1.00000 1.00000 1.00000"/>
+        <mesh filename="${mesh_dir}/G-__564753.005.dae" scale="1.00000 1.00000 1.00000"/>
       </geometry>
     </visual>
@@ -673,5 +675,5 @@
       <origin rpy="-0.00792 -0.00000 -0.00000" xyz="-2.08983 1.12391 -12.92101"/>
       <geometry>
-        <mesh filename="../meshes/dae/G-__564753.006.dae" scale="1.00000 1.00000 1.00000"/>
+        <mesh filename="${mesh_dir}/G-__564753.006.dae" scale="1.00000 1.00000 1.00000"/>
       </geometry>
     </visual>
@@ -680,5 +682,5 @@
       <origin rpy="-0.00792 -0.00000 -0.00000" xyz="-2.08983 1.12391 -12.92101"/>
       <geometry>
-        <mesh filename="../meshes/dae/G-__564753.007.dae" scale="1.00000 1.00000 1.00000"/>
+        <mesh filename="${mesh_dir}/G-__564753.007.dae" scale="1.00000 1.00000 1.00000"/>
       </geometry>
     </visual>
@@ -687,5 +689,5 @@
       <origin rpy="-0.00792 -0.00000 -0.00000" xyz="-2.08983 1.12391 -12.92101"/>
       <geometry>
-        <mesh filename="../meshes/dae/G-__564753.008.dae" scale="1.00000 1.00000 1.00000"/>
+        <mesh filename="${mesh_dir}/G-__564753.008.dae" scale="1.00000 1.00000 1.00000"/>
       </geometry>
     </visual>
@@ -694,5 +696,5 @@
       <origin rpy="-0.00792 -0.00000 -0.00000" xyz="-2.08983 1.12391 -12.92101"/>
       <geometry>
-        <mesh filename="../meshes/dae/G-__564753.009.dae" scale="1.00000 1.00000 1.00000"/>
+        <mesh filename="${mesh_dir}/G-__564753.009.dae" scale="1.00000 1.00000 1.00000"/>
       </geometry>
     </visual>
@@ -701,5 +703,5 @@
       <origin rpy="-0.00792 -0.00000 -0.00000" xyz="-2.08983 1.12391 -12.92101"/>
       <geometry>
-        <mesh filename="../meshes/dae/G-__564753.010.dae" scale="1.00000 1.00000 1.00000"/>
+        <mesh filename="${mesh_dir}/G-__564753.010.dae" scale="1.00000 1.00000 1.00000"/>
       </geometry>
     </visual>
@@ -708,5 +710,5 @@
       <origin rpy="-0.00792 -0.00000 -0.00000" xyz="-2.08983 1.12391 -12.92101"/>
       <geometry>
-        <mesh filename="../meshes/dae/G-__564753.011.dae" scale="1.00000 1.00000 1.00000"/>
+        <mesh filename="${mesh_dir}/G-__564753.011.dae" scale="1.00000 1.00000 1.00000"/>
       </geometry>
     </visual>
@@ -715,5 +717,5 @@
       <origin rpy="-0.00792 -0.00000 -0.00000" xyz="-2.08983 1.12391 -12.92101"/>
       <geometry>
-        <mesh filename="../meshes/dae/G-__564753.012.dae" scale="1.00000 1.00000 1.00000"/>
+        <mesh filename="${mesh_dir}/G-__564753.012.dae" scale="1.00000 1.00000 1.00000"/>
       </geometry>
     </visual>
@@ -722,5 +724,5 @@
       <origin rpy="-0.00792 -0.00000 -0.00000" xyz="-2.08983 1.12391 -12.92101"/>
       <geometry>
-        <mesh filename="../meshes/dae/G-__564753.013.dae" scale="1.00000 1.00000 1.00000"/>
+        <mesh filename="${mesh_dir}/G-__564753.013.dae" scale="1.00000 1.00000 1.00000"/>
       </geometry>
     </visual>
@@ -729,5 +731,5 @@
       <origin rpy="-0.00792 -0.00000 -0.00000" xyz="-2.08983 1.12391 -12.92101"/>
       <geometry>
-        <mesh filename="../meshes/dae/G-__564753.014.dae" scale="1.00000 1.00000 1.00000"/>
+        <mesh filename="${mesh_dir}/G-__564753.014.dae" scale="1.00000 1.00000 1.00000"/>
       </geometry>
     </visual>
@@ -736,5 +738,5 @@
       <origin rpy="-0.00792 -0.00000 -0.00000" xyz="-2.08983 1.12391 -12.92101"/>
       <geometry>
-        <mesh filename="../meshes/dae/G-__564753.015.dae" scale="1.00000 1.00000 1.00000"/>
+        <mesh filename="${mesh_dir}/G-__564753.015.dae" scale="1.00000 1.00000 1.00000"/>
       </geometry>
     </visual>
@@ -743,5 +745,5 @@
       <origin rpy="-0.00792 -0.00000 -0.00000" xyz="-2.08983 1.12391 -12.92101"/>
       <geometry>
-        <mesh filename="../meshes/dae/G-__564753.016.dae" scale="1.00000 1.00000 1.00000"/>
+        <mesh filename="${mesh_dir}/G-__564753.016.dae" scale="1.00000 1.00000 1.00000"/>
       </geometry>
     </visual>
@@ -750,5 +752,5 @@
       <origin rpy="-0.00792 -0.00000 -0.00000" xyz="-2.08983 1.12391 -12.92101"/>
       <geometry>
-        <mesh filename="../meshes/dae/G-__564753.017.dae" scale="1.00000 1.00000 1.00000"/>
+        <mesh filename="${mesh_dir}/G-__564753.017.dae" scale="1.00000 1.00000 1.00000"/>
       </geometry>
     </visual>
@@ -757,5 +759,5 @@
       <origin rpy="-0.00792 -0.00000 -0.00000" xyz="-2.08983 1.12391 -12.92101"/>
       <geometry>
-        <mesh filename="../meshes/dae/G-__564753.018.dae" scale="1.00000 1.00000 1.00000"/>
+        <mesh filename="${mesh_dir}/G-__564753.018.dae" scale="1.00000 1.00000 1.00000"/>
       </geometry>
     </visual>
@@ -764,5 +766,5 @@
       <origin rpy="-0.00792 -0.00000 -0.00000" xyz="-2.08983 1.12391 -12.92101"/>
       <geometry>
-        <mesh filename="../meshes/dae/G-__564753.019.dae" scale="1.00000 1.00000 1.00000"/>
+        <mesh filename="${mesh_dir}/G-__564753.019.dae" scale="1.00000 1.00000 1.00000"/>
       </geometry>
     </visual>
@@ -771,5 +773,5 @@
       <origin rpy="-0.00792 -0.00000 -0.00000" xyz="-2.08983 1.12391 -12.92101"/>
       <geometry>
-        <mesh filename="../meshes/dae/G-__564753.020.dae" scale="1.00000 1.00000 1.00000"/>
+        <mesh filename="${mesh_dir}/G-__564753.020.dae" scale="1.00000 1.00000 1.00000"/>
       </geometry>
     </visual>
@@ -780,5 +782,5 @@
       <origin rpy="-0.00000 0.00000 0.00000" xyz="-2.07702 0.12073 -10.83652"/>
       <geometry>
-        <mesh filename="../meshes/dae/Texture.007.dae" scale="1.00000 1.00000 1.00000"/>
+        <mesh filename="${mesh_dir}/Texture.007.dae" scale="1.00000 1.00000 1.00000"/>
       </geometry>
     </visual>
@@ -787,5 +789,5 @@
       <origin rpy="-0.00000 0.00000 0.00000" xyz="-2.07702 0.12073 -10.83652"/>
       <geometry>
-        <mesh filename="../meshes/dae/Texture.236.dae" scale="1.00000 1.00000 1.00000"/>
+        <mesh filename="${mesh_dir}/Texture.236.dae" scale="1.00000 1.00000 1.00000"/>
       </geometry>
     </visual>
@@ -794,5 +796,5 @@
       <origin rpy="-0.00000 0.00000 0.00000" xyz="-2.07702 0.12073 -10.83652"/>
       <geometry>
-        <mesh filename="../meshes/dae/Texture.237.dae" scale="1.00000 1.00000 1.00000"/>
+        <mesh filename="${mesh_dir}/Texture.237.dae" scale="1.00000 1.00000 1.00000"/>
       </geometry>
     </visual>
@@ -801,5 +803,5 @@
       <origin rpy="-0.00000 0.00000 0.00000" xyz="-2.07702 0.12073 -10.83652"/>
       <geometry>
-        <mesh filename="../meshes/dae/Texture.238.dae" scale="1.00000 1.00000 1.00000"/>
+        <mesh filename="${mesh_dir}/Texture.238.dae" scale="1.00000 1.00000 1.00000"/>
       </geometry>
     </visual>
@@ -808,5 +810,5 @@
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
File: inmoov/urdf/inmoov.urdf.xacro (robot description, xacro)
@@ -2,6 +2,6 @@
 <robot xmlns:xacro="http://wiki.ros.org/xacro" name="r6bot">
   <!-- Import inmoov physical description (urdf) macro -->
-  <xacro:include filename="/home/dev/thais_urdf/inmoov/urdf/robot_description.urdf.xacro"/>
+  <xacro:include filename="/home/samuel/sentience/local_ws/src/thais_urdf/inmoov/3dmodel/robot_description.urdf.xacro"/>
   <!-- Import inmoov ros2_control description -->
-  <xacro:include filename="/home/dev/thais_urdf/inmoov/ros2_control/inmoov_ros2_control.xacro" />
+  <xacro:include filename="/home/samuel/sentience/local_ws/src/thais_urdf/inmoov/ros2_control/inmoov_ros2_control.xacro" />
 </robot>
