Commit message: evol(urdf): rviz ros2control
Signed-off-by: Charles Madjeri <charles@madjeri.com>

File: inmoov/3dmodel/robot_description.urdf.xacro (robot description, xacro)
@@ -1,5 +1,5 @@
 <?xml version="1.0"?>
 <robot xmlns:xacro="http://www.ros.org/wiki/xacro" name="inmoov" version="1.0">
-  <xacro:property name="mesh_dir" value="file:///home/samuel/sentience/local_ws/src/thais_urdf/inmoov/meshes/dae"/>
+  <!-- mesh_dir set by parent (inmoov.urdf.xacro) from base_path -->
   <joint name="Empty.001_link_joint" type="fixed">
     <origin rpy="0.00000 0.00000 0.00000" xyz="-0.00394 0.00025 -0.19163"/>
@@ -408,5 +408,5 @@
   <link name="base_node">
     <visual name="stand">
-      <material name="None"/>
+      <material name="Gazebo/Grey"/>
       <origin rpy="3.14159 -0.00000 3.14159" xyz="-0.00394 -0.00730 9.35280"/>
       <geometry>
@@ -414,6 +414,23 @@
       </geometry>
     </visual>
-  </link>
-  <link name="stand_link"/>
+    <!-- Minimal collision and inertial so sdformat/urdf2sdf includes this root link in Gazebo -->
+    <collision name="base_node_collision">
+      <geometry><box size="0.01 0.01 0.01"/></geometry>
+    </collision>
+    <inertial>
+      <mass value="0.001"/>
+      <inertia ixx="1e-6" ixy="0" ixz="0" iyy="1e-6" iyz="0" izz="1e-6"/>
+    </inertial>
+  </link>
+  <link name="stand_link">
+    <!-- Minimal geometry so urdf2sdf does not drop this link in Gazebo -->
+    <collision name="stand_link_collision">
+      <geometry><box size="0.01 0.01 0.01"/></geometry>
+    </collision>
+    <inertial>
+      <mass value="0.001"/>
+      <inertia ixx="1e-6" ixy="0" ixz="0" iyy="1e-6" iyz="0" izz="1e-6"/>
+    </inertial>
+  </link>
   <link name="i01.head.eyeRight.001_link"/>
   <link name="i01.head.eyeRight_link">

File: inmoov/ros2_control/inmoov_ros2_control.xacro (robot description, xacro)
@@ -8,26 +8,27 @@
           <param name="node_name">lucy_hardware_interface_left_arm</param>
       </hardware>
-      <joint name="left_shoulder_yaw">
+      <!-- Joint names must match URDF exactly for correct TF tree in RViz/Gazebo -->
+      <joint name="left_shoulder_y_link_joint">
           <command_interface name="position">
           </command_interface>
           <state_interface name="position" />
       </joint>
-      <joint name="left_shoulder_roll">
+      <joint name="left_shoulder_x_link_joint">
           <command_interface name="position" />
           <state_interface name="position" />
       </joint>
-      <joint name="left_elbow">
+      <joint name="left_elbow_x_link_joint">
           <command_interface name="position" />
           <state_interface name="position" />
       </joint>
-      <joint name="left_wrist">
+      <joint name="left_wrist_z_link_joint">
           <command_interface name="position" />
           <state_interface name="position" />
       </joint>
-      <joint name="left_thumb">
+      <joint name="i01.leftHand.thumb_link_joint">
           <command_interface name="position" />
           <state_interface name="position" />
       </joint>
-      <joint name="left_index">
+      <joint name="i01.leftHand.index_link_joint">
           <command_interface name="position">
           <param name="min">0</param>
@@ -36,13 +37,13 @@
           <state_interface name="position" />
       </joint>
-      <joint name="left_middle">
+      <joint name="i01.leftHand.majeure_link_joint">
           <command_interface name="position" />
           <state_interface name="position" />
       </joint>
-      <joint name="left_ring">
+      <joint name="i01.leftHand.ringFinger_link_joint">
           <command_interface name="position" />
           <state_interface name="position" />
       </joint>
-      <joint name="left_pinky">
+      <joint name="i01.leftHand.pinky_link_joint">
           <command_interface name="position" />
           <state_interface name="position" />
@@ -56,10 +57,11 @@
           <param name="node_name">lucy_hardware_interface_right_arm</param>
       </hardware>
-      <joint name="right_shoulder_yaw">
+      <!-- Joint names must match URDF exactly (URDF has right_elbow without _link_joint) -->
+      <joint name="right_shoulder_y_link_joint">
           <command_interface name="position">
           </command_interface>
           <state_interface name="position" />
       </joint>
-      <joint name="right_shoulder_roll">
+      <joint name="right_shoulder_x_link_joint">
           <command_interface name="position" />
           <state_interface name="position" />
@@ -69,13 +71,13 @@
           <state_interface name="position" />
       </joint>
-      <joint name="right_wrist">
+      <joint name="right_wrist_z_link_joint">
           <command_interface name="position" />
           <state_interface name="position" />
       </joint>
-      <joint name="right_thumb">
+      <joint name="i01.rightHand.thumb_link_joint">
           <command_interface name="position" />
           <state_interface name="position" />
       </joint>
-      <joint name="right_index">
+      <joint name="i01.rightHand.index_link_joint">
           <command_interface name="position">
           <param name="min">0</param>
@@ -84,13 +86,13 @@
           <state_interface name="position" />
       </joint>
-      <joint name="right_middle">
+      <joint name="i01.rightHand.majeure_link_joint">
           <command_interface name="position" />
           <state_interface name="position" />
       </joint>
-      <joint name="right_ring">
+      <joint name="i01.rightHand.ringFinger_link_joint">
           <command_interface name="position" />
           <state_interface name="position" />
       </joint>
-      <joint name="right_pinky">
+      <joint name="i01.rightHand.pinky_link_joint">
           <command_interface name="position" />
           <state_interface name="position" />

File: inmoov/urdf/inmoov.urdf.xacro (robot description, xacro)
@@ -1,7 +1,10 @@
 <?xml version="1.0"?>
 <robot xmlns:xacro="http://wiki.ros.org/xacro" name="r6bot">
+  <!-- base_path: set by launch file (host-independent). When running xacro standalone, use . or pass base_path. -->
+  <xacro:arg name="base_path" default="."/>
+  <xacro:property name="mesh_dir" value="file://$(arg base_path)/meshes/dae"/>
   <!-- Import inmoov physical description (urdf) macro -->
-  <xacro:include filename="/home/samuel/sentience/local_ws/src/thais_urdf/inmoov/3dmodel/robot_description.urdf.xacro"/>
+  <xacro:include filename="../3dmodel/robot_description.urdf.xacro"/>
   <!-- Import inmoov ros2_control description -->
-  <xacro:include filename="/home/samuel/sentience/local_ws/src/thais_urdf/inmoov/ros2_control/inmoov_ros2_control.xacro" />
+  <xacro:include filename="../ros2_control/inmoov_ros2_control.xacro" />
 </robot>
