Commit message: feat(gazebo): add gazebo and rviz support
Signed-off-by: Charles Madjeri <charles@madjeri.com>

File: inmoov/3dmodel/robot_description.urdf.xacro (robot description, xacro)
@@ -1,5 +1,5 @@
 <?xml version="1.0"?>
 <robot xmlns:xacro="http://www.ros.org/wiki/xacro" name="inmoov" version="1.0">
-  <!-- mesh_dir set by parent (inmoov.urdf.xacro) from base_path -->
+  <!-- mesh_dir and use_gazebo_sim set by parent (inmoov.urdf.xacro) -->
   <joint name="Empty.001_link_joint" type="fixed">
     <origin rpy="0.00000 0.00000 0.00000" xyz="-0.00394 0.00025 -0.19163"/>
@@ -419,6 +419,12 @@
     </collision>
     <inertial>
-      <mass value="0.001"/>
-      <inertia ixx="1e-6" ixy="0" ixz="0" iyy="1e-6" iyz="0" izz="1e-6"/>
+      <xacro:if value="${use_gazebo_sim}">
+        <mass value="10000"/>
+        <inertia ixx="100" ixy="0" ixz="0" iyy="100" iyz="0" izz="100"/>
+      </xacro:if>
+      <xacro:unless value="${use_gazebo_sim}">
+        <mass value="0.001"/>
+        <inertia ixx="1e-6" ixy="0" ixz="0" iyy="1e-6" iyz="0" izz="1e-6"/>
+      </xacro:unless>
     </inertial>
   </link>
@@ -429,9 +435,17 @@
     </collision>
     <inertial>
-      <mass value="0.001"/>
-      <inertia ixx="1e-6" ixy="0" ixz="0" iyy="1e-6" iyz="0" izz="1e-6"/>
+      <xacro:if value="${use_gazebo_sim}">
+        <mass value="10000"/>
+        <inertia ixx="100" ixy="0" ixz="0" iyy="100" iyz="0" izz="100"/>
+      </xacro:if>
+      <xacro:unless value="${use_gazebo_sim}">
+        <mass value="0.001"/>
+        <inertia ixx="1e-6" ixy="0" ixz="0" iyy="1e-6" iyz="0" izz="1e-6"/>
+      </xacro:unless>
     </inertial>
   </link>
-  <link name="i01.head.eyeRight.001_link"/>
+  <link name="i01.head.eyeRight.001_link">
+    <inertial><mass value="0.001"/><inertia ixx="1e-6" ixy="0" ixz="0" iyy="1e-6" iyz="0" izz="1e-6"/></inertial>
+  </link>
   <link name="i01.head.eyeRight_link">
     <visual name="i01.head.eyeRight.full">
@@ -442,4 +456,5 @@
       </geometry>
     </visual>
+    <inertial><mass value="0.001"/><inertia ixx="1e-6" ixy="0" ixz="0" iyy="1e-6" iyz="0" izz="1e-6"/></inertial>
   </link>
   <link name="i01.head.jaw_link">
@@ -465,4 +480,5 @@
       </geometry>
     </visual>
+    <inertial><mass value="0.001"/><inertia ixx="1e-6" ixy="0" ixz="0" iyy="1e-6" iyz="0" izz="1e-6"/></inertial>
   </link>
   <link name="left_shoulder_y_link">
@@ -516,4 +532,5 @@
       </geometry>
     </visual>
+    <inertial><mass value="0.001"/><inertia ixx="1e-6" ixy="0" ixz="0" iyy="1e-6" iyz="0" izz="1e-6"/></inertial>
   </link>
   <link name="left_shoulder_x_link">
@@ -602,18 +619,4 @@
       </geometry>
     </visual>
-    <visual name="i01..leftArm.shoulder.full.012">
-      <material name="Material.390"/>
-      <origin rpy="0.06568 0.00000 0.00000" xyz="-1.46578 1.11459 -13.51522"/>
-      <geometry>
-        <mesh filename="${mesh_dir}/Texture.265.dae" scale="1.00000 1.00000 1.00000"/>
-      </geometry>
-    </visual>
-    <visual name="i01..leftArm.shoulder.full.013">
-      <material name="Material.390"/>
-      <origin rpy="0.06568 0.00000 0.00000" xyz="-1.46578 1.11459 -13.51522"/>
-      <geometry>
-        <mesh filename="${mesh_dir}/Texture.266.dae" scale="1.00000 1.00000 1.00000"/>
-      </geometry>
-    </visual>
     <visual name="i01..leftArm.shoulder.full.014">
       <material name="Material.390"/>
@@ -644,4 +647,5 @@
       </geometry>
     </visual>
+    <inertial><mass value="0.001"/><inertia ixx="1e-6" ixy="0" ixz="0" iyy="1e-6" iyz="0" izz="1e-6"/></inertial>
   </link>
   <link name="left_shoulder_z_link">
@@ -793,4 +797,5 @@
       </geometry>
     </visual>
+    <inertial><mass value="0.001"/><inertia ixx="1e-6" ixy="0" ixz="0" iyy="1e-6" iyz="0" izz="1e-6"/></inertial>
   </link>
   <link name="left_elbow_x_link">
@@ -886,4 +891,5 @@
       </geometry>
     </visual>
+    <inertial><mass value="0.001"/><inertia ixx="1e-6" ixy="0" ixz="0" iyy="1e-6" iyz="0" izz="1e-6"/></inertial>
   </link>
   <link name="left_wrist_z_link">
@@ -895,4 +901,5 @@
       </geometry>
     </visual>
+    <inertial><mass value="0.001"/><inertia ixx="1e-6" ixy="0" ixz="0" iyy="1e-6" iyz="0" izz="1e-6"/></inertial>
   </link>
   <link name="i01.leftHand.wrist.001_link">
@@ -904,4 +911,5 @@
       </geometry>
     </visual>
+    <inertial><mass value="0.001"/><inertia ixx="1e-6" ixy="0" ixz="0" iyy="1e-6" iyz="0" izz="1e-6"/></inertial>
   </link>
   <link name="i01.leftHand.index_link">
@@ -913,4 +921,5 @@
       </geometry>
     </visual>
+    <inertial><mass value="0.001"/><inertia ixx="1e-6" ixy="0" ixz="0" iyy="1e-6" iyz="0" izz="1e-6"/></inertial>
   </link>
   <link name="torso_bottom_link">
@@ -985,4 +994,9 @@
       </geometry>
     </visual>
+    <!-- Minimal inertial so urdf2sdf includes this link in Gazebo (required for child links/joints) -->
+    <inertial>
+      <mass value="0.001"/>
+      <inertia ixx="1e-6" ixy="0" ixz="0" iyy="1e-6" iyz="0" izz="1e-6"/>
+    </inertial>
   </link>
   <link name="i01.leftHand.index2_link">
@@ -994,4 +1008,5 @@
       </geometry>
     </visual>
+    <inertial><mass value="0.001"/><inertia ixx="1e-6" ixy="0" ixz="0" iyy="1e-6" iyz="0" izz="1e-6"/></inertial>
   </link>
   <link name="i01.leftHand.index3_link">
@@ -1003,4 +1018,5 @@
       </geometry>
     </visual>
+    <inertial><mass value="0.001"/><inertia ixx="1e-6" ixy="0" ixz="0" iyy="1e-6" iyz="0" izz="1e-6"/></inertial>
   </link>
   <link name="i01.leftHand.majeure_link">
@@ -1012,4 +1028,5 @@
       </geometry>
     </visual>
+    <inertial><mass value="0.001"/><inertia ixx="1e-6" ixy="0" ixz="0" iyy="1e-6" iyz="0" izz="1e-6"/></inertial>
   </link>
   <link name="i01.leftHand.majeure2_link">
@@ -1021,4 +1038,5 @@
       </geometry>
     </visual>
+    <inertial><mass value="0.001"/><inertia ixx="1e-6" ixy="0" ixz="0" iyy="1e-6" iyz="0" izz="1e-6"/></inertial>
   </link>
   <link name="i01.leftHand.majeure3_link">
@@ -1030,4 +1048,5 @@
       </geometry>
     </visual>
+    <inertial><mass value="0.001"/><inertia ixx="1e-6" ixy="0" ixz="0" iyy="1e-6" iyz="0" izz="1e-6"/></inertial>
   </link>
   <link name="i01.leftHand.pinky0_link">
@@ -1039,4 +1058,5 @@
       </geometry>
     </visual>
+    <inertial><mass value="0.001"/><inertia ixx="1e-6" ixy="0" ixz="0" iyy="1e-6" iyz="0" izz="1e-6"/></inertial>
   </link>
   <link name="i01.leftHand.pinky_link">
@@ -1048,4 +1068,5 @@
       </geometry>
     </visual>
+    <inertial><mass value="0.001"/><inertia ixx="1e-6" ixy="0" ixz="0" iyy="1e-6" iyz="0" izz="1e-6"/></inertial>
   </link>
   <link name="i01.leftHand.pinky2_link">
@@ -1057,4 +1078,5 @@
       </geometry>
     </visual>
+    <inertial><mass value="0.001"/><inertia ixx="1e-6" ixy="0" ixz="0" iyy="1e-6" iyz="0" izz="1e-6"/></inertial>
   </link>
   <link name="i01.leftHand.pinky3_link">
@@ -1066,4 +1088,5 @@
       </geometry>
     </visual>
+    <inertial><mass value="0.001"/><inertia ixx="1e-6" ixy="0" ixz="0" iyy="1e-6" iyz="0" izz="1e-6"/></inertial>
   </link>
   <link name="i01.leftHand.ringfinger0_link">
@@ -1075,4 +1098,5 @@
       </geometry>
     </visual>
+    <inertial><mass value="0.001"/><inertia ixx="1e-6" ixy="0" ixz="0" iyy="1e-6" iyz="0" izz="1e-6"/></inertial>
   </link>
   <link name="torso_z_link">
@@ -1280,4 +1304,9 @@
       </geometry>
     </visual>
+    <!-- Minimal inertial so urdf2sdf includes this link in Gazebo -->
+    <inertial>
+      <mass value="0.001"/>
+      <inertia ixx="1e-6" ixy="0" ixz="0" iyy="1e-6" iyz="0" izz="1e-6"/>
+    </inertial>
   </link>
   <link name="i01.leftHand.ringFinger_link">
@@ -1289,4 +1318,5 @@
       </geometry>
     </visual>
+    <inertial><mass value="0.001"/><inertia ixx="1e-6" ixy="0" ixz="0" iyy="1e-6" iyz="0" izz="1e-6"/></inertial>
   </link>
   <link name="i01.leftHand.ringfinger2_link">
@@ -1298,4 +1328,5 @@
       </geometry>
     </visual>
+    <inertial><mass value="0.001"/><inertia ixx="1e-6" ixy="0" ixz="0" iyy="1e-6" iyz="0" izz="1e-6"/></inertial>
   </link>
   <link name="i01.leftHand.ringfinger3_link">
@@ -1307,4 +1338,5 @@
       </geometry>
     </visual>
+    <inertial><mass value="0.001"/><inertia ixx="1e-6" ixy="0" ixz="0" iyy="1e-6" iyz="0" izz="1e-6"/></inertial>
   </link>
   <link name="i01.leftHand.thumb1_link">
@@ -1316,4 +1348,5 @@
       </geometry>
     </visual>
+    <inertial><mass value="0.001"/><inertia ixx="1e-6" ixy="0" ixz="0" iyy="1e-6" iyz="0" izz="1e-6"/></inertial>
   </link>
   <link name="i01.leftHand.thumb_link">
@@ -1325,4 +1358,5 @@
       </geometry>
     </visual>
+    <inertial><mass value="0.001"/><inertia ixx="1e-6" ixy="0" ixz="0" iyy="1e-6" iyz="0" izz="1e-6"/></inertial>
   </link>
   <link name="i01.leftHand.thumb3_link">
@@ -1334,4 +1368,5 @@
       </geometry>
     </visual>
+    <inertial><mass value="0.001"/><inertia ixx="1e-6" ixy="0" ixz="0" iyy="1e-6" iyz="0" izz="1e-6"/></inertial>
   </link>
   <link name="right_shoulder_y_link">
@@ -1385,4 +1420,5 @@
       </geometry>
     </visual>
+    <inertial><mass value="0.001"/><inertia ixx="1e-6" ixy="0" ixz="0" iyy="1e-6" iyz="0" izz="1e-6"/></inertial>
   </link>
   <link name="right_shoulder_x_link">
@@ -1471,4 +1507,5 @@
       </geometry>
     </visual>
+    <inertial><mass value="0.001"/><inertia ixx="1e-6" ixy="0" ixz="0" iyy="1e-6" iyz="0" izz="1e-6"/></inertial>
   </link>
   <link name="right_shoulder_z_link">
@@ -1613,11 +1650,5 @@
       </geometry>
     </visual>
-    <visual name="i01.rightArm.rotate.full.020">
-      <material name="[0131_Silver]"/>
-      <origin rpy="3.13367 0.00000 0.00000" xyz="2.08983 1.12392 -12.92101"/>
-      <geometry>
-        <mesh filename="${mesh_dir}/G-__566220.020.dae" scale="1.00000 1.00000 1.00000"/>
-      </geometry>
-    </visual>
+    <inertial><mass value="0.001"/><inertia ixx="1e-6" ixy="0" ixz="0" iyy="1e-6" iyz="0" izz="1e-6"/></inertial>
   </link>
   <link name="right_elbow_x_link">
@@ -1713,4 +1744,5 @@
       </geometry>
     </visual>
+    <inertial><mass value="0.001"/><inertia ixx="1e-6" ixy="0" ixz="0" iyy="1e-6" iyz="0" izz="1e-6"/></inertial>
   </link>
   <link name="torso_y_link">
@@ -2275,4 +2307,9 @@
       </geometry>
     </visual>
+    <!-- Minimal inertial so urdf2sdf includes this link in Gazebo -->
+    <inertial>
+      <mass value="0.001"/>
+      <inertia ixx="1e-6" ixy="0" ixz="0" iyy="1e-6" iyz="0" izz="1e-6"/>
+    </inertial>
   </link>
   <link name="right_wrist_z_link">
@@ -2284,4 +2321,5 @@
       </geometry>
     </visual>
+    <inertial><mass value="0.001"/><inertia ixx="1e-6" ixy="0" ixz="0" iyy="1e-6" iyz="0" izz="1e-6"/></inertial>
   </link>
   <link name="i01.rightHand.wrist.001_link">
@@ -2293,4 +2331,5 @@
       </geometry>
     </visual>
+    <inertial><mass value="0.001"/><inertia ixx="1e-6" ixy="0" ixz="0" iyy="1e-6" iyz="0" izz="1e-6"/></inertial>
   </link>
   <link name="i01.rightHand.index_link">
@@ -2302,4 +2341,5 @@
       </geometry>
     </visual>
+    <inertial><mass value="0.001"/><inertia ixx="1e-6" ixy="0" ixz="0" iyy="1e-6" iyz="0" izz="1e-6"/></inertial>
   </link>
   <link name="i01.rightHand.index2_link">
@@ -2311,4 +2351,5 @@
       </geometry>
     </visual>
+    <inertial><mass value="0.001"/><inertia ixx="1e-6" ixy="0" ixz="0" iyy="1e-6" iyz="0" izz="1e-6"/></inertial>
   </link>
   <link name="i01.rightHand.index3_link">
@@ -2320,4 +2361,5 @@
       </geometry>
     </visual>
+    <inertial><mass value="0.001"/><inertia ixx="1e-6" ixy="0" ixz="0" iyy="1e-6" iyz="0" izz="1e-6"/></inertial>
   </link>
   <link name="i01.rightHand.majeure_link">
@@ -2329,4 +2371,5 @@
       </geometry>
     </visual>
+    <inertial><mass value="0.001"/><inertia ixx="1e-6" ixy="0" ixz="0" iyy="1e-6" iyz="0" izz="1e-6"/></inertial>
   </link>
   <link name="i01.rightHand.majeure2_link">
@@ -2338,4 +2381,5 @@
       </geometry>
     </visual>
+    <inertial><mass value="0.001"/><inertia ixx="1e-6" ixy="0" ixz="0" iyy="1e-6" iyz="0" izz="1e-6"/></inertial>
   </link>
   <link name="i01.rightHand.majeure3_link">
@@ -2347,4 +2391,5 @@
       </geometry>
     </visual>
+    <inertial><mass value="0.001"/><inertia ixx="1e-6" ixy="0" ixz="0" iyy="1e-6" iyz="0" izz="1e-6"/></inertial>
   </link>
   <link name="i01.rightHand.pinky0_link">
@@ -2356,4 +2401,5 @@
       </geometry>
     </visual>
+    <inertial><mass value="0.001"/><inertia ixx="1e-6" ixy="0" ixz="0" iyy="1e-6" iyz="0" izz="1e-6"/></inertial>
   </link>
   <link name="i01.rightHand.pinky_link">
@@ -2365,6 +2411,9 @@
       </geometry>
     </visual>
-  </link>
-  <link name="i01.head.neck.001_link"/>
+    <inertial><mass value="0.001"/><inertia ixx="1e-6" ixy="0" ixz="0" iyy="1e-6" iyz="0" izz="1e-6"/></inertial>
+  </link>
+  <link name="i01.head.neck.001_link">
+    <inertial><mass value="0.001"/><inertia ixx="1e-6" ixy="0" ixz="0" iyy="1e-6" iyz="0" izz="1e-6"/></inertial>
+  </link>
   <link name="i01.rightHand.pinky2_link">
     <visual name="i01.rightHand.pinkyPhal2">
@@ -2375,4 +2424,5 @@
       </geometry>
     </visual>
+    <inertial><mass value="0.001"/><inertia ixx="1e-6" ixy="0" ixz="0" iyy="1e-6" iyz="0" izz="1e-6"/></inertial>
   </link>
   <link name="i01.rightHand.pinky3_link">
@@ -2384,4 +2434,5 @@
       </geometry>
     </visual>
+    <inertial><mass value="0.001"/><inertia ixx="1e-6" ixy="0" ixz="0" iyy="1e-6" iyz="0" izz="1e-6"/></inertial>
   </link>
   <link name="i01.rightHand.ringfinger0_link">
@@ -2393,4 +2444,5 @@
       </geometry>
     </visual>
+    <inertial><mass value="0.001"/><inertia ixx="1e-6" ixy="0" ixz="0" iyy="1e-6" iyz="0" izz="1e-6"/></inertial>
   </link>
   <link name="i01.rightHand.ringFinger_link">
@@ -2402,4 +2454,5 @@
       </geometry>
     </visual>
+    <inertial><mass value="0.001"/><inertia ixx="1e-6" ixy="0" ixz="0" iyy="1e-6" iyz="0" izz="1e-6"/></inertial>
   </link>
   <link name="i01.rightHand.ringfinger2_link">
@@ -2411,4 +2464,5 @@
       </geometry>
     </visual>
+    <inertial><mass value="0.001"/><inertia ixx="1e-6" ixy="0" ixz="0" iyy="1e-6" iyz="0" izz="1e-6"/></inertial>
   </link>
   <link name="i01.rightHand.ringfinger3_link">
@@ -2420,4 +2474,5 @@
       </geometry>
     </visual>
+    <inertial><mass value="0.001"/><inertia ixx="1e-6" ixy="0" ixz="0" iyy="1e-6" iyz="0" izz="1e-6"/></inertial>
   </link>
   <link name="i01.rightHand.thumb1_link">
@@ -2429,4 +2484,5 @@
       </geometry>
     </visual>
+    <inertial><mass value="0.001"/><inertia ixx="1e-6" ixy="0" ixz="0" iyy="1e-6" iyz="0" izz="1e-6"/></inertial>
   </link>
   <link name="i01.rightHand.thumb_link">
@@ -2438,4 +2494,5 @@
       </geometry>
     </visual>
+    <inertial><mass value="0.001"/><inertia ixx="1e-6" ixy="0" ixz="0" iyy="1e-6" iyz="0" izz="1e-6"/></inertial>
   </link>
   <link name="i01.rightHand.thumb3_link">
@@ -2447,4 +2504,5 @@
       </geometry>
     </visual>
+    <inertial><mass value="0.001"/><inertia ixx="1e-6" ixy="0" ixz="0" iyy="1e-6" iyz="0" izz="1e-6"/></inertial>
   </link>
   <link name="neck_link">
@@ -2477,4 +2535,5 @@
       </geometry>
     </visual>
+    <inertial><mass value="0.001"/><inertia ixx="1e-6" ixy="0" ixz="0" iyy="1e-6" iyz="0" izz="1e-6"/></inertial>
   </link>
   <link name="i01.head.rothead_link">
@@ -2591,6 +2650,9 @@
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
File: inmoov/ros2_control/inmoov_ros2_control.xacro (robot description, xacro)
@@ -1,10 +1,15 @@
 <?xml version="1.0"?>
 <robot xmlns:xacro="http://www.ros.org/wiki/xacro" name="inmoov" version="1.0">
+  <xacro:arg name="use_gazebo_sim" default="false" />
 <ros2_control name="LucyHardwareLeftArm" type="system">
       <hardware>
-          <plugin>lucy_ros2_control/LucySystemHardware</plugin>
-          <!-- <plugin>mock_components/GenericSystem</plugin> -->
-          <param name="publisher_topic">joints/left_arm</param>
-          <param name="node_name">lucy_hardware_interface_left_arm</param>
+          <xacro:if value="$(arg use_gazebo_sim)">
+            <plugin>gz_ros2_control/GazeboSimSystem</plugin>
+          </xacro:if>
+          <xacro:unless value="$(arg use_gazebo_sim)">
+            <plugin>lucy_ros2_control/LucySystemHardware</plugin>
+            <param name="publisher_topic">joints/left_arm</param>
+            <param name="node_name">lucy_hardware_interface_left_arm</param>
+          </xacro:unless>
       </hardware>
       <!-- Joint names must match URDF exactly for correct TF tree in RViz/Gazebo -->
@@ -52,8 +57,12 @@
   <ros2_control name="LucyHardwareRightArm" type="system">
       <hardware>
-          <plugin>lucy_ros2_control/LucySystemHardware</plugin>
-          <!-- <plugin>mock_components/GenericSystem</plugin> -->
-          <param name="publisher_topic">joints/right_arm</param>
-          <param name="node_name">lucy_hardware_interface_right_arm</param>
+          <xacro:if value="$(arg use_gazebo_sim)">
+            <plugin>gz_ros2_control/GazeboSimSystem</plugin>
+          </xacro:if>
+          <xacro:unless value="$(arg use_gazebo_sim)">
+            <plugin>lucy_ros2_control/LucySystemHardware</plugin>
+            <param name="publisher_topic">joints/right_arm</param>
+            <param name="node_name">lucy_hardware_interface_right_arm</param>
+          </xacro:unless>
       </hardware>
       <!-- Joint names must match URDF exactly (URDF has right_elbow without _link_joint) -->

File: inmoov/urdf/inmoov.urdf.xacro (robot description, xacro)
@@ -3,8 +3,15 @@
   <!-- base_path: set by launch file (host-independent). When running xacro standalone, use . or pass base_path. -->
   <xacro:arg name="base_path" default="."/>
+  <xacro:arg name="use_gazebo_sim" default="false"/>
+  <xacro:arg name="controller_config" default=""/>
   <xacro:property name="mesh_dir" value="file://$(arg base_path)/meshes/dae"/>
-  <!-- Import inmoov physical description (urdf) macro -->
+  <xacro:property name="use_gazebo_sim" value="$(arg use_gazebo_sim)"/>
+  <!-- Import inmoov physical description (urdf) macro (uses use_gazebo_sim for heavy stand in sim) -->
   <xacro:include filename="../3dmodel/robot_description.urdf.xacro"/>
-  <!-- Import inmoov ros2_control description -->
+  <!-- Import inmoov ros2_control description (use_gazebo_sim switches to gz_ros2_control in Gazebo launch) -->
   <xacro:include filename="../ros2_control/inmoov_ros2_control.xacro" />
+  <!-- gz_ros2_control plugin: only when use_gazebo_sim=true (controller_manager runs inside Gazebo) -->
+  <xacro:if value="$(arg use_gazebo_sim)">
+    <xacro:include filename="../ros2_control/inmoov_gazebo.xacro"/>
+  </xacro:if>
 </robot>
