Commit message: fix(ros2control): add missing shoulder z joint
Signed-off-by: Charles Madjeri <charles@madjeri.com>

File: inmoov/ros2_control/inmoov_ros2_control.xacro (robot description, xacro)
@@ -15,4 +15,9 @@
       <!-- Joint names must match URDF exactly for correct TF tree in RViz/Gazebo -->
       <joint name="left_shoulder_y_link_joint">
+          <command_interface name="position">
+          </command_interface>
+          <state_interface name="position" />
+      </joint>
+      <joint name="left_shoulder_z_link_joint">
           <command_interface name="position">
           </command_interface>
@@ -72,4 +77,9 @@
           <state_interface name="position" />
       </joint>
+      <joint name="right_shoulder_z_link_joint">
+          <command_interface name="position">
+          </command_interface>
+          <state_interface name="position" />
+      </joint>
       <joint name="right_shoulder_x_link_joint">
           <command_interface name="position" />
