Commit message: clean(urdf): clean urdf
Signed-off-by: m-brl <103381146+m-brl@users.noreply.github.com>

File: description/ros2_control/inmoov_ros2_control.xacro (robot description, xacro)
@@ -15,5 +15,4 @@
       </hardware>
       <joint name="left_shoulder_z_link_joint">
-          <dynamics damping="0.7" friction="0.5"/>
           <param name="virtual_pin">0</param>
           <param name="servo_type">270</param>
@@ -24,11 +23,6 @@
           <param name="servo_max_deg">270.0</param>
           <param name="servo_default_deg">135.0</param>
-          <dynamics damping="0.7" friction="0.5"/>
-          <command_interface name="position">
-            <param name="min">-1.57</param>
-            <param name="max">1.57</param>
-          </command_interface>
-          <state_interface name="position"/>
-          <state_interface name="velocity"/>
+          <command_interface name="position" />
+          <state_interface name="position" />
       </joint>
       <joint name="left_shoulder_x_link_joint">
@@ -41,14 +35,8 @@
           <param name="servo_max_deg">270.0</param>
           <param name="servo_default_deg">135.0</param>
-          <dynamics damping="0.7" friction="0.5"/>
-          <command_interface name="position">
-            <param name="min">-1.57</param>
-            <param name="max">1.57</param>
-          </command_interface>
-          <state_interface name="position"/>
-          <state_interface name="velocity"/>
+          <command_interface name="position" />
+          <state_interface name="position" />
       </joint>
       <joint name="left_elbow_x_link_joint">
-          <dynamics damping="0.7" friction="0.5"/>
           <param name="virtual_pin">2</param>
           <param name="servo_type">270</param>
@@ -63,5 +51,4 @@
       </joint>
       <joint name="left_wrist_z_link_joint">
-          <dynamics damping="0.7" friction="0.5"/>
           <param name="virtual_pin">3</param>
           <param name="servo_type">300</param>
@@ -76,5 +63,4 @@
       </joint>
       <joint name="i01.leftHand.thumb_link_joint">
-          <dynamics damping="0.7" friction="0.5"/>
           <param name="virtual_pin">4</param>
           <param name="servo_type">300</param>
@@ -89,5 +75,4 @@
       </joint>
       <joint name="i01.leftHand.index_link_joint">
-          <dynamics damping="0.7" friction="0.5"/>
           <param name="virtual_pin">5</param>
           <param name="servo_type">300</param>
@@ -102,5 +87,4 @@
       </joint>
       <joint name="i01.leftHand.majeure_link_joint">
-          <dynamics damping="0.7" friction="0.5"/>
           <param name="virtual_pin">6</param>
           <param name="servo_type">300</param>
@@ -115,5 +99,4 @@
       </joint>
       <joint name="i01.leftHand.ringFinger_link_joint">
-          <dynamics damping="0.7" friction="0.5"/>
           <param name="virtual_pin">7</param>
           <param name="servo_type">300</param>
@@ -128,5 +111,4 @@
       </joint>
       <joint name="i01.leftHand.pinky_link_joint">
-          <dynamics damping="0.7" friction="0.5"/>
           <param name="virtual_pin">8</param>
           <param name="servo_type">300</param>
@@ -153,5 +135,4 @@
       </hardware>
       <joint name="right_shoulder_z_link_joint">
-          <dynamics damping="0.7" friction="0.5"/>
           <param name="virtual_pin">0</param>
           <param name="servo_type">270</param>
@@ -166,5 +147,4 @@
       </joint>
       <joint name="right_shoulder_x_link_joint">
-          <dynamics damping="0.7" friction="0.5"/>
           <param name="virtual_pin">1</param>
           <param name="servo_type">270</param>
@@ -179,5 +159,4 @@
       </joint>
       <joint name="right_elbow">
-          <dynamics damping="0.7" friction="0.5"/>
           <param name="virtual_pin">2</param>
           <param name="servo_type">270</param>
@@ -192,5 +171,4 @@
       </joint>
       <joint name="right_wrist_z_link_joint">
-          <dynamics damping="0.7" friction="0.5"/>
           <param name="virtual_pin">3</param>
           <param name="servo_type">300</param>
@@ -205,5 +183,4 @@
       </joint>
       <joint name="i01.rightHand.thumb_link_joint">
-          <dynamics damping="0.7" friction="0.5"/>
           <param name="virtual_pin">4</param>
           <param name="servo_type">300</param>
@@ -218,5 +195,4 @@
       </joint>
       <joint name="i01.rightHand.index_link_joint">
-          <dynamics damping="0.7" friction="0.5"/>
           <param name="virtual_pin">5</param>
           <param name="servo_type">300</param>
@@ -231,5 +207,4 @@
       </joint>
       <joint name="i01.rightHand.majeure_link_joint">
-          <dynamics damping="0.7" friction="0.5"/>
           <param name="virtual_pin">6</param>
           <param name="servo_type">300</param>
@@ -244,5 +219,4 @@
       </joint>
       <joint name="i01.rightHand.ringFinger_link_joint">
-          <dynamics damping="0.7" friction="0.5"/>
           <param name="virtual_pin">7</param>
           <param name="servo_type">300</param>
@@ -257,5 +231,4 @@
       </joint>
       <joint name="i01.rightHand.pinky_link_joint">
-          <dynamics damping="0.7" friction="0.5"/>
           <param name="virtual_pin">8</param>
           <param name="servo_type">300</param>
@@ -282,5 +255,4 @@
       </hardware>
       <joint name="left_shoulder_y_link_joint">
-          <dynamics damping="0.7" friction="0.5"/>
           <param name="virtual_pin">0</param>
           <param name="servo_type">270</param>
@@ -295,5 +267,4 @@
       </joint>
       <joint name="right_shoulder_y_link_joint">
-          <dynamics damping="0.7" friction="0.5"/>
           <param name="virtual_pin">1</param>
           <param name="servo_type">270</param>
