Commit message: evol(urdf): archive legacy assets, split Gazebo xacro, and refresh docs

File: description/gazebo/inmoov_gazebo_physics.xacro (robot description, xacro)
@@ -1,10 +1,14 @@
 <?xml version="1.0"?>
-<!-- Gazebo plugin for gz_ros2_control: runs controller_manager inside Gazebo and drives simulated joints.
-     Expects controller_config arg from parent (inmoov.urdf.xacro).
-     Collision strategy: every URDF link reuses its visual mesh as the collision
-     mesh (see scripts/inject_collisions.py). Gazebo macros below only assign
-     surface/contact properties — `gazebo_body_link` disables self_collide on
-     adjacent body meshes (avoids jitter), `gazebo_hand_link` enables it with
-     friction tuned for grasping. -->
+<!-- Gazebo (gz-sim) physics + surface tuning, included only when
+     use_gazebo_sim:=true. This file is pure simulation tuning: world
+     anchoring, friction, contact stiffness, and self-collision flags.
+     The gz_ros2_control plugin itself lives next door in
+     description/ros2_control/inmoov_gz_ros2_control.xacro because it is the
+     ros2_control bridge into Gazebo, not a physics property.
+     Collision strategy: every URDF link reuses its visual mesh as the
+     collision mesh (see scripts/inject_collisions.py). The macros below only
+     assign surface/contact properties — `gazebo_body_link` disables
+     self_collide on adjacent body meshes (avoids jitter), `gazebo_hand_link`
+     enables it with friction tuned for grasping. -->
 <robot xmlns:xacro="http://www.ros.org/wiki/xacro">
   <!-- Fix entire stand to the world so the robot does not fall (gz-sim may still move root; heavy mass in URDF is fallback). -->
@@ -78,10 +82,3 @@
   <xacro:gazebo_hand_side side="left"/>
   <xacro:gazebo_hand_side side="right"/>
-  <gazebo>
-    <plugin filename="gz_ros2_control-system" name="gz_ros2_control::GazeboSimROS2ControlPlugin">
-      <parameters>$(arg controller_config)</parameters>
-      <!-- Empty namespace so controller topics stay at /left_arm_controller, /right_arm_controller (panel expects these). -->
-      <namespace></namespace>
-    </plugin>
-  </gazebo>
 </robot>

File: description/robot_description/urdf/properties.xacro (robot description, xacro)
@@ -8,9 +8,9 @@
 collision sizes (box/cylinder/sphere). Mesh <mesh scale="..."> is left at
 1 1 1 so DAE files are never re-exported.
-Default 0.1163 targets the measured Lucy crown height of 1.75 m. Previous
-0.113 produced ~1.70 m — bumped by the 1.75/1.70 ratio. Replace if the
-measured factor changes.
+Default 0.1196 targets a measured crown height of 1.80 m. Earlier values:
+0.1163 ≈ 1.75 m, 0.113 ≈ 1.70 m — each bump is the height ratio. Replace
+if the measured factor changes.
 -->
 <robot xmlns:xacro="http://www.ros.org/wiki/xacro">
-  <xacro:property name="model_scale" value="0.1163"/>
+  <xacro:property name="model_scale" value="0.1196"/>
 </robot>

File: description/urdf/inmoov.urdf.xacro (robot description, xacro)
@@ -14,7 +14,13 @@
   <!-- Import inmoov ros2_control description (use_gazebo_sim switches to gz_ros2_control in Gazebo launch) -->
   <xacro:include filename="../ros2_control/inmoov_ros2_control.xacro" />
-  <!-- gz_ros2_control plugin: only when use_gazebo_sim=true (controller_manager runs inside Gazebo) -->
+  <!-- Gazebo-only bits, gated on use_gazebo_sim:=true:
+         - gazebo/inmoov_gazebo_physics.xacro    physics + surface tuning
+                                                 (static stand, friction, self_collide, kp/kd)
+         - ros2_control/inmoov_gz_ros2_control.xacro
+                                                 gz_ros2_control plugin so the same
+                                                 controllers drive simulated joints -->
   <xacro:if value="$(arg use_gazebo_sim)">
-    <xacro:include filename="../ros2_control/inmoov_gazebo.xacro"/>
+    <xacro:include filename="../gazebo/inmoov_gazebo_physics.xacro"/>
+    <xacro:include filename="../ros2_control/inmoov_gz_ros2_control.xacro"/>
   </xacro:if>
 </robot>
