Commit message: feat(config): regenerate config
Signed-off-by: m-brl <103381146+m-brl@users.noreply.github.com>

File: description/gazebo/gazebo.xacro (robot description, xacro)
@@ -9,10 +9,10 @@
       <param name="virtual_pin">0</param>
       <param name="servo_type">270</param>
-      <param name="offset_deg">0.0</param>
-      <param name="direction">1</param>
-      <param name="scale">1.0</param>
-      <param name="servo_min_deg">0.0</param>
-      <param name="servo_max_deg">270.0</param>
-      <param name="servo_default_deg">135.0</param>
+      <param name="offset_deg">90</param>
+      <param name="direction">1</param>
+      <param name="scale">1</param>
+      <param name="servo_min_deg">0</param>
+      <param name="servo_max_deg">180</param>
+      <param name="servo_default_deg">90</param>
       <command_interface name="position" />
       <state_interface name="position" />
@@ -21,10 +21,10 @@
       <param name="virtual_pin">1</param>
       <param name="servo_type">270</param>
-      <param name="offset_deg">0.0</param>
-      <param name="direction">1</param>
-      <param name="scale">1.0</param>
-      <param name="servo_min_deg">0.0</param>
-      <param name="servo_max_deg">270.0</param>
-      <param name="servo_default_deg">135.0</param>
+      <param name="offset_deg">0</param>
+      <param name="direction">1</param>
+      <param name="scale">1</param>
+      <param name="servo_min_deg">0</param>
+      <param name="servo_max_deg">180</param>
+      <param name="servo_default_deg">0</param>
       <command_interface name="position" />
       <state_interface name="position" />
@@ -33,10 +33,10 @@
       <param name="virtual_pin">2</param>
       <param name="servo_type">270</param>
-      <param name="offset_deg">0.0</param>
-      <param name="direction">1</param>
-      <param name="scale">1.0</param>
-      <param name="servo_min_deg">0.0</param>
-      <param name="servo_max_deg">270.0</param>
-      <param name="servo_default_deg">90.0</param>
+      <param name="offset_deg">0</param>
+      <param name="direction">1</param>
+      <param name="scale">1</param>
+      <param name="servo_min_deg">0</param>
+      <param name="servo_max_deg">180</param>
+      <param name="servo_default_deg">0</param>
       <command_interface name="position" />
       <state_interface name="position" />
@@ -45,10 +45,10 @@
       <param name="virtual_pin">3</param>
       <param name="servo_type">300</param>
-      <param name="offset_deg">0.0</param>
-      <param name="direction">1</param>
-      <param name="scale">1.0</param>
-      <param name="servo_min_deg">0.0</param>
-      <param name="servo_max_deg">150.0</param>
-      <param name="servo_default_deg">50.0</param>
+      <param name="offset_deg">150</param>
+      <param name="direction">1</param>
+      <param name="scale">1</param>
+      <param name="servo_min_deg">0</param>
+      <param name="servo_max_deg">300</param>
+      <param name="servo_default_deg">150</param>
       <command_interface name="position" />
       <state_interface name="position" />
@@ -57,10 +57,10 @@
       <param name="virtual_pin">4</param>
       <param name="servo_type">300</param>
-      <param name="offset_deg">0.0</param>
-      <param name="direction">1</param>
-      <param name="scale">1.0</param>
-      <param name="servo_min_deg">0.0</param>
-      <param name="servo_max_deg">150.0</param>
-      <param name="servo_default_deg">50.0</param>
+      <param name="offset_deg">0</param>
+      <param name="direction">1</param>
+      <param name="scale">1</param>
+      <param name="servo_min_deg">0</param>
+      <param name="servo_max_deg">180</param>
+      <param name="servo_default_deg">0</param>
       <command_interface name="position" />
       <state_interface name="position" />
@@ -69,10 +69,10 @@
       <param name="virtual_pin">5</param>
       <param name="servo_type">300</param>
-      <param name="offset_deg">0.0</param>
-      <param name="direction">1</param>
-      <param name="scale">1.0</param>
-      <param name="servo_min_deg">0.0</param>
-      <param name="servo_max_deg">150.0</param>
-      <param name="servo_default_deg">50.0</param>
+      <param name="offset_deg">0</param>
+      <param name="direction">1</param>
+      <param name="scale">1</param>
+      <param name="servo_min_deg">0</param>
+      <param name="servo_max_deg">180</param>
+      <param name="servo_default_deg">0</param>
       <command_interface name="position" />
       <state_interface name="position" />
@@ -81,10 +81,10 @@
       <param name="virtual_pin">6</param>
       <param name="servo_type">300</param>
-      <param name="offset_deg">0.0</param>
-      <param name="direction">1</param>
-      <param name="scale">1.0</param>
-      <param name="servo_min_deg">0.0</param>
-      <param name="servo_max_deg">150.0</param>
-      <param name="servo_default_deg">50.0</param>
+      <param name="offset_deg">0</param>
+      <param name="direction">1</param>
+      <param name="scale">1</param>
+      <param name="servo_min_deg">0</param>
+      <param name="servo_max_deg">180</param>
+      <param name="servo_default_deg">0</param>
       <command_interface name="position" />
       <state_interface name="position" />
@@ -93,10 +93,10 @@
       <param name="virtual_pin">7</param>
       <param name="servo_type">300</param>
-      <param name="offset_deg">0.0</param>
-      <param name="direction">1</param>
-      <param name="scale">1.0</param>
-      <param name="servo_min_deg">0.0</param>
-      <param name="servo_max_deg">150.0</param>
-      <param name="servo_default_deg">50.0</param>
+      <param name="offset_deg">0</param>
+      <param name="direction">1</param>
+      <param name="scale">1</param>
+      <param name="servo_min_deg">0</param>
+      <param name="servo_max_deg">180</param>
+      <param name="servo_default_deg">0</param>
       <command_interface name="position" />
       <state_interface name="position" />
@@ -105,10 +105,10 @@
       <param name="virtual_pin">8</param>
       <param name="servo_type">300</param>
-      <param name="offset_deg">0.0</param>
-      <param name="direction">1</param>
-      <param name="scale">1.0</param>
-      <param name="servo_min_deg">0.0</param>
-      <param name="servo_max_deg">150.0</param>
-      <param name="servo_default_deg">50.0</param>
+      <param name="offset_deg">0</param>
+      <param name="direction">1</param>
+      <param name="scale">0.25</param>
+      <param name="servo_min_deg">0</param>
+      <param name="servo_max_deg">180</param>
+      <param name="servo_default_deg">0</param>
       <command_interface name="position" />
       <state_interface name="position" />
@@ -122,10 +122,10 @@
       <param name="virtual_pin">0</param>
       <param name="servo_type">270</param>
-      <param name="offset_deg">0.0</param>
-      <param name="direction">1</param>
-      <param name="scale">1.0</param>
-      <param name="servo_min_deg">155.0</param>
-      <param name="servo_max_deg">165.0</param>
-      <param name="servo_default_deg">160.0</param>
+      <param name="offset_deg">90</param>
+      <param name="direction">-1</param>
+      <param name="scale">1</param>
+      <param name="servo_min_deg">0</param>
+      <param name="servo_max_deg">180</param>
+      <param name="servo_default_deg">90</param>
       <command_interface name="position" />
       <state_interface name="position" />
@@ -134,10 +134,10 @@
       <param name="virtual_pin">1</param>
       <param name="servo_type">270</param>
-      <param name="offset_deg">0.0</param>
-      <param name="direction">1</param>
-      <param name="scale">1.0</param>
-      <param name="servo_min_deg">140.0</param>
-      <param name="servo_max_deg">180.0</param>
-      <param name="servo_default_deg">180.0</param>
+      <param name="offset_deg">0</param>
+      <param name="direction">1</param>
+      <param name="scale">1</param>
+      <param name="servo_min_deg">0</param>
+      <param name="servo_max_deg">180</param>
+      <param name="servo_default_deg">0</param>
       <command_interface name="position" />
       <state_interface name="position" />
@@ -146,10 +146,10 @@
       <param name="virtual_pin">2</param>
       <param name="servo_type">270</param>
-      <param name="offset_deg">0.0</param>
-      <param name="direction">1</param>
-      <param name="scale">1.0</param>
-      <param name="servo_min_deg">100.0</param>
-      <param name="servo_max_deg">110.0</param>
-      <param name="servo_default_deg">100.0</param>
+      <param name="offset_deg">0</param>
+      <param name="direction">1</param>
+      <param name="scale">1</param>
+      <param name="servo_min_deg">0</param>
+      <param name="servo_max_deg">180</param>
+      <param name="servo_default_deg">0</param>
       <command_interface name="position" />
       <state_interface name="position" />
@@ -158,10 +158,10 @@
       <param name="virtual_pin">3</param>
       <param name="servo_type">300</param>
-      <param name="offset_deg">0.0</param>
-      <param name="direction">1</param>
-      <param name="scale">1.0</param>
-      <param name="servo_min_deg">0.0</param>
-      <param name="servo_max_deg">230.0</param>
-      <param name="servo_default_deg">150.0</param>
+      <param name="offset_deg">150</param>
+      <param name="direction">-1</param>
+      <param name="scale">1</param>
+      <param name="servo_min_deg">0</param>
+      <param name="servo_max_deg">300</param>
+      <param name="servo_default_deg">150</param>
       <command_interface name="position" />
       <state_interface name="position" />
@@ -170,10 +170,10 @@
       <param name="virtual_pin">4</param>
       <param name="servo_type">300</param>
-      <param name="offset_deg">0.0</param>
-      <param name="direction">1</param>
-      <param name="scale">1.0</param>
-      <param name="servo_min_deg">36.0</param>
-      <param name="servo_max_deg">150.0</param>
-      <param name="servo_default_deg">36.0</param>
+      <param name="offset_deg">0</param>
+      <param name="direction">1</param>
+      <param name="scale">1</param>
+      <param name="servo_min_deg">0</param>
+      <param name="servo_max_deg">180</param>
+      <param name="servo_default_deg">0</param>
       <command_interface name="position" />
       <state_interface name="position" />
@@ -182,10 +182,10 @@
       <param name="virtual_pin">5</param>
       <param name="servo_type">300</param>
-      <param name="offset_deg">0.0</param>
-      <param name="direction">1</param>
-      <param name="scale">1.0</param>
-      <param name="servo_min_deg">16.0</param>
-      <param name="servo_max_deg">150.0</param>
-      <param name="servo_default_deg">16.0</param>
+      <param name="offset_deg">0</param>
+      <param name="direction">1</param>
+      <param name="scale">1</param>
+      <param name="servo_min_deg">0</param>
+      <param name="servo_max_deg">180</param>
+      <param name="servo_default_deg">0</param>
       <command_interface name="position" />
       <state_interface name="position" />
@@ -194,10 +194,10 @@
       <param name="virtual_pin">6</param>
       <param name="servo_type">300</param>
-      <param name="offset_deg">0.0</param>
-      <param name="direction">1</param>
-      <param name="scale">1.0</param>
-      <param name="servo_min_deg">21.0</param>
-      <param name="servo_max_deg">150.0</param>
-      <param name="servo_default_deg">21.0</param>
+      <param name="offset_deg">0</param>
+      <param name="direction">1</param>
+      <param name="scale">1</param>
+      <param name="servo_min_deg">0</param>
+      <param name="servo_max_deg">180</param>
+      <param name="servo_default_deg">0</param>
       <command_interface name="position" />
       <state_interface name="position" />
@@ -206,10 +206,10 @@
       <param name="virtual_pin">7</param>
       <param name="servo_type">300</param>
-      <param name="offset_deg">0.0</param>
-      <param name="direction">1</param>
-      <param name="scale">1.0</param>
-      <param name="servo_min_deg">33.0</param>
-      <param name="servo_max_deg">150.0</param>
-      <param name="servo_default_deg">33.0</param>
+      <param name="offset_deg">0</param>
+      <param name="direction">1</param>
+      <param name="scale">1</param>
+      <param name="servo_min_deg">0</param>
+      <param name="servo_max_deg">180</param>
+      <param name="servo_default_deg">0</param>
       <command_interface name="position" />
       <state_interface name="position" />
@@ -218,10 +218,10 @@
       <param name="virtual_pin">8</param>
       <param name="servo_type">300</param>
-      <param name="offset_deg">0.0</param>
-      <param name="direction">1</param>
-      <param name="scale">1.0</param>
-      <param name="servo_min_deg">30.0</param>
-      <param name="servo_max_deg">150.0</param>
-      <param name="servo_default_deg">30.0</param>
+      <param name="offset_deg">0</param>
+      <param name="direction">1</param>
+      <param name="scale">1</param>
+      <param name="servo_min_deg">0</param>
+      <param name="servo_max_deg">180</param>
+      <param name="servo_default_deg">0</param>
       <command_interface name="position" />
       <state_interface name="position" />
@@ -235,10 +235,10 @@
       <param name="virtual_pin">0</param>
       <param name="servo_type">270</param>
-      <param name="offset_deg">0.0</param>
-      <param name="direction">1</param>
-      <param name="scale">1.0</param>
-      <param name="servo_min_deg">0.0</param>
-      <param name="servo_max_deg">270.0</param>
-      <param name="servo_default_deg">0.0</param>
+      <param name="offset_deg">0</param>
+      <param name="direction">1</param>
+      <param name="scale">1</param>
+      <param name="servo_min_deg">0</param>
+      <param name="servo_max_deg">180</param>
+      <param name="servo_default_deg">0</param>
       <command_interface name="position" />
       <state_interface name="position" />
@@ -247,10 +247,130 @@
       <param name="virtual_pin">1</param>
       <param name="servo_type">270</param>
-      <param name="offset_deg">0.0</param>
-      <param name="direction">1</param>
-      <param name="scale">1.0</param>
-      <param name="servo_min_deg">0.0</param>
-      <param name="servo_max_deg">270.0</param>
-      <param name="servo_default_deg">0.0</param>
+      <param name="offset_deg">0</param>
+      <param name="direction">1</param>
+      <param name="scale">1</param>
+      <param name="servo_min_deg">0</param>
+      <param name="servo_max_deg">180</param>
+      <param name="servo_default_deg">0</param>
+      <command_interface name="position" />
+      <state_interface name="position" />
+    </joint>
+    <joint name="i01.torso.midStom_link_joint">
+      <param name="virtual_pin">2</param>
+      <param name="servo_type">270</param>
+      <param name="offset_deg">135</param>
+      <param name="direction">1</param>
+      <param name="scale">1</param>
+      <param name="servo_min_deg">0</param>
+      <param name="servo_max_deg">270</param>
+      <param name="servo_default_deg">135</param>
+      <command_interface name="position" />
+      <state_interface name="position" />
+    </joint>
+    <joint name="i01.torso.topStom_link_joint">
+      <param name="virtual_pin">3</param>
+      <param name="servo_type">270</param>
+      <param name="offset_deg">90</param>
+      <param name="direction">1</param>
+      <param name="scale">1</param>
+      <param name="servo_min_deg">0</param>
+      <param name="servo_max_deg">180</param>
+      <param name="servo_default_deg">90</param>
+      <command_interface name="position" />
+      <state_interface name="position" />
+    </joint>
+    <joint name="i01.head.rothead_link_joint">
+      <param name="virtual_pin">4</param>
+      <param name="servo_type">270</param>
+      <param name="offset_deg">90</param>
+      <param name="direction">1</param>
+      <param name="scale">1</param>
+      <param name="servo_min_deg">0</param>
+      <param name="servo_max_deg">180</param>
+      <param name="servo_default_deg">90</param>
+      <command_interface name="position" />
+      <state_interface name="position" />
+    </joint>
+    <joint name="i01.head.rollNeck_link_joint">
+      <param name="virtual_pin">5</param>
+      <param name="servo_type">270</param>
+      <param name="offset_deg">90</param>
+      <param name="direction">1</param>
+      <param name="scale">1</param>
+      <param name="servo_min_deg">0</param>
+      <param name="servo_max_deg">180</param>
+      <param name="servo_default_deg">90</param>
+      <command_interface name="position" />
+      <state_interface name="position" />
+    </joint>
+    <joint name="i01.head.neck.001_link_joint">
+      <param name="virtual_pin">6</param>
+      <param name="servo_type">300</param>
+      <param name="offset_deg">90</param>
+      <param name="direction">1</param>
+      <param name="scale">1</param>
+      <param name="servo_min_deg">0</param>
+      <param name="servo_max_deg">180</param>
+      <param name="servo_default_deg">90</param>
+      <command_interface name="position" />
+      <state_interface name="position" />
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