Commit message: Replace Docker with Pixi (#29)
* fix(gazebo): NixOS EGL env, spawn delay, and conditional GPU setup

Signed-off-by: Charles Madjeri <80175305+charlesmadjeri@users.noreply.github.com>

* Merge pull request #27 from Sentience-Robotics/aes/macos-gazebo

Make the Gazebo GUI work on macOS and keep the robot upright

---------

Signed-off-by: Charles Madjeri <80175305+charlesmadjeri@users.noreply.github.com>
Co-authored-by: Charles Madjeri <80175305+charlesmadjeri@users.noreply.github.com>

File: description/gazebo/gazebo.xacro (robot description, xacro)
@@ -378,5 +378,5 @@
   </ros2_control>
   <gazebo>
-    <plugin filename="libmock_sensor.so" name="mock_sensor::MockSensorSystem">
+    <plugin filename="mock_sensor" name="mock_sensor::MockSensorSystem">
       <update_rate>10</update_rate>
       <topic_name>sensors/left_arm</topic_name>
@@ -389,5 +389,5 @@
   </gazebo>
   <gazebo>
-    <plugin filename="libmock_sensor.so" name="mock_sensor::MockSensorSystem">
+    <plugin filename="mock_sensor" name="mock_sensor::MockSensorSystem">
       <update_rate>10</update_rate>
       <topic_name>sensors/right_arm</topic_name>

File: description/gazebo/inmoov_gazebo_physics.xacro (robot description, xacro)
@@ -12,8 +12,18 @@
      enables it with friction tuned for grasping. -->
 <robot xmlns:xacro="http://www.ros.org/wiki/xacro">
-  <!-- Fix entire stand to the world so the robot does not fall (gz-sim may still move root; heavy mass in URDF is fallback). -->
-  <gazebo reference="base_node">
-    <static>true</static>
-  </gazebo>
+  <!-- Anchor the stand to the world so the robot does not fall over.
+       <gazebo reference="..."><static>true</static></gazebo> does not survive
+       urdf->sdf conversion: sdformat only honours <static> on the model, not on
+       a link, so the stand stayed dynamic and gravity toppled the robot. A fixed
+       joint to a `world` link is the conversion-stable way to pin the base, and
+       leaves every upper-body joint (torso, neck, arms, fingers) free to move.
+       This file is included only under use_gazebo_sim:=true, so the extra link
+       never reaches the real/mock-hardware description or its TF tree. -->
+  <link name="world"/>
+  <joint name="world_to_base_node" type="fixed">
+    <parent link="world"/>
+    <child link="base_node"/>
+    <origin xyz="0 0 0.02" rpy="0 0 0"/>
+  </joint>
   <gazebo reference="stand_link">
     <static>true</static>
