Commit message: evol(thais_urdf): control launch from YAML; RViz uses shared control; robot_description for RViz
- Add config/control.launch.yaml defaults for urdf/controllers paths
- control.launch: spawn controllers from controllers.yaml; fix /robot_description for RViz + ros2_control subscription
- rviz.launch: include control.launch only; drop duplicate ros2_control/spawners
- controllers.yaml: explicit trajectory end velocity; regen-aligned joint lists
- hardware YAML: internal_servo_slots per board; doc + fixture + test updates
- URDF: declare white/black materials for base/stand visuals

Refs: #95

File: description/robot_description/urdf/robot_description.urdf.xacro (robot description, xacro)
@@ -2,4 +2,10 @@
 <robot xmlns:xacro="http://www.ros.org/wiki/xacro" name="inmoov" version="1.0">
   <!-- mesh_dir and use_gazebo_sim set by parent (inmoov.urdf.xacro) -->
+  <material name="white">
+    <color rgba="1.0 1.0 1.0 1.0"/>
+  </material>
+  <material name="black">
+    <color rgba="0.05 0.05 0.05 1.0"/>
+  </material>
   <joint name="Empty.001_link_joint" type="fixed">
     <origin rpy="0.00000 0.00000 0.00000" xyz="-0.00394 0.00025 -0.19163"/>
@@ -408,5 +414,5 @@
   <link name="base_node">
     <visual name="stand">
-      <material name="Gazebo/Grey"/>
+      <material name="white"/>
       <origin rpy="3.14159 -0.00000 3.14159" xyz="-0.00394 -0.00730 9.35280"/>
       <geometry>
@@ -430,4 +436,10 @@
   </link>
   <link name="stand_link">
+    <visual name="stand_anchor">
+      <material name="black"/>
+      <geometry>
+        <box size="0.01 0.01 0.01"/>
+      </geometry>
+    </visual>
     <!-- Minimal geometry so urdf2sdf does not drop this link in Gazebo -->
     <collision name="stand_link_collision">

File: description/ros2_control/inmoov_ros2_control.xacro (robot description, xacro)
@@ -1,6 +1,7 @@
 <?xml version="1.0"?>
+<!-- Generated by lucy_config_generator — do not edit. -->
 <robot xmlns:xacro="http://www.ros.org/wiki/xacro" name="inmoov" version="1.0">
   <xacro:arg name="use_gazebo_sim" default="false" />
-<ros2_control name="LucyHardwareLeftArm" type="system">
+  <ros2_control name="LucyHardwareLeftArm" type="system">
       <hardware>
           <xacro:if value="$(arg use_gazebo_sim)">
@@ -13,47 +14,109 @@
           </xacro:unless>
       </hardware>
-      <!-- Joint names must match URDF exactly for correct TF tree in RViz/Gazebo -->
-      <joint name="left_shoulder_y_link_joint">
-          <command_interface name="position">
-          </command_interface>
-          <state_interface name="position" />
-      </joint>
       <joint name="left_shoulder_z_link_joint">
-          <command_interface name="position">
-          </command_interface>
+          <param name="virtual_pin">0</param>
+          <param name="servo_type">270</param>
+          <param name="offset_deg">0.0</param>
+          <param name="direction">1</param>
+          <param name="scale">1.0</param>
+          <param name="servo_min_deg">0.0</param>
+          <param name="servo_max_deg">270.0</param>
+          <param name="servo_default_deg">135.0</param>
+          <command_interface name="position" />
           <state_interface name="position" />
       </joint>
       <joint name="left_shoulder_x_link_joint">
+          <param name="virtual_pin">1</param>
+          <param name="servo_type">270</param>
+          <param name="offset_deg">0.0</param>
+          <param name="direction">1</param>
+          <param name="scale">1.0</param>
+          <param name="servo_min_deg">0.0</param>
+          <param name="servo_max_deg">270.0</param>
+          <param name="servo_default_deg">135.0</param>
           <command_interface name="position" />
           <state_interface name="position" />
       </joint>
       <joint name="left_elbow_x_link_joint">
+          <param name="virtual_pin">2</param>
+          <param name="servo_type">270</param>
+          <param name="offset_deg">0.0</param>
+          <param name="direction">1</param>
+          <param name="scale">1.0</param>
+          <param name="servo_min_deg">0.0</param>
+          <param name="servo_max_deg">270.0</param>
+          <param name="servo_default_deg">90.0</param>
           <command_interface name="position" />
           <state_interface name="position" />
       </joint>
       <joint name="left_wrist_z_link_joint">
+          <param name="virtual_pin">3</param>
+          <param name="servo_type">300</param>
+          <param name="offset_deg">0.0</param>
+          <param name="direction">1</param>
+          <param name="scale">1.0</param>
+          <param name="servo_min_deg">0.0</param>
+          <param name="servo_max_deg">150.0</param>
+          <param name="servo_default_deg">50.0</param>
           <command_interface name="position" />
           <state_interface name="position" />
       </joint>
       <joint name="i01.leftHand.thumb_link_joint">
+          <param name="virtual_pin">4</param>
+          <param name="servo_type">300</param>
+          <param name="offset_deg">0.0</param>
+          <param name="direction">1</param>
+          <param name="scale">1.0</param>
+          <param name="servo_min_deg">0.0</param>
+          <param name="servo_max_deg">150.0</param>
+          <param name="servo_default_deg">50.0</param>
           <command_interface name="position" />
           <state_interface name="position" />
       </joint>
       <joint name="i01.leftHand.index_link_joint">
-          <command_interface name="position">
-          <param name="min">0</param>
-          <param name="max">1</param>
-          </command_interface>
+          <param name="virtual_pin">5</param>
+          <param name="servo_type">300</param>
+          <param name="offset_deg">0.0</param>
+          <param name="direction">1</param>
+          <param name="scale">1.0</param>
+          <param name="servo_min_deg">0.0</param>
+          <param name="servo_max_deg">150.0</param>
+          <param name="servo_default_deg">50.0</param>
+          <command_interface name="position" />
           <state_interface name="position" />
       </joint>
       <joint name="i01.leftHand.majeure_link_joint">
+          <param name="virtual_pin">6</param>
+          <param name="servo_type">300</param>
+          <param name="offset_deg">0.0</param>
+          <param name="direction">1</param>
+          <param name="scale">1.0</param>
+          <param name="servo_min_deg">0.0</param>
+          <param name="servo_max_deg">150.0</param>
+          <param name="servo_default_deg">50.0</param>
           <command_interface name="position" />
           <state_interface name="position" />
       </joint>
       <joint name="i01.leftHand.ringFinger_link_joint">
+          <param name="virtual_pin">7</param>
+          <param name="servo_type">300</param>
+          <param name="offset_deg">0.0</param>
+          <param name="direction">1</param>
+          <param name="scale">1.0</param>
+          <param name="servo_min_deg">0.0</param>
+          <param name="servo_max_deg">150.0</param>
+          <param name="servo_default_deg">50.0</param>
           <command_interface name="position" />
           <state_interface name="position" />
       </joint>
       <joint name="i01.leftHand.pinky_link_joint">
+          <param name="virtual_pin">8</param>
+          <param name="servo_type">300</param>
+          <param name="offset_deg">0.0</param>
+          <param name="direction">1</param>
+          <param name="scale">1.0</param>
+          <param name="servo_min_deg">0.0</param>
+          <param name="servo_max_deg">150.0</param>
+          <param name="servo_default_deg">50.0</param>
           <command_interface name="position" />
           <state_interface name="position" />
@@ -71,47 +134,145 @@
           </xacro:unless>
       </hardware>
-      <!-- Joint names must match URDF exactly (URDF has right_elbow without _link_joint) -->
+      <joint name="right_shoulder_z_link_joint">
+          <param name="virtual_pin">0</param>
+          <param name="servo_type">270</param>
+          <param name="offset_deg">0.0</param>
+          <param name="direction">1</param>
+          <param name="scale">1.0</param>
+          <param name="servo_min_deg">155.0</param>
+          <param name="servo_max_deg">165.0</param>
+          <param name="servo_default_deg">160.0</param>
+          <command_interface name="position" />
+          <state_interface name="position" />
+      </joint>
+      <joint name="right_shoulder_x_link_joint">
+          <param name="virtual_pin">1</param>
+          <param name="servo_type">270</param>
+          <param name="offset_deg">0.0</param>
+          <param name="direction">1</param>
+          <param name="scale">1.0</param>
+          <param name="servo_min_deg">140.0</param>
+          <param name="servo_max_deg">180.0</param>
+          <param name="servo_default_deg">180.0</param>
+          <command_interface name="position" />
+          <state_interface name="position" />
+      </joint>
+      <joint name="right_elbow">
+          <param name="virtual_pin">2</param>
+          <param name="servo_type">270</param>
+          <param name="offset_deg">0.0</param>
+          <param name="direction">1</param>
+          <param name="scale">1.0</param>
+          <param name="servo_min_deg">100.0</param>
+          <param name="servo_max_deg">110.0</param>
+          <param name="servo_default_deg">100.0</param>
+          <command_interface name="position" />
+          <state_interface name="position" />
+      </joint>
+      <joint name="right_wrist_z_link_joint">
+          <param name="virtual_pin">3</param>
+          <param name="servo_type">300</param>
+          <param name="offset_deg">0.0</param>
+          <param name="direction">1</param>
+          <param name="scale">1.0</param>
+          <param name="servo_min_deg">0.0</param>
+          <param name="servo_max_deg">230.0</param>
+          <param name="servo_default_deg">150.0</param>
+          <command_interface name="position" />
+          <state_interface name="position" />
+      </joint>
+      <joint name="i01.rightHand.thumb_link_joint">
+          <param name="virtual_pin">4</param>
+          <param name="servo_type">300</param>
+          <param name="offset_deg">0.0</param>
+          <param name="direction">1</param>
+          <param name="scale">1.0</param>
+          <param name="servo_min_deg">36.0</param>
+          <param name="servo_max_deg">150.0</param>
+          <param name="servo_default_deg">36.0</param>
+          <command_interface name="position" />
+          <state_interface name="position" />
+      </joint>
+      <joint name="i01.rightHand.index_link_joint">
+          <param name="virtual_pin">5</param>
+          <param name="servo_type">300</param>
+          <param name="offset_deg">0.0</param>
+          <param name="direction">1</param>
+          <param name="scale">1.0</param>
+          <param name="servo_min_deg">16.0</param>
+          <param name="servo_max_deg">150.0</param>
+          <param name="servo_default_deg">16.0</param>
+          <command_interface name="position" />
+          <state_interface name="position" />
+      </joint>
+      <joint name="i01.rightHand.majeure_link_joint">
+          <param name="virtual_pin">6</param>
+          <param name="servo_type">300</param>
+          <param name="offset_deg">0.0</param>
+          <param name="direction">1</param>
+          <param name="scale">1.0</param>
+          <param name="servo_min_deg">21.0</param>
+          <param name="servo_max_deg">150.0</param>
+          <param name="servo_default_deg">21.0</param>
+          <command_interface name="position" />
+          <state_interface name="position" />
+      </joint>
+      <joint name="i01.rightHand.ringFinger_link_joint">
+          <param name="virtual_pin">7</param>
+          <param name="servo_type">300</param>
+          <param name="offset_deg">0.0</param>
+          <param name="direction">1</param>
+          <param name="scale">1.0</param>
+          <param name="servo_min_deg">33.0</param>
+          <param name="servo_max_deg">150.0</param>
+          <param name="servo_default_deg">33.0</param>
+          <command_interface name="position" />
+          <state_interface name="position" />
+      </joint>
+      <joint name="i01.rightHand.pinky_link_joint">
+          <param name="virtual_pin">8</param>
+          <param name="servo_type">300</param>
+          <param name="offset_deg">0.0</param>
+          <param name="direction">1</param>
+          <param name="scale">1.0</param>
+          <param name="servo_min_deg">30.0</param>
+          <param name="servo_max_deg">150.0</param>
+          <param name="servo_default_deg">30.0</param>
+          <command_interface name="position" />
+          <state_interface name="position" />
+      </joint>
+  </ros2_control>
+  <ros2_control name="LucyHardwareTorsoHead" type="system">
+      <hardware>
+          <xacro:if value="$(arg use_gazebo_sim)">
+            <plugin>gz_ros2_control/GazeboSimSystem</plugin>
+          </xacro:if>
+          <xacro:unless value="$(arg use_gazebo_sim)">
+            <plugin>lucy_ros2_control/LucySystemHardware</plugin>
+            <param name="publisher_topic">actuators/torso</param>
+            <param name="node_name">lucy_hardware_interface_torso_head</param>
+          </xacro:unless>
+      </hardware>
+      <joint name="left_shoulder_y_link_joint">
+          <param name="virtual_pin">0</param>
+          <param name="servo_type">270</param>
+          <param name="offset_deg">0.0</param>
+          <param name="direction">1</param>
+          <param name="scale">1.0</param>
+          <param name="servo_min_deg">0.0</param>
+          <param name="servo_max_deg">270.0</param>
+          <param name="servo_default_deg">0.0</param>
+          <command_interface name="position" />
+          <state_interface name="position" />
+      </joint>
       <joint name="right_shoulder_y_link_joint">
-          <command_interface name="position">
-          </command_interface>
-          <state_interface name="position" />
-      </joint>
-      <joint name="right_shoulder_z_link_joint">
-          <command_interface name="position">
-          </command_interface>
-          <state_interface name="position" />
-      </joint>
-      <joint name="right_shoulder_x_link_joint">
-          <command_interface name="position" />
-          <state_interface name="position" />
-      </joint>
-      <joint name="right_elbow">
-          <command_interface name="position" />
-          <state_interface name="position" />
-      </joint>
-      <joint name="right_wrist_z_link_joint">
-          <command_interface name="position" />
-          <state_interface name="position" />
-      </joint>
-      <joint name="i01.rightHand.thumb_link_joint">
-          <command_interface name="position" />
-          <state_interface name="position" />
-      </joint>
-      <joint name="i01.rightHand.index_link_joint">
-          <command_interface name="position">
-          <param name="min">0</param>
-          <param name="max">1</param>
-          </command_interface>
-          <state_interface name="position" />
-      </joint>
-      <joint name="i01.rightHand.majeure_link_joint">
-          <command_interface name="position" />
-          <state_interface name="position" />
-      </joint>
-      <joint name="i01.rightHand.ringFinger_link_joint">
-          <command_interface name="position" />
-          <state_interface name="position" />
-      </joint>
-      <joint name="i01.rightHand.pinky_link_joint">
+          <param name="virtual_pin">1</param>
+          <param name="servo_type">270</param>
+          <param name="offset_deg">0.0</param>
+          <param name="direction">1</param>
+          <param name="scale">1.0</param>
+          <param name="servo_min_deg">0.0</param>
+          <param name="servo_max_deg">270.0</param>
+          <param name="servo_default_deg">0.0</param>
           <command_interface name="position" />
           <state_interface name="position" />
