Commit message: feat(simulator): add gazebo simulation
fix(physical urdf): add effort to urdf
feat(launch file): delete useless gazebo node
refacto(rviz): refacto rviz launch file
clean(launch file)

To lauch gazebo, use lucy bringup.
Gazebo and rviz no longer launch rsp, jsp...

Signed-off-by: m-brl <103381146+m-brl@users.noreply.github.com>

File: description/robot_description/urdf/robot_description.urdf.xacro (robot description, xacro)
@@ -14,5 +14,6 @@
   </joint>
   <joint name="Empty.002_link_joint" type="continuous">
-    <limit lower="0" upper="0" effort="0.00000" velocity="0.78540"/>
+    <limit lower="0" upper="0" effort="100.00000" velocity="0.78540"/>
+    <dynamics damping="0.7" friction="0.5"/>
     <origin rpy="0.00000 0.00000 0.00000" xyz="0.00000 0.00000 8.97279"/>
     <parent link="stand_link"/>
@@ -21,5 +22,6 @@
   </joint>
   <joint name="i01.head.eyeRight_link_joint" type="revolute">
-    <limit lower="-0.78530" upper="0.78530" effort="0.00000" velocity="0.78540"/>
+    <limit lower="-0.78530" upper="0.78530" effort="100.00000" velocity="0.78540"/>
+    <dynamics damping="0.7" friction="0.5"/>
     <origin rpy="0.00000 -0.00000 0.00000" xyz="-0.00000 -0.00590 0.00000"/>
     <parent link="i01.head.eyeRight.001_link"/>
@@ -28,5 +30,6 @@
   </joint>
   <joint name="i01.head.jaw_link_joint" type="revolute">
-    <limit lower="0.00000" upper="0.17453" effort="0.00000" velocity="0.78540"/>
+    <limit lower="0.00000" upper="0.17453" effort="100.00000" velocity="0.78540"/>
+    <dynamics damping="0.7" friction="0.5"/>
     <origin rpy="-0.00000 -0.00000 -1.57080" xyz="-0.36176 0.01121 0.32442"/>
     <parent link="i01.head.rothead_link"/>
@@ -35,5 +38,6 @@
   </joint>
   <joint name="left_shoulder_y_link_joint" type="revolute">
-    <limit lower="0.00000" upper="1.57080" effort="0.00000" velocity="0.78540"/>
+    <limit lower="0.00000" upper="1.57080" effort="100.00000" velocity="0.78540"/>
+    <dynamics damping="0.7" friction="0.5"/>
     <origin rpy="0.00021 -0.00000 -0.00000" xyz="1.35472 -0.00337 2.80749"/>
     <parent link="torso_y_link"/>
@@ -42,5 +46,6 @@
   </joint>
   <joint name="left_shoulder_x_link_joint" type="revolute">
-    <limit lower="-1.57080" upper="2.35619" effort="0.00000" velocity="0.78540"/>
+    <limit lower="-1.57080" upper="2.35619" effort="100.00000" velocity="0.78540"/>
+    <dynamics damping="0.7" friction="0.5"/>
     <origin rpy="-0.00000 -0.00000 -0.00000" xyz="0.11351 0.00189 -0.37504"/>
     <parent link="left_shoulder_y_link"/>
@@ -49,5 +54,6 @@
   </joint>
   <joint name="left_shoulder_z_link_joint" type="revolute">
-    <limit lower="-1.57080" upper="1.57080" effort="0.00000" velocity="0.78540"/>
+    <limit lower="-1.57080" upper="1.57080" effort="100.00000" velocity="0.78540"/>
+    <dynamics damping="0.7" friction="0.5"/>
     <origin rpy="0.00000 0.00000 0.00000" xyz="0.62406 -0.00937 -0.59421"/>
     <parent link="left_shoulder_x_link"/>
@@ -56,5 +62,6 @@
   </joint>
   <joint name="left_elbow_x_link_joint" type="revolute">
-    <limit lower="0.00000" upper="1.57080" effort="0.00000" velocity="0.78540"/>
+    <limit lower="0.00000" upper="1.57080" effort="100.00000" velocity="0.78540"/>
+    <dynamics damping="0.7" friction="0.5"/>
     <origin rpy="0.06567 -0.00000 -0.00000" xyz="-0.01281 0.29228 -2.11577"/>
     <parent link="left_shoulder_z_link"/>
@@ -63,5 +70,6 @@
   </joint>
   <joint name="left_wrist_z_link_joint" type="revolute">
-    <limit lower="-1.57080" upper="1.57080" effort="0.00000" velocity="0.78540"/>
+    <limit lower="-1.57080" upper="1.57080" effort="100.00000" velocity="0.78540"/>
+    <dynamics damping="0.7" friction="0.5"/>
     <origin rpy="-0.41605 -0.00000 0.00000" xyz="-0.08767 -0.98766 -2.53936"/>
     <parent link="left_elbow_x_link"/>
@@ -70,5 +78,6 @@
   </joint>
   <joint name="i01.leftHand.wrist.001_link_joint" type="revolute">
-    <limit lower="0.00000" upper="1.57080" effort="0.00000" velocity="0.78540"/>
+    <limit lower="0.00000" upper="1.57080" effort="100.00000" velocity="0.78540"/>
+    <dynamics damping="0.7" friction="0.5"/>
     <origin rpy="-0.00000 0.00000 -0.61611" xyz="-0.00000 -0.00000 -0.16925"/>
     <parent link="left_wrist_z_link"/>
@@ -77,5 +86,6 @@
   </joint>
   <joint name="i01.leftHand.index_link_joint" type="revolute">
-    <limit lower="0.00000" upper="1.57080" effort="0.00000" velocity="0.78540"/>
+    <limit lower="0.00000" upper="1.57080" effort="100.00000" velocity="0.78540"/>
+    <dynamics damping="0.7" friction="0.5"/>
     <origin rpy="-1.56854 -0.09096 -0.00330" xyz="0.32645 -0.01145 -0.94982"/>
     <parent link="i01.leftHand.wrist.001_link"/>
@@ -84,5 +94,6 @@
   </joint>
   <joint name="i01.leftHand.index2_link_joint" type="revolute">
-    <limit lower="0.00000" upper="1.57080" effort="0.00000" velocity="0.78540"/>
+    <limit lower="0.00000" upper="1.57080" effort="100.00000" velocity="0.78540"/>
+    <dynamics damping="0.7" friction="0.5"/>
     <origin rpy="-0.00000 0.00000 -0.00000" xyz="0.00258 0.34105 0.00685"/>
     <parent link="i01.leftHand.index_link"/>
@@ -91,5 +102,6 @@
   </joint>
   <joint name="i01.torso.midStom_link_joint" type="revolute">
-    <limit lower="-2.35619" upper="2.35619" effort="0.00000" velocity="0.78540"/>
+    <limit lower="-2.35619" upper="2.35619" effort="100.00000" velocity="0.78540"/>
+    <dynamics damping="0.7" friction="0.5"/>
     <origin rpy="0.00000 0.06589 1.57080" xyz="-0.00213 0.05565 1.13807"/>
     <parent link="torso_bottom_link"/>
@@ -98,5 +110,6 @@
   </joint>
   <joint name="i01.leftHand.index3_link_joint" type="revolute">
-    <limit lower="0.00000" upper="1.57080" effort="0.00000" velocity="0.78540"/>
+    <limit lower="0.00000" upper="1.57080" effort="100.00000" velocity="0.78540"/>
+    <dynamics damping="0.7" friction="0.5"/>
     <origin rpy="0.00000 -0.00000 -0.00000" xyz="0.00103 0.22697 0.00433"/>
     <parent link="i01.leftHand.index2_link"/>
@@ -105,5 +118,6 @@
   </joint>
   <joint name="i01.leftHand.majeure_link_joint" type="revolute">
-    <limit lower="0.00000" upper="1.57080" effort="0.00000" velocity="0.78540"/>
+    <limit lower="0.00000" upper="1.57080" effort="100.00000" velocity="0.78540"/>
+    <dynamics damping="0.7" friction="0.5"/>
     <origin rpy="-1.56854 0.00160 -0.00309" xyz="0.07161 -0.01170 -0.98881"/>
     <parent link="i01.leftHand.wrist.001_link"/>
@@ -112,5 +126,6 @@
   </joint>
   <joint name="i01.leftHand.majeure2_link_joint" type="revolute">
-    <limit lower="0.00000" upper="1.57080" effort="0.00000" velocity="0.78540"/>
+    <limit lower="0.00000" upper="1.57080" effort="100.00000" velocity="0.78540"/>
+    <dynamics damping="0.7" friction="0.5"/>
     <origin rpy="-0.00000 -0.00000 0.00000" xyz="0.00272 0.35935 0.00722"/>
     <parent link="i01.leftHand.majeure_link"/>
@@ -119,5 +134,6 @@
   </joint>
   <joint name="i01.leftHand.majeure3_link_joint" type="revolute">
-    <limit lower="0.00000" upper="1.57080" effort="0.00000" velocity="0.78540"/>
+    <limit lower="0.00000" upper="1.57080" effort="100.00000" velocity="0.78540"/>
+    <dynamics damping="0.7" friction="0.5"/>
     <origin rpy="0.00000 -0.00000 -0.00000" xyz="0.00109 0.23915 0.00456"/>
     <parent link="i01.leftHand.majeure2_link"/>
@@ -126,5 +142,6 @@
   </joint>
   <joint name="i01.leftHand.pinky0_link_joint" type="revolute">
-    <limit lower="0.00000" upper="1.57080" effort="0.00000" velocity="0.78540"/>
+    <limit lower="0.00000" upper="1.57080" effort="100.00000" velocity="0.78540"/>
+    <dynamics damping="0.7" friction="0.5"/>
     <origin rpy="-1.56789 -0.68643 -0.00494" xyz="-0.24002 0.00108 -0.35218"/>
     <parent link="i01.leftHand.wrist.001_link"/>
@@ -133,5 +150,6 @@
   </joint>
   <joint name="i01.leftHand.pinky_link_joint" type="revolute">
-    <limit lower="0.00000" upper="1.57080" effort="0.00000" velocity="0.78540"/>
+    <limit lower="0.00000" upper="1.57080" effort="100.00000" velocity="0.78540"/>
+    <dynamics damping="0.7" friction="0.5"/>
     <origin rpy="-0.00000 0.00000 0.94526" xyz="-0.43178 0.20489 0.00726"/>
     <parent link="i01.leftHand.pinky0_link"/>
@@ -140,5 +158,6 @@
   </joint>
   <joint name="i01.leftHand.pinky2_link_joint" type="revolute">
-    <limit lower="0.00000" upper="1.57080" effort="0.00000" velocity="0.78540"/>
+    <limit lower="0.00000" upper="1.57080" effort="100.00000" velocity="0.78540"/>
+    <dynamics damping="0.7" friction="0.5"/>
     <origin rpy="-0.00000 0.00000 -0.00000" xyz="0.00225 0.29796 0.00599"/>
     <parent link="i01.leftHand.pinky_link"/>
@@ -147,5 +166,6 @@
   </joint>
   <joint name="i01.leftHand.pinky3_link_joint" type="revolute">
-    <limit lower="0.00000" upper="1.57080" effort="0.00000" velocity="0.78540"/>
+    <limit lower="0.00000" upper="1.57080" effort="100.00000" velocity="0.78540"/>
+    <dynamics damping="0.7" friction="0.5"/>
     <origin rpy="-0.00000 -0.00000 -0.00000" xyz="0.00090 0.19830 0.00378"/>
     <parent link="i01.leftHand.pinky2_link"/>
@@ -154,5 +174,6 @@
   </joint>
   <joint name="i01.leftHand.ringfinger0_link_joint" type="revolute">
-    <limit lower="0.00000" upper="1.57080" effort="0.00000" velocity="0.78540"/>
+    <limit lower="0.00000" upper="1.57080" effort="100.00000" velocity="0.78540"/>
+    <dynamics damping="0.7" friction="0.5"/>
     <origin rpy="-1.56789 -0.68643 -0.00494" xyz="-0.05673 0.00101 -0.57588"/>
     <parent link="i01.leftHand.wrist.001_link"/>
@@ -161,5 +182,6 @@
   </joint>
   <joint name="i01.leftHand.ringFinger_link_joint" type="revolute">
-    <limit lower="0.00000" upper="1.57080" effort="0.00000" velocity="0.78540"/>
+    <limit lower="0.00000" upper="1.57080" effort="100.00000" velocity="0.78540"/>
+    <dynamics damping="0.7" friction="0.5"/>
     <origin rpy="-0.00000 0.00000 0.77485" xyz="-0.33329 0.15280 -0.00664"/>
     <parent link="i01.leftHand.ringfinger0_link"/>
@@ -168,5 +190,6 @@
   </joint>
   <joint name="i01.torso.topStom_link_joint" type="revolute">
-    <limit lower="-0.34907" upper="0.34907" effort="0.00000" velocity="0.78540"/>
+    <limit lower="-0.34907" upper="0.34907" effort="100.00000" velocity="0.78540"/>
+    <dynamics damping="0.7" friction="0.5"/>
     <origin rpy="0.00000 0.00000 -1.57080" xyz="-0.06317 0.00033 1.01916"/>
     <parent link="torso_z_link"/>
@@ -175,5 +198,6 @@
   </joint>
   <joint name="i01.leftHand.ringfinger2_link_joint" type="revolute">
-    <limit lower="0.00000" upper="1.57080" effort="0.00000" velocity="0.78540"/>
+    <limit lower="0.00000" upper="1.57080" effort="100.00000" velocity="0.78540"/>
+    <dynamics damping="0.7" friction="0.5"/>
     <origin rpy="-0.00000 -0.00000 0.00000" xyz="0.00258 0.34105 0.00685"/>
     <parent link="i01.leftHand.ringFinger_link"/>
@@ -182,5 +206,6 @@
   </joint>
   <joint name="i01.leftHand.ringfinger3_link_joint" type="revolute">
-    <limit lower="0.00000" upper="1.57080" effort="0.00000" velocity="0.78540"/>
+    <limit lower="0.00000" upper="1.57080" effort="100.00000" velocity="0.78540"/>
+    <dynamics damping="0.7" friction="0.5"/>
     <origin rpy="-0.00000 0.00000 -0.00000" xyz="0.00103 0.22697 0.00433"/>
     <parent link="i01.leftHand.ringfinger2_link"/>
@@ -189,5 +214,6 @@
   </joint>
   <joint name="i01.leftHand.thumb1_link_joint" type="revolute">
-    <limit lower="0.00000" upper="1.57080" effort="0.00000" velocity="0.78540"/>
+    <limit lower="0.00000" upper="1.57080" effort="100.00000" velocity="0.78540"/>
+    <dynamics damping="0.7" friction="0.5"/>
     <origin rpy="1.51635 -0.09893 -0.00332" xyz="0.28234 -0.00002 -0.37340"/>
     <parent link="i01.leftHand.wrist.001_link"/>
@@ -196,5 +222,6 @@
   </joint>
   <joint name="i01.leftHand.thumb_link_joint" type="revolute">
-    <limit lower="0.00000" upper="1.57080" effort="0.00000" velocity="0.78540"/>
+    <limit lower="0.00000" upper="1.57080" effort="100.00000" velocity="0.78540"/>
+    <dynamics damping="0.7" friction="0.5"/>
     <origin rpy="-0.03182 -0.32566 0.83064" xyz="0.25977 -0.13332 -0.00800"/>
     <parent link="i01.leftHand.thumb1_link"/>
@@ -203,5 +230,6 @@
   </joint>
   <joint name="i01.leftHand.thumb3_link_joint" type="revolute">
-    <limit lower="0.00000" upper="1.57080" effort="0.00000" velocity="0.78540"/>
+    <limit lower="0.00000" upper="1.57080" effort="100.00000" velocity="0.78540"/>
+    <dynamics damping="0.7" friction="0.5"/>
     <origin rpy="0.00001 -0.00000 0.00000" xyz="0.01229 -0.33047 -0.00704"/>
     <parent link="i01.leftHand.thumb_link"/>
@@ -210,5 +238,6 @@
   </joint>
   <joint name="right_shoulder_y_link_joint" type="revolute">
-    <limit lower="0.00000" upper="1.57080" effort="0.00000" velocity="0.78540"/>
+    <limit lower="0.00000" upper="1.57080" effort="100.00000" velocity="0.78540"/>
+    <dynamics damping="0.7" friction="0.5"/>
     <origin rpy="0.00021 -0.00000 -0.00000" xyz="-1.34979 -0.00337 2.80749"/>
     <parent link="torso_y_link"/>
@@ -217,5 +246,6 @@
   </joint>
   <joint name="right_shoulder_x_link_joint" type="revolute">
-    <limit lower="-1.57080" upper="2.35619" effort="0.00000" velocity="0.78540"/>
+    <limit lower="-1.57080" upper="2.35619" effort="100.00000" velocity="0.78540"/>
+    <dynamics damping="0.7" friction="0.5"/>
     <origin rpy="-0.00000 -0.00000 -0.00000" xyz="-0.11351 0.00189 -0.37504"/>
     <parent link="right_shoulder_y_link"/>
@@ -224,5 +254,6 @@
   </joint>
   <joint name="right_shoulder_z_link_joint" type="revolute">
-    <limit lower="-1.57080" upper="1.57080" effort="0.00000" velocity="0.78540"/>
+    <limit lower="-1.57080" upper="1.57080" effort="100.00000" velocity="0.78540"/>
+    <dynamics damping="0.7" friction="0.5"/>
     <origin rpy="0.00000 0.00000 0.00000" xyz="-0.62406 -0.00937 -0.59421"/>
     <parent link="right_shoulder_x_link"/>
@@ -231,5 +262,6 @@
   </joint>
   <joint name="right_elbow" type="revolute">
-    <limit lower="0.00000" upper="1.57080" effort="0.00000" velocity="0.78540"/>
+    <limit lower="0.00000" upper="1.57080" effort="100.00000" velocity="0.78540"/>
+    <dynamics damping="0.7" friction="0.5"/>
     <origin rpy="0.06567 0.00000 0.00000" xyz="0.00858 0.29228 -2.11577"/>
     <parent link="right_shoulder_z_link"/>
@@ -238,5 +270,6 @@
   </joint>
   <joint name="right_wrist_z_link_joint" type="revolute">
-    <limit lower="-1.57080" upper="1.57080" effort="0.00000" velocity="0.78540"/>
+    <limit lower="-1.57080" upper="1.57080" effort="100.00000" velocity="0.78540"/>
+    <dynamics damping="0.7" friction="0.5"/>
     <origin rpy="-0.41605 0.00000 0.00000" xyz="0.08767 -0.98766 -2.53936"/>
     <parent link="right_elbow_x_link"/>
@@ -245,5 +278,6 @@
   </joint>
   <joint name="i01.head.neck.001_link_joint" type="revolute">
-    <limit lower="-0.34907" upper="0.34907" effort="0.00000" velocity="0.78540"/>
+    <limit lower="-0.34907" upper="0.34907" effort="100.00000" velocity="0.78540"/>
+    <dynamics damping="0.7" friction="0.5"/>
     <origin rpy="0.06589 -0.00000 -0.00000" xyz="0.00390 0.29817 4.29073"/>
     <parent link="torso_y_link"/>
@@ -252,5 +286,6 @@
   </joint>
   <joint name="i01.rightHand.wrist.001_link_joint" type="revolute">
-    <limit lower="0.00000" upper="1.57080" effort="0.00000" velocity="0.78540"/>
+    <limit lower="0.00000" upper="1.57080" effort="100.00000" velocity="0.78540"/>
+    <dynamics damping="0.7" friction="0.5"/>
     <origin rpy="0.00000 0.00000 0.63517" xyz="-0.00000 -0.00000 -0.16508"/>
     <parent link="right_wrist_z_link"/>
@@ -259,5 +294,6 @@
   </joint>
   <joint name="i01.rightHand.index_link_joint" type="revolute">
-    <limit lower="0.00000" upper="1.57080" effort="0.00000" velocity="0.78540"/>
+    <limit lower="0.00000" upper="1.57080" effort="100.00000" velocity="0.78540"/>
+    <dynamics damping="0.7" friction="0.5"/>
     <origin rpy="1.57305 0.09096 -0.01576" xyz="-0.32320 -0.00773 -0.95398"/>
     <parent link="i01.rightHand.wrist.001_link"/>
@@ -266,5 +302,6 @@
   </joint>
   <joint name="i01.rightHand.index2_link_joint" type="revolute">
-    <limit lower="0.00000" upper="1.57080" effort="0.00000" velocity="0.78540"/>
+    <limit lower="0.00000" upper="1.57080" effort="100.00000" velocity="0.78540"/>
+    <dynamics damping="0.7" friction="0.5"/>
     <origin rpy="0.00000 -0.00000 0.00000" xyz="-0.00258 -0.34105 -0.00685"/>
     <parent link="i01.rightHand.index_link"/>
@@ -273,5 +310,6 @@
   </joint>
   <joint name="i01.rightHand.index3_link_joint" type="revolute">
-    <limit lower="0.00000" upper="1.57080" effort="0.00000" velocity="0.78540"/>
+    <limit lower="0.00000" upper="1.57080" effort="100.00000" velocity="0.78540"/>
+    <dynamics damping="0.7" friction="0.5"/>
     <origin rpy="0.00000 0.00000 -0.00000" xyz="-0.00103 -0.22697 -0.00432"/>
     <parent link="i01.rightHand.index2_link"/>
@@ -280,5 +318,6 @@
   </joint>
   <joint name="i01.rightHand.majeure_link_joint" type="revolute">
-    <limit lower="0.00000" upper="1.57080" effort="0.00000" velocity="0.78540"/>
+    <limit lower="0.00000" upper="1.57080" effort="100.00000" velocity="0.78540"/>
+    <dynamics damping="0.7" friction="0.5"/>
     <origin rpy="1.57305 -0.00160 -0.01597" xyz="-0.06841 -0.01284 -0.99297"/>
     <parent link="i01.rightHand.wrist.001_link"/>
@@ -287,5 +326,6 @@
   </joint>
   <joint name="i01.rightHand.majeure2_link_joint" type="revolute">
-    <limit lower="0.00000" upper="1.57080" effort="0.00000" velocity="0.78540"/>
+    <limit lower="0.00000" upper="1.57080" effort="100.00000" velocity="0.78540"/>
+    <dynamics damping="0.7" friction="0.5"/>
     <origin rpy="-0.00000 -0.00000 -0.00000" xyz="-0.00272 -0.35935 -0.00722"/>
     <parent link="i01.rightHand.majeure_link"/>
@@ -294,5 +334,6 @@
   </joint>
   <joint name="i01.rightHand.majeure3_link_joint" type="revolute">
-    <limit lower="0.00000" upper="1.57080" effort="0.00000" velocity="0.78540"/>
+    <limit lower="0.00000" upper="1.57080" effort="100.00000" velocity="0.78540"/>
+    <dynamics damping="0.7" friction="0.5"/>
     <origin rpy="0.00000 -0.00000 0.00000" xyz="-0.00109 -0.23915 -0.00456"/>
     <parent link="i01.rightHand.majeure2_link"/>
@@ -301,5 +342,6 @@
   </joint>
   <joint name="i01.rightHand.pinky0_link_joint" type="revolute">
-    <limit lower="0.00000" upper="1.57080" effort="0.00000" velocity="0.78540"/>
+    <limit lower="0.00000" upper="1.57080" effort="100.00000" velocity="0.78540"/>
+    <dynamics damping="0.7" friction="0.5"/>
     <origin rpy="1.57370 0.68643 -0.01412" xyz="0.24340 -0.00601 -0.35634"/>
     <parent link="i01.rightHand.wrist.001_link"/>
@@ -308,5 +350,6 @@
   </joint>
   <joint name="i01.rightHand.pinky_link_joint" type="revolute">
-    <limit lower="0.00000" upper="1.57080" effort="0.00000" velocity="0.78540"/>
+    <limit lower="0.00000" upper="1.57080" effort="100.00000" velocity="0.78540"/>
+    <dynamics damping="0.7" friction="0.5"/>
     <origin rpy="-0.00000 -0.00000 0.94526" xyz="0.43178 -0.20489 -0.00726"/>
     <parent link="i01.rightHand.pinky0_link"/>
@@ -315,5 +358,6 @@
   </joint>
   <joint name="i01.rightHand.pinky2_link_joint" type="revolute">
-    <limit lower="0.00000" upper="1.57080" effort="0.00000" velocity="0.78540"/>
+    <limit lower="0.00000" upper="1.57080" effort="100.00000" velocity="0.78540"/>
+    <dynamics damping="0.7" friction="0.5"/>
     <origin rpy="0.00000 0.00000 -0.00000" xyz="-0.00225 -0.29796 -0.00598"/>
     <parent link="i01.rightHand.pinky_link"/>
@@ -322,5 +366,6 @@
   </joint>
   <joint name="i01.head.rollNeck_link_joint" type="revolute">
-    <limit lower="-0.34907" upper="0.34907" effort="0.00000" velocity="0.78540"/>
+    <limit lower="-0.34907" upper="0.34907" effort="100.00000" velocity="0.78540"/>
+    <dynamics damping="0.7" friction="0.5"/>
     <origin rpy="-0.00000 0.00000 -0.00000" xyz="0.00000 -0.00000 0.00435"/>
     <parent link="i01.head.neck.001_link"/>
@@ -329,5 +374,6 @@
   </joint>
   <joint name="i01.rightHand.pinky3_link_joint" type="revolute">
-    <limit lower="0.00000" upper="1.57080" effort="0.00000" velocity="0.78540"/>
+    <limit lower="0.00000" upper="1.57080" effort="100.00000" velocity="0.78540"/>
+    <dynamics damping="0.7" friction="0.5"/>
     <origin rpy="0.00000 0.00000 0.00000" xyz="-0.00090 -0.19830 -0.00378"/>
     <parent link="i01.rightHand.pinky2_link"/>
@@ -336,5 +382,6 @@
   </joint>
   <joint name="i01.rightHand.ringfinger0_link_joint" type="revolute">
-    <limit lower="0.00000" upper="1.57080" effort="0.00000" velocity="0.78540"/>
+    <limit lower="0.00000" upper="1.57080" effort="100.00000" velocity="0.78540"/>
+    <dynamics damping="0.7" friction="0.5"/>
     <origin rpy="1.57370 0.68643 -0.01412" xyz="0.06015 -0.00258 -0.58004"/>
     <parent link="i01.rightHand.wrist.001_link"/>
@@ -343,5 +390,6 @@
   </joint>
   <joint name="i01.rightHand.ringFinger_link_joint" type="revolute">
-    <limit lower="0.00000" upper="1.57080" effort="0.00000" velocity="0.78540"/>
+    <limit lower="0.00000" upper="1.57080" effort="100.00000" velocity="0.78540"/>
+    <dynamics damping="0.7" friction="0.5"/>
     <origin rpy="-0.00000 -0.00000 0.77485" xyz="0.33328 -0.15280 0.00664"/>
     <parent link="i01.rightHand.ringfinger0_link"/>
@@ -350,5 +398,6 @@
   </joint>
   <joint name="i01.rightHand.ringfinger2_link_joint" type="revolute">
-    <limit lower="0.00000" upper="1.57080" effort="0.00000" velocity="0.78540"/>
+    <limit lower="0.00000" upper="1.57080" effort="100.00000" velocity="0.78540"/>
+    <dynamics damping="0.7" friction="0.5"/>
     <origin rpy="-0.00000 -0.00000 0.00000" xyz="-0.00258 -0.34105 -0.00685"/>
     <parent link="i01.rightHand.ringFinger_link"/>
@@ -357,5 +406,6 @@
   </joint>
   <joint name="i01.rightHand.ringfinger3_link_joint" type="revolute">
-    <limit lower="0.00000" upper="1.57080" effort="0.00000" velocity="0.78540"/>
+    <limit lower="0.00000" upper="1.57080" effort="100.00000" velocity="0.78540"/>
+    <dynamics damping="0.7" friction="0.5"/>
     <origin rpy="-0.00000 0.00000 -0.00000" xyz="-0.00103 -0.22697 -0.00432"/>
     <parent link="i01.rightHand.ringfinger2_link"/>
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