Commit message: feat(simulator): add gazebo simulation
fix(physical urdf): add effort to urdf
feat(launch file): delete useless gazebo node
refacto(rviz): refacto rviz launch file
clean(launch file)

To lauch gazebo, use lucy bringup.
Gazebo and rviz no longer launch rsp, jsp...

Signed-off-by: m-brl <103381146+m-brl@users.noreply.github.com>

File: description/ros2_control/inmoov_ros2_control.xacro (robot description, xacro)
@@ -15,4 +15,5 @@
       </hardware>
       <joint name="left_shoulder_z_link_joint">
+          <dynamics damping="0.7" friction="0.5"/>
           <param name="virtual_pin">0</param>
           <param name="servo_type">270</param>
@@ -23,6 +24,11 @@
           <param name="servo_max_deg">270.0</param>
           <param name="servo_default_deg">135.0</param>
-          <command_interface name="position" />
-          <state_interface name="position" />
+          <dynamics damping="0.7" friction="0.5"/>
+          <command_interface name="position">
+            <param name="min">-1.57</param>
+            <param name="max">1.57</param>
+          </command_interface>
+          <state_interface name="position"/>
+          <state_interface name="velocity"/>
       </joint>
       <joint name="left_shoulder_x_link_joint">
@@ -35,8 +41,14 @@
           <param name="servo_max_deg">270.0</param>
           <param name="servo_default_deg">135.0</param>
-          <command_interface name="position" />
-          <state_interface name="position" />
+          <dynamics damping="0.7" friction="0.5"/>
+          <command_interface name="position">
+            <param name="min">-1.57</param>
+            <param name="max">1.57</param>
+          </command_interface>
+          <state_interface name="position"/>
+          <state_interface name="velocity"/>
       </joint>
       <joint name="left_elbow_x_link_joint">
+          <dynamics damping="0.7" friction="0.5"/>
           <param name="virtual_pin">2</param>
           <param name="servo_type">270</param>
@@ -51,4 +63,5 @@
       </joint>
       <joint name="left_wrist_z_link_joint">
+          <dynamics damping="0.7" friction="0.5"/>
           <param name="virtual_pin">3</param>
           <param name="servo_type">300</param>
@@ -63,4 +76,5 @@
       </joint>
       <joint name="i01.leftHand.thumb_link_joint">
+          <dynamics damping="0.7" friction="0.5"/>
           <param name="virtual_pin">4</param>
           <param name="servo_type">300</param>
@@ -75,4 +89,5 @@
       </joint>
       <joint name="i01.leftHand.index_link_joint">
+          <dynamics damping="0.7" friction="0.5"/>
           <param name="virtual_pin">5</param>
           <param name="servo_type">300</param>
@@ -87,4 +102,5 @@
       </joint>
       <joint name="i01.leftHand.majeure_link_joint">
+          <dynamics damping="0.7" friction="0.5"/>
           <param name="virtual_pin">6</param>
           <param name="servo_type">300</param>
@@ -99,4 +115,5 @@
       </joint>
       <joint name="i01.leftHand.ringFinger_link_joint">
+          <dynamics damping="0.7" friction="0.5"/>
           <param name="virtual_pin">7</param>
           <param name="servo_type">300</param>
@@ -111,4 +128,5 @@
       </joint>
       <joint name="i01.leftHand.pinky_link_joint">
+          <dynamics damping="0.7" friction="0.5"/>
           <param name="virtual_pin">8</param>
           <param name="servo_type">300</param>
@@ -135,4 +153,5 @@
       </hardware>
       <joint name="right_shoulder_z_link_joint">
+          <dynamics damping="0.7" friction="0.5"/>
           <param name="virtual_pin">0</param>
           <param name="servo_type">270</param>
@@ -147,4 +166,5 @@
       </joint>
       <joint name="right_shoulder_x_link_joint">
+          <dynamics damping="0.7" friction="0.5"/>
           <param name="virtual_pin">1</param>
           <param name="servo_type">270</param>
@@ -159,4 +179,5 @@
       </joint>
       <joint name="right_elbow">
+          <dynamics damping="0.7" friction="0.5"/>
           <param name="virtual_pin">2</param>
           <param name="servo_type">270</param>
@@ -171,4 +192,5 @@
       </joint>
       <joint name="right_wrist_z_link_joint">
+          <dynamics damping="0.7" friction="0.5"/>
           <param name="virtual_pin">3</param>
           <param name="servo_type">300</param>
@@ -183,4 +205,5 @@
       </joint>
       <joint name="i01.rightHand.thumb_link_joint">
+          <dynamics damping="0.7" friction="0.5"/>
           <param name="virtual_pin">4</param>
           <param name="servo_type">300</param>
@@ -195,4 +218,5 @@
       </joint>
       <joint name="i01.rightHand.index_link_joint">
+          <dynamics damping="0.7" friction="0.5"/>
           <param name="virtual_pin">5</param>
           <param name="servo_type">300</param>
@@ -207,4 +231,5 @@
       </joint>
       <joint name="i01.rightHand.majeure_link_joint">
+          <dynamics damping="0.7" friction="0.5"/>
           <param name="virtual_pin">6</param>
           <param name="servo_type">300</param>
@@ -219,4 +244,5 @@
       </joint>
       <joint name="i01.rightHand.ringFinger_link_joint">
+          <dynamics damping="0.7" friction="0.5"/>
           <param name="virtual_pin">7</param>
           <param name="servo_type">300</param>
@@ -231,4 +257,5 @@
       </joint>
       <joint name="i01.rightHand.pinky_link_joint">
+          <dynamics damping="0.7" friction="0.5"/>
           <param name="virtual_pin">8</param>
           <param name="servo_type">300</param>
@@ -255,4 +282,5 @@
       </hardware>
       <joint name="left_shoulder_y_link_joint">
+          <dynamics damping="0.7" friction="0.5"/>
           <param name="virtual_pin">0</param>
           <param name="servo_type">270</param>
@@ -267,4 +295,5 @@
       </joint>
       <joint name="right_shoulder_y_link_joint">
+          <dynamics damping="0.7" friction="0.5"/>
           <param name="virtual_pin">1</param>
           <param name="servo_type">270</param>

Commit message: fix(naming): right_elbow renamed to right_elbow_x_link_joint

File: description/robot_description/urdf/robot_description.urdf.xacro (robot description, xacro)
@@ -261,5 +261,5 @@
     <axis xyz="0.00000 0.00000 1.00000"/>
   </joint>
-  <joint name="right_elbow" type="revolute">
+  <joint name="right_elbow_x_link_joint" type="revolute">
     <limit lower="0.00000" upper="1.57080" effort="100.00000" velocity="0.78540"/>
     <dynamics damping="0.7" friction="0.5"/>

File: description/ros2_control/inmoov_ros2_control.xacro (robot description, xacro)
@@ -158,5 +158,5 @@
           <state_interface name="position" />
       </joint>
-      <joint name="right_elbow">
+      <joint name="right_elbow_x_link_joint">
           <param name="virtual_pin">2</param>
           <param name="servo_type">270</param>
