Commit message: feat(urdf): mesh collisions, joint limit calibration, and preview tooling

File: description/robot_description/urdf/robot_description.urdf.xacro (robot description, xacro)
@@ -9,5 +9,5 @@
   </material>
   <joint name="Empty.001_link_joint" type="fixed">
-    <origin rpy="0.00000 0.00000 0.00000" xyz="-0.00394 0.00025 -0.19163"/>
+    <origin rpy="0.00000 0.00000 0.00000" xyz="${model_scale * -0.00394} ${model_scale * 0.00025} ${model_scale * -0.19163}"/>
     <parent link="base_node"/>
     <child link="stand_link"/>
@@ -16,5 +16,5 @@
     <limit lower="0" upper="0" effort="100.00000" velocity="0.78540"/>
     <dynamics damping="0.7" friction="0.5"/>
-    <origin rpy="0.00000 0.00000 0.00000" xyz="0.00000 0.00000 8.97279"/>
+    <origin rpy="0.00000 0.00000 0.00000" xyz="${model_scale * 0.00000} ${model_scale * 0.00000} ${model_scale * 8.97279}"/>
     <parent link="stand_link"/>
     <child link="torso_bottom_link"/>
@@ -22,7 +22,7 @@
   </joint>
   <joint name="i01.head.eyeRight_link_joint" type="revolute">
-    <limit lower="-0.78530" upper="0.78530" effort="100.00000" velocity="0.78540"/>
-    <dynamics damping="0.7" friction="0.5"/>
-    <origin rpy="0.00000 -0.00000 0.00000" xyz="-0.00000 -0.00590 0.00000"/>
+    <limit lower="-0.78530" upper="0.78530" effort="100.00000" velocity="0.78540"/><!-- autocalibrated: -45.0 deg .. 45.0 deg (hit_lower=False, hit_upper=False) -->
+    <dynamics damping="0.7" friction="0.5"/>
+    <origin rpy="0.00000 -0.00000 0.00000" xyz="${model_scale * -0.00000} ${model_scale * -0.00590} ${model_scale * 0.00000}"/>
     <parent link="i01.head.eyeRight.001_link"/>
     <child link="i01.head.eyeRight_link"/>
@@ -30,7 +30,7 @@
   </joint>
   <joint name="i01.head.jaw_link_joint" type="revolute">
-    <limit lower="0.00000" upper="0.17453" effort="100.00000" velocity="0.78540"/>
-    <dynamics damping="0.7" friction="0.5"/>
-    <origin rpy="-0.00000 -0.00000 -1.57080" xyz="-0.36176 0.01121 0.32442"/>
+    <limit lower="0.00000" upper="0.17453" effort="100.00000" velocity="0.78540"/><!-- autocalibrated: 0.0 deg .. 10.0 deg (hit_lower=False, hit_upper=False) -->
+    <dynamics damping="0.7" friction="0.5"/>
+    <origin rpy="-0.00000 -0.00000 -1.57080" xyz="${model_scale * -0.36176} ${model_scale * 0.01121} ${model_scale * 0.32442}"/>
     <parent link="i01.head.rothead_link"/>
     <child link="i01.head.jaw_link"/>
@@ -38,7 +38,7 @@
   </joint>
   <joint name="left_shoulder_y_link_joint" type="revolute">
-    <limit lower="0.00000" upper="1.57080" effort="100.00000" velocity="0.78540"/>
-    <dynamics damping="0.7" friction="0.5"/>
-    <origin rpy="0.00021 -0.00000 -0.00000" xyz="1.35472 -0.00337 2.80749"/>
+    <limit lower="0.00000" upper="1.57080" effort="100.00000" velocity="0.78540"/><!-- autocalibrated: 0.0 deg .. 90.0 deg (hit_lower=False, hit_upper=False) -->
+    <dynamics damping="0.7" friction="0.5"/>
+    <origin rpy="0.00021 -0.00000 -0.00000" xyz="${model_scale * 1.35472} ${model_scale * -0.00337} ${model_scale * 2.80749}"/>
     <parent link="torso_y_link"/>
     <child link="left_shoulder_y_link"/>
@@ -46,7 +46,7 @@
   </joint>
   <joint name="left_shoulder_x_link_joint" type="revolute">
-    <limit lower="-1.57080" upper="2.35619" effort="100.00000" velocity="0.78540"/>
-    <dynamics damping="0.7" friction="0.5"/>
-    <origin rpy="-0.00000 -0.00000 -0.00000" xyz="0.11351 0.00189 -0.37504"/>
+    <limit lower="-1.57080" upper="2.35619" effort="100.00000" velocity="0.78540"/><!-- autocalibrated: -90.0 deg .. 135.0 deg (hit_lower=False, hit_upper=False) -->
+    <dynamics damping="0.7" friction="0.5"/>
+    <origin rpy="-0.00000 -0.00000 -0.00000" xyz="${model_scale * 0.11351} ${model_scale * 0.00189} ${model_scale * -0.37504}"/>
     <parent link="left_shoulder_y_link"/>
     <child link="left_shoulder_x_link"/>
@@ -54,7 +54,7 @@
   </joint>
   <joint name="left_shoulder_z_link_joint" type="revolute">
-    <limit lower="-1.57080" upper="1.57080" effort="100.00000" velocity="0.78540"/>
-    <dynamics damping="0.7" friction="0.5"/>
-    <origin rpy="0.00000 0.00000 0.00000" xyz="0.62406 -0.00937 -0.59421"/>
+    <limit lower="-0.91630" upper="0.47124" effort="100.00000" velocity="0.78540"/><!-- autocalibrated: -52.5 deg .. 27.0 deg (hit_lower=False, hit_upper=False) -->
+    <dynamics damping="0.7" friction="0.5"/>
+    <origin rpy="0.00000 0.00000 0.00000" xyz="${model_scale * 0.62406} ${model_scale * -0.00937} ${model_scale * -0.59421}"/>
     <parent link="left_shoulder_x_link"/>
     <child link="left_shoulder_z_link"/>
@@ -62,7 +62,7 @@
   </joint>
   <joint name="left_elbow_x_link_joint" type="revolute">
-    <limit lower="0.00000" upper="1.57080" effort="100.00000" velocity="0.78540"/>
-    <dynamics damping="0.7" friction="0.5"/>
-    <origin rpy="0.06567 -0.00000 -0.00000" xyz="-0.01281 0.29228 -2.11577"/>
+    <limit lower="0.00000" upper="1.57080" effort="100.00000" velocity="0.78540"/><!-- autocalibrated: 0.0 deg .. 90.0 deg (hit_lower=False, hit_upper=False) -->
+    <dynamics damping="0.7" friction="0.5"/>
+    <origin rpy="0.06567 -0.00000 -0.00000" xyz="${model_scale * -0.01281} ${model_scale * 0.29228} ${model_scale * -2.11577}"/>
     <parent link="left_shoulder_z_link"/>
     <child link="left_elbow_x_link"/>
@@ -70,7 +70,7 @@
   </joint>
   <joint name="left_wrist_z_link_joint" type="revolute">
-    <limit lower="-1.57080" upper="1.57080" effort="100.00000" velocity="0.78540"/>
-    <dynamics damping="0.7" friction="0.5"/>
-    <origin rpy="-0.41605 -0.00000 0.00000" xyz="-0.08767 -0.98766 -2.53936"/>
+    <limit lower="-1.57080" upper="1.57080" effort="100.00000" velocity="0.78540"/><!-- autocalibrated: -90.0 deg .. 90.0 deg (hit_lower=False, hit_upper=False) -->
+    <dynamics damping="0.7" friction="0.5"/>
+    <origin rpy="-0.41605 -0.00000 0.00000" xyz="${model_scale * -0.08767} ${model_scale * -0.98766} ${model_scale * -2.53936}"/>
     <parent link="left_elbow_x_link"/>
     <child link="left_wrist_z_link"/>
@@ -80,5 +80,5 @@
     <limit lower="0.00000" upper="1.57080" effort="100.00000" velocity="0.78540"/>
     <dynamics damping="0.7" friction="0.5"/>
-    <origin rpy="-0.00000 0.00000 -0.61611" xyz="-0.00000 -0.00000 -0.16925"/>
+    <origin rpy="-0.00000 0.00000 -0.61611" xyz="${model_scale * -0.00000} ${model_scale * -0.00000} ${model_scale * -0.16925}"/>
     <parent link="left_wrist_z_link"/>
     <child link="i01.leftHand.wrist.001_link"/>
@@ -86,7 +86,7 @@
   </joint>
   <joint name="i01.leftHand.index_link_joint" type="revolute">
-    <limit lower="0.00000" upper="1.57080" effort="100.00000" velocity="0.78540"/>
-    <dynamics damping="0.7" friction="0.5"/>
-    <origin rpy="-1.56854 -0.09096 -0.00330" xyz="0.32645 -0.01145 -0.94982"/>
+    <limit lower="0.00000" upper="1.57080" effort="100.00000" velocity="0.78540"/><!-- autocalibrated: 0.0 deg .. 90.0 deg (hit_lower=False, hit_upper=False) -->
+    <dynamics damping="0.7" friction="0.5"/>
+    <origin rpy="-1.56854 -0.09096 -0.00330" xyz="${model_scale * 0.32645} ${model_scale * -0.01145} ${model_scale * -0.94982}"/>
     <parent link="i01.leftHand.wrist.001_link"/>
     <child link="i01.leftHand.index_link"/>
@@ -96,5 +96,5 @@
     <limit lower="0.00000" upper="1.57080" effort="100.00000" velocity="0.78540"/>
     <dynamics damping="0.7" friction="0.5"/>
-    <origin rpy="-0.00000 0.00000 -0.00000" xyz="0.00258 0.34105 0.00685"/>
+    <origin rpy="-0.00000 0.00000 -0.00000" xyz="${model_scale * 0.00258} ${model_scale * 0.34105} ${model_scale * 0.00685}"/>
     <parent link="i01.leftHand.index_link"/>
     <child link="i01.leftHand.index2_link"/>
@@ -102,7 +102,7 @@
   </joint>
   <joint name="i01.torso.midStom_link_joint" type="revolute">
-    <limit lower="-2.35619" upper="2.35619" effort="100.00000" velocity="0.78540"/>
-    <dynamics damping="0.7" friction="0.5"/>
-    <origin rpy="0.00000 0.06589 1.57080" xyz="-0.00213 0.05565 1.13807"/>
+    <limit lower="-0.50615" upper="0.50615" effort="100.00000" velocity="0.78540"/><!-- autocalibrated: -29.0 deg .. 29.0 deg (hit_lower=False, hit_upper=False) -->
+    <dynamics damping="0.7" friction="0.5"/>
+    <origin rpy="0.00000 0.06589 1.57080" xyz="${model_scale * -0.00213} ${model_scale * 0.05565} ${model_scale * 1.13807}"/>
     <parent link="torso_bottom_link"/>
     <child link="torso_z_link"/>
@@ -112,5 +112,5 @@
     <limit lower="0.00000" upper="1.57080" effort="100.00000" velocity="0.78540"/>
     <dynamics damping="0.7" friction="0.5"/>
-    <origin rpy="0.00000 -0.00000 -0.00000" xyz="0.00103 0.22697 0.00433"/>
+    <origin rpy="0.00000 -0.00000 -0.00000" xyz="${model_scale * 0.00103} ${model_scale * 0.22697} ${model_scale * 0.00433}"/>
     <parent link="i01.leftHand.index2_link"/>
     <child link="i01.leftHand.index3_link"/>
@@ -118,7 +118,7 @@
   </joint>
   <joint name="i01.leftHand.majeure_link_joint" type="revolute">
-    <limit lower="0.00000" upper="1.57080" effort="100.00000" velocity="0.78540"/>
-    <dynamics damping="0.7" friction="0.5"/>
-    <origin rpy="-1.56854 0.00160 -0.00309" xyz="0.07161 -0.01170 -0.98881"/>
+    <limit lower="0.00000" upper="1.57080" effort="100.00000" velocity="0.78540"/><!-- autocalibrated: 0.0 deg .. 90.0 deg (hit_lower=False, hit_upper=False) -->
+    <dynamics damping="0.7" friction="0.5"/>
+    <origin rpy="-1.56854 0.00160 -0.00309" xyz="${model_scale * 0.07161} ${model_scale * -0.01170} ${model_scale * -0.98881}"/>
     <parent link="i01.leftHand.wrist.001_link"/>
     <child link="i01.leftHand.majeure_link"/>
@@ -128,5 +128,5 @@
     <limit lower="0.00000" upper="1.57080" effort="100.00000" velocity="0.78540"/>
     <dynamics damping="0.7" friction="0.5"/>
-    <origin rpy="-0.00000 -0.00000 0.00000" xyz="0.00272 0.35935 0.00722"/>
+    <origin rpy="-0.00000 -0.00000 0.00000" xyz="${model_scale * 0.00272} ${model_scale * 0.35935} ${model_scale * 0.00722}"/>
     <parent link="i01.leftHand.majeure_link"/>
     <child link="i01.leftHand.majeure2_link"/>
@@ -136,5 +136,5 @@
     <limit lower="0.00000" upper="1.57080" effort="100.00000" velocity="0.78540"/>
     <dynamics damping="0.7" friction="0.5"/>
-    <origin rpy="0.00000 -0.00000 -0.00000" xyz="0.00109 0.23915 0.00456"/>
+    <origin rpy="0.00000 -0.00000 -0.00000" xyz="${model_scale * 0.00109} ${model_scale * 0.23915} ${model_scale * 0.00456}"/>
     <parent link="i01.leftHand.majeure2_link"/>
     <child link="i01.leftHand.majeure3_link"/>
@@ -144,5 +144,5 @@
     <limit lower="0.00000" upper="1.57080" effort="100.00000" velocity="0.78540"/>
     <dynamics damping="0.7" friction="0.5"/>
-    <origin rpy="-1.56789 -0.68643 -0.00494" xyz="-0.24002 0.00108 -0.35218"/>
+    <origin rpy="-1.56789 -0.68643 -0.00494" xyz="${model_scale * -0.24002} ${model_scale * 0.00108} ${model_scale * -0.35218}"/>
     <parent link="i01.leftHand.wrist.001_link"/>
     <child link="i01.leftHand.pinky0_link"/>
@@ -150,7 +150,7 @@
   </joint>
   <joint name="i01.leftHand.pinky_link_joint" type="revolute">
-    <limit lower="0.00000" upper="1.57080" effort="100.00000" velocity="0.78540"/>
-    <dynamics damping="0.7" friction="0.5"/>
-    <origin rpy="-0.00000 0.00000 0.94526" xyz="-0.43178 0.20489 0.00726"/>
+    <limit lower="0.00000" upper="1.57080" effort="100.00000" velocity="0.78540"/><!-- autocalibrated: 0.0 deg .. 90.0 deg (hit_lower=False, hit_upper=False) -->
+    <dynamics damping="0.7" friction="0.5"/>
+    <origin rpy="-0.00000 0.00000 0.94526" xyz="${model_scale * -0.43178} ${model_scale * 0.20489} ${model_scale * 0.00726}"/>
     <parent link="i01.leftHand.pinky0_link"/>
     <child link="i01.leftHand.pinky_link"/>
@@ -160,5 +160,5 @@
     <limit lower="0.00000" upper="1.57080" effort="100.00000" velocity="0.78540"/>
     <dynamics damping="0.7" friction="0.5"/>
-    <origin rpy="-0.00000 0.00000 -0.00000" xyz="0.00225 0.29796 0.00599"/>
+    <origin rpy="-0.00000 0.00000 -0.00000" xyz="${model_scale * 0.00225} ${model_scale * 0.29796} ${model_scale * 0.00599}"/>
     <parent link="i01.leftHand.pinky_link"/>
     <child link="i01.leftHand.pinky2_link"/>
@@ -168,5 +168,5 @@
     <limit lower="0.00000" upper="1.57080" effort="100.00000" velocity="0.78540"/>
     <dynamics damping="0.7" friction="0.5"/>
-    <origin rpy="-0.00000 -0.00000 -0.00000" xyz="0.00090 0.19830 0.00378"/>
+    <origin rpy="-0.00000 -0.00000 -0.00000" xyz="${model_scale * 0.00090} ${model_scale * 0.19830} ${model_scale * 0.00378}"/>
     <parent link="i01.leftHand.pinky2_link"/>
     <child link="i01.leftHand.pinky3_link"/>
@@ -176,5 +176,5 @@
     <limit lower="0.00000" upper="1.57080" effort="100.00000" velocity="0.78540"/>
     <dynamics damping="0.7" friction="0.5"/>
-    <origin rpy="-1.56789 -0.68643 -0.00494" xyz="-0.05673 0.00101 -0.57588"/>
+    <origin rpy="-1.56789 -0.68643 -0.00494" xyz="${model_scale * -0.05673} ${model_scale * 0.00101} ${model_scale * -0.57588}"/>
     <parent link="i01.leftHand.wrist.001_link"/>
     <child link="i01.leftHand.ringfinger0_link"/>
@@ -182,7 +182,7 @@
   </joint>
   <joint name="i01.leftHand.ringFinger_link_joint" type="revolute">
-    <limit lower="0.00000" upper="1.57080" effort="100.00000" velocity="0.78540"/>
-    <dynamics damping="0.7" friction="0.5"/>
-    <origin rpy="-0.00000 0.00000 0.77485" xyz="-0.33329 0.15280 -0.00664"/>
+    <limit lower="0.00000" upper="1.57080" effort="100.00000" velocity="0.78540"/><!-- autocalibrated: 0.0 deg .. 90.0 deg (hit_lower=False, hit_upper=False) -->
+    <dynamics damping="0.7" friction="0.5"/>
+    <origin rpy="-0.00000 0.00000 0.77485" xyz="${model_scale * -0.33329} ${model_scale * 0.15280} ${model_scale * -0.00664}"/>
     <parent link="i01.leftHand.ringfinger0_link"/>
     <child link="i01.leftHand.ringFinger_link"/>
@@ -190,7 +190,7 @@
   </joint>
   <joint name="i01.torso.topStom_link_joint" type="revolute">
-    <limit lower="-0.34907" upper="0.34907" effort="100.00000" velocity="0.78540"/>
-    <dynamics damping="0.7" friction="0.5"/>
-    <origin rpy="0.00000 0.00000 -1.57080" xyz="-0.06317 0.00033 1.01916"/>
+    <limit lower="-0.12217" upper="0.12217" effort="100.00000" velocity="0.78540"/><!-- autocalibrated: -7.0 deg .. 7.0 deg (hit_lower=False, hit_upper=False) -->
+    <dynamics damping="0.7" friction="0.5"/>
+    <origin rpy="0.00000 0.00000 -1.57080" xyz="${model_scale * -0.06317} ${model_scale * 0.00033} ${model_scale * 1.01916}"/>
     <parent link="torso_z_link"/>
     <child link="torso_y_link"/>
@@ -200,5 +200,5 @@
     <limit lower="0.00000" upper="1.57080" effort="100.00000" velocity="0.78540"/>
     <dynamics damping="0.7" friction="0.5"/>
-    <origin rpy="-0.00000 -0.00000 0.00000" xyz="0.00258 0.34105 0.00685"/>
+    <origin rpy="-0.00000 -0.00000 0.00000" xyz="${model_scale * 0.00258} ${model_scale * 0.34105} ${model_scale * 0.00685}"/>
     <parent link="i01.leftHand.ringFinger_link"/>
     <child link="i01.leftHand.ringfinger2_link"/>
@@ -208,5 +208,5 @@
     <limit lower="0.00000" upper="1.57080" effort="100.00000" velocity="0.78540"/>
     <dynamics damping="0.7" friction="0.5"/>
-    <origin rpy="-0.00000 0.00000 -0.00000" xyz="0.00103 0.22697 0.00433"/>
+    <origin rpy="-0.00000 0.00000 -0.00000" xyz="${model_scale * 0.00103} ${model_scale * 0.22697} ${model_scale * 0.00433}"/>
     <parent link="i01.leftHand.ringfinger2_link"/>
     <child link="i01.leftHand.ringfinger3_link"/>
@@ -216,5 +216,5 @@
     <limit lower="0.00000" upper="1.57080" effort="100.00000" velocity="0.78540"/>
     <dynamics damping="0.7" friction="0.5"/>
-    <origin rpy="1.51635 -0.09893 -0.00332" xyz="0.28234 -0.00002 -0.37340"/>
+    <origin rpy="1.51635 -0.09893 -0.00332" xyz="${model_scale * 0.28234} ${model_scale * -0.00002} ${model_scale * -0.37340}"/>
     <parent link="i01.leftHand.wrist.001_link"/>
     <child link="i01.leftHand.thumb1_link"/>
@@ -222,7 +222,7 @@
   </joint>
   <joint name="i01.leftHand.thumb_link_joint" type="revolute">
-    <limit lower="0.00000" upper="1.57080" effort="100.00000" velocity="0.78540"/>
-    <dynamics damping="0.7" friction="0.5"/>
-    <origin rpy="-0.03182 -0.32566 0.83064" xyz="0.25977 -0.13332 -0.00800"/>
+    <limit lower="0.00000" upper="1.57080" effort="100.00000" velocity="0.78540"/><!-- autocalibrated: 0.0 deg .. 90.0 deg (hit_lower=False, hit_upper=False) -->
+    <dynamics damping="0.7" friction="0.5"/>
+    <origin rpy="-0.03182 -0.32566 0.83064" xyz="${model_scale * 0.25977} ${model_scale * -0.13332} ${model_scale * -0.00800}"/>
     <parent link="i01.leftHand.thumb1_link"/>
     <child link="i01.leftHand.thumb_link"/>
@@ -232,5 +232,5 @@
     <limit lower="0.00000" upper="1.57080" effort="100.00000" velocity="0.78540"/>
     <dynamics damping="0.7" friction="0.5"/>
-    <origin rpy="0.00001 -0.00000 0.00000" xyz="0.01229 -0.33047 -0.00704"/>
+    <origin rpy="0.00001 -0.00000 0.00000" xyz="${model_scale * 0.01229} ${model_scale * -0.33047} ${model_scale * -0.00704}"/>
     <parent link="i01.leftHand.thumb_link"/>
     <child link="i01.leftHand.thumb3_link"/>
@@ -238,7 +238,7 @@
   </joint>
   <joint name="right_shoulder_y_link_joint" type="revolute">
-    <limit lower="0.00000" upper="1.57080" effort="100.00000" velocity="0.78540"/>
-    <dynamics damping="0.7" friction="0.5"/>
-    <origin rpy="0.00021 -0.00000 -0.00000" xyz="-1.34979 -0.00337 2.80749"/>
+    <limit lower="0.00000" upper="1.57080" effort="100.00000" velocity="0.78540"/><!-- autocalibrated: 0.0 deg .. 90.0 deg (hit_lower=False, hit_upper=False) -->
+    <dynamics damping="0.7" friction="0.5"/>
+    <origin rpy="0.00021 -0.00000 -0.00000" xyz="${model_scale * -1.34979} ${model_scale * -0.00337} ${model_scale * 2.80749}"/>
     <parent link="torso_y_link"/>
     <child link="right_shoulder_y_link"/>
@@ -246,7 +246,7 @@
   </joint>
   <joint name="right_shoulder_x_link_joint" type="revolute">
-    <limit lower="-1.57080" upper="2.35619" effort="100.00000" velocity="0.78540"/>
-    <dynamics damping="0.7" friction="0.5"/>
-    <origin rpy="-0.00000 -0.00000 -0.00000" xyz="-0.11351 0.00189 -0.37504"/>
+    <limit lower="-1.57080" upper="2.35619" effort="100.00000" velocity="0.78540"/><!-- autocalibrated: -90.0 deg .. 135.0 deg (hit_lower=False, hit_upper=False) -->
+    <dynamics damping="0.7" friction="0.5"/>
+    <origin rpy="-0.00000 -0.00000 -0.00000" xyz="${model_scale * -0.11351} ${model_scale * 0.00189} ${model_scale * -0.37504}"/>
     <parent link="right_shoulder_y_link"/>
     <child link="right_shoulder_x_link"/>
@@ -254,7 +254,7 @@
   </joint>
   <joint name="right_shoulder_z_link_joint" type="revolute">
-    <limit lower="-1.57080" upper="1.57080" effort="100.00000" velocity="0.78540"/>
-    <dynamics damping="0.7" friction="0.5"/>
-    <origin rpy="0.00000 0.00000 0.00000" xyz="-0.62406 -0.00937 -0.59421"/>
+    <limit lower="-0.42761" upper="0.83776" effort="100.00000" velocity="0.78540"/><!-- autocalibrated: -24.5 deg .. 48.0 deg (hit_lower=False, hit_upper=False) -->
+    <dynamics damping="0.7" friction="0.5"/>
+    <origin rpy="0.00000 0.00000 0.00000" xyz="${model_scale * -0.62406} ${model_scale * -0.00937} ${model_scale * -0.59421}"/>
     <parent link="right_shoulder_x_link"/>
     <child link="right_shoulder_z_link"/>
@@ -262,7 +262,7 @@
   </joint>
   <joint name="right_elbow_x_link_joint" type="revolute">
-    <limit lower="0.00000" upper="1.57080" effort="100.00000" velocity="0.78540"/>
-    <dynamics damping="0.7" friction="0.5"/>
-    <origin rpy="0.06567 0.00000 0.00000" xyz="0.00858 0.29228 -2.11577"/>
+    <limit lower="0.00000" upper="1.57080" effort="100.00000" velocity="0.78540"/><!-- autocalibrated: 0.0 deg .. 90.0 deg (hit_lower=False, hit_upper=False) -->
+    <dynamics damping="0.7" friction="0.5"/>
+    <origin rpy="0.06567 0.00000 0.00000" xyz="${model_scale * 0.00858} ${model_scale * 0.29228} ${model_scale * -2.11577}"/>
     <parent link="right_shoulder_z_link"/>
     <child link="right_elbow_x_link"/>
@@ -270,7 +270,7 @@
   </joint>
   <joint name="right_wrist_z_link_joint" type="revolute">
-    <limit lower="-1.57080" upper="1.57080" effort="100.00000" velocity="0.78540"/>
-    <dynamics damping="0.7" friction="0.5"/>
-    <origin rpy="-0.41605 0.00000 0.00000" xyz="0.08767 -0.98766 -2.53936"/>
+    <limit lower="-1.57080" upper="1.57080" effort="100.00000" velocity="0.78540"/><!-- autocalibrated: -90.0 deg .. 90.0 deg (hit_lower=False, hit_upper=False) -->
+    <dynamics damping="0.7" friction="0.5"/>
+    <origin rpy="-0.41605 0.00000 0.00000" xyz="${model_scale * 0.08767} ${model_scale * -0.98766} ${model_scale * -2.53936}"/>
     <parent link="right_elbow_x_link"/>
     <child link="right_wrist_z_link"/>
@@ -278,7 +278,7 @@
   </joint>
   <joint name="i01.head.neck.001_link_joint" type="revolute">
-    <limit lower="-0.34907" upper="0.34907" effort="100.00000" velocity="0.78540"/>
-    <dynamics damping="0.7" friction="0.5"/>
-    <origin rpy="0.06589 -0.00000 -0.00000" xyz="0.00390 0.29817 4.29073"/>
+    <limit lower="-0.34907" upper="0.00000" effort="100.00000" velocity="0.78540"/><!-- autocalibrated: -20.0 deg .. 0.0 deg (hit_lower=False, hit_upper=False) -->
+    <dynamics damping="0.7" friction="0.5"/>
+    <origin rpy="0.06589 -0.00000 -0.00000" xyz="${model_scale * 0.00390} ${model_scale * 0.29817} ${model_scale * 4.29073}"/>
     <parent link="torso_y_link"/>
     <child link="i01.head.neck.001_link"/>
@@ -288,5 +288,5 @@
     <limit lower="0.00000" upper="1.57080" effort="100.00000" velocity="0.78540"/>
     <dynamics damping="0.7" friction="0.5"/>
-    <origin rpy="0.00000 0.00000 0.63517" xyz="-0.00000 -0.00000 -0.16508"/>
+    <origin rpy="0.00000 0.00000 0.63517" xyz="${model_scale * -0.00000} ${model_scale * -0.00000} ${model_scale * -0.16508}"/>
     <parent link="right_wrist_z_link"/>
     <child link="i01.rightHand.wrist.001_link"/>
@@ -294,7 +294,7 @@
   </joint>
   <joint name="i01.rightHand.index_link_joint" type="revolute">
-    <limit lower="0.00000" upper="1.57080" effort="100.00000" velocity="0.78540"/>
-    <dynamics damping="0.7" friction="0.5"/>
-    <origin rpy="1.57305 0.09096 -0.01576" xyz="-0.32320 -0.00773 -0.95398"/>
+    <limit lower="0.00000" upper="1.57080" effort="100.00000" velocity="0.78540"/><!-- autocalibrated: 0.0 deg .. 90.0 deg (hit_lower=False, hit_upper=False) -->
+    <dynamics damping="0.7" friction="0.5"/>
+    <origin rpy="1.57305 0.09096 -0.01576" xyz="${model_scale * -0.32320} ${model_scale * -0.00773} ${model_scale * -0.95398}"/>
     <parent link="i01.rightHand.wrist.001_link"/>
     <child link="i01.rightHand.index_link"/>
@@ -304,5 +304,5 @@
     <limit lower="0.00000" upper="1.57080" effort="100.00000" velocity="0.78540"/>
     <dynamics damping="0.7" friction="0.5"/>
-    <origin rpy="0.00000 -0.00000 0.00000" xyz="-0.00258 -0.34105 -0.00685"/>
+    <origin rpy="0.00000 -0.00000 0.00000" xyz="${model_scale * -0.00258} ${model_scale * -0.34105} ${model_scale * -0.00685}"/>
     <parent link="i01.rightHand.index_link"/>
     <child link="i01.rightHand.index2_link"/>
@@ -312,5 +312,5 @@
     <limit lower="0.00000" upper="1.57080" effort="100.00000" velocity="0.78540"/>
     <dynamics damping="0.7" friction="0.5"/>
-    <origin rpy="0.00000 0.00000 -0.00000" xyz="-0.00103 -0.22697 -0.00432"/>
+    <origin rpy="0.00000 0.00000 -0.00000" xyz="${model_scale * -0.00103} ${model_scale * -0.22697} ${model_scale * -0.00432}"/>
     <parent link="i01.rightHand.index2_link"/>
     <child link="i01.rightHand.index3_link"/>
@@ -318,7 +318,7 @@
   </joint>
   <joint name="i01.rightHand.majeure_link_joint" type="revolute">
-    <limit lower="0.00000" upper="1.57080" effort="100.00000" velocity="0.78540"/>
-    <dynamics damping="0.7" friction="0.5"/>
-    <origin rpy="1.57305 -0.00160 -0.01597" xyz="-0.06841 -0.01284 -0.99297"/>
+    <limit lower="0.00000" upper="1.57080" effort="100.00000" velocity="0.78540"/><!-- autocalibrated: 0.0 deg .. 90.0 deg (hit_lower=False, hit_upper=False) -->
+    <dynamics damping="0.7" friction="0.5"/>
+    <origin rpy="1.57305 -0.00160 -0.01597" xyz="${model_scale * -0.06841} ${model_scale * -0.01284} ${model_scale * -0.99297}"/>
     <parent link="i01.rightHand.wrist.001_link"/>
     <child link="i01.rightHand.majeure_link"/>
@@ -328,5 +328,5 @@
     <limit lower="0.00000" upper="1.57080" effort="100.00000" velocity="0.78540"/>
     <dynamics damping="0.7" friction="0.5"/>
-    <origin rpy="-0.00000 -0.00000 -0.00000" xyz="-0.00272 -0.35935 -0.00722"/>
+    <origin rpy="-0.00000 -0.00000 -0.00000" xyz="${model_scale * -0.00272} ${model_scale * -0.35935} ${model_scale * -0.00722}"/>
     <parent link="i01.rightHand.majeure_link"/>
     <child link="i01.rightHand.majeure2_link"/>
@@ -336,5 +336,5 @@
     <limit lower="0.00000" upper="1.57080" effort="100.00000" velocity="0.78540"/>
     <dynamics damping="0.7" friction="0.5"/>
-    <origin rpy="0.00000 -0.00000 0.00000" xyz="-0.00109 -0.23915 -0.00456"/>
+    <origin rpy="0.00000 -0.00000 0.00000" xyz="${model_scale * -0.00109} ${model_scale * -0.23915} ${model_scale * -0.00456}"/>
     <parent link="i01.rightHand.majeure2_link"/>
     <child link="i01.rightHand.majeure3_link"/>
@@ -344,5 +344,5 @@
     <limit lower="0.00000" upper="1.57080" effort="100.00000" velocity="0.78540"/>
     <dynamics damping="0.7" friction="0.5"/>
-    <origin rpy="1.57370 0.68643 -0.01412" xyz="0.24340 -0.00601 -0.35634"/>
+    <origin rpy="1.57370 0.68643 -0.01412" xyz="${model_scale * 0.24340} ${model_scale * -0.00601} ${model_scale * -0.35634}"/>
     <parent link="i01.rightHand.wrist.001_link"/>
     <child link="i01.rightHand.pinky0_link"/>
@@ -350,7 +350,7 @@
   </joint>
   <joint name="i01.rightHand.pinky_link_joint" type="revolute">
-    <limit lower="0.00000" upper="1.57080" effort="100.00000" velocity="0.78540"/>
-    <dynamics damping="0.7" friction="0.5"/>
-    <origin rpy="-0.00000 -0.00000 0.94526" xyz="0.43178 -0.20489 -0.00726"/>
+    <limit lower="0.00000" upper="1.57080" effort="100.00000" velocity="0.78540"/><!-- autocalibrated: 0.0 deg .. 90.0 deg (hit_lower=False, hit_upper=False) -->
+    <dynamics damping="0.7" friction="0.5"/>
+    <origin rpy="-0.00000 -0.00000 0.94526" xyz="${model_scale * 0.43178} ${model_scale * -0.20489} ${model_scale * -0.00726}"/>
     <parent link="i01.rightHand.pinky0_link"/>
     <child link="i01.rightHand.pinky_link"/>
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