Commit message: feat(urdf): mesh collisions, joint limit calibration, and preview tooling

File: description/ros2_control/inmoov_gazebo.xacro (robot description, xacro)
@@ -1,5 +1,10 @@
 <?xml version="1.0"?>
 <!-- Gazebo plugin for gz_ros2_control: runs controller_manager inside Gazebo and drives simulated joints.
-     Expects controller_config arg from parent (inmoov.urdf.xacro). -->
+     Expects controller_config arg from parent (inmoov.urdf.xacro).
+     Collision strategy: every URDF link reuses its visual mesh as the collision
+     mesh (see scripts/inject_collisions.py). Gazebo macros below only assign
+     surface/contact properties — `gazebo_body_link` disables self_collide on
+     adjacent body meshes (avoids jitter), `gazebo_hand_link` enables it with
+     friction tuned for grasping. -->
 <robot xmlns:xacro="http://www.ros.org/wiki/xacro">
   <!-- Fix entire stand to the world so the robot does not fall (gz-sim may still move root; heavy mass in URDF is fallback). -->
@@ -10,4 +15,67 @@
     <static>true</static>
   </gazebo>
+  <!-- Body links: full-mesh collisions with self-collision disabled. Adjacent
+       shoulder/elbow meshes overlap at neutral pose; enabling self-collide
+       there causes jitter in gz-sim. Tighten contact stiffness defaults. -->
+  <xacro:macro name="gazebo_body_link" params="link">
+    <gazebo reference="${link}">
+      <mu1>0.6</mu1>
+      <mu2>0.6</mu2>
+      <kp>1e6</kp>
+      <kd>10</kd>
+      <self_collide>false</self_collide>
+    </gazebo>
+  </xacro:macro>
+  <xacro:gazebo_body_link link="torso_bottom_link"/>
+  <xacro:gazebo_body_link link="torso_z_link"/>
+  <xacro:gazebo_body_link link="torso_y_link"/>
+  <xacro:gazebo_body_link link="left_shoulder_y_link"/>
+  <xacro:gazebo_body_link link="left_shoulder_x_link"/>
+  <xacro:gazebo_body_link link="left_shoulder_z_link"/>
+  <xacro:gazebo_body_link link="left_elbow_x_link"/>
+  <xacro:gazebo_body_link link="left_wrist_z_link"/>
+  <xacro:gazebo_body_link link="right_shoulder_y_link"/>
+  <xacro:gazebo_body_link link="right_shoulder_x_link"/>
+  <xacro:gazebo_body_link link="right_shoulder_z_link"/>
+  <xacro:gazebo_body_link link="right_elbow_x_link"/>
+  <xacro:gazebo_body_link link="right_wrist_z_link"/>
+  <xacro:gazebo_body_link link="neck_link"/>
+  <xacro:gazebo_body_link link="i01.head.rothead_link"/>
+  <xacro:gazebo_body_link link="i01.head.jaw_link"/>
+  <!-- Finger / palm links: mesh collisions with high friction + self-collide
+       so finger-finger and finger-palm contacts work for grasping. Every
+       phalanx (proximal/medial/distal), abductor base, and the wrist palm
+       carry the same surface props. -->
+  <xacro:macro name="gazebo_hand_link" params="link">
+    <gazebo reference="${link}">
+      <mu1>0.9</mu1>
+      <mu2>0.9</mu2>
+      <kp>1e6</kp>
+      <kd>10</kd>
+      <self_collide>true</self_collide>
+    </gazebo>
+  </xacro:macro>
+  <xacro:macro name="gazebo_hand_side" params="side">
+    <xacro:gazebo_hand_link link="i01.${side}Hand.wrist.001_link"/>
+    <xacro:gazebo_hand_link link="i01.${side}Hand.index_link"/>
+    <xacro:gazebo_hand_link link="i01.${side}Hand.index2_link"/>
+    <xacro:gazebo_hand_link link="i01.${side}Hand.index3_link"/>
+    <xacro:gazebo_hand_link link="i01.${side}Hand.majeure_link"/>
+    <xacro:gazebo_hand_link link="i01.${side}Hand.majeure2_link"/>
+    <xacro:gazebo_hand_link link="i01.${side}Hand.majeure3_link"/>
+    <xacro:gazebo_hand_link link="i01.${side}Hand.ringfinger0_link"/>
+    <xacro:gazebo_hand_link link="i01.${side}Hand.ringFinger_link"/>
+    <xacro:gazebo_hand_link link="i01.${side}Hand.ringfinger2_link"/>
+    <xacro:gazebo_hand_link link="i01.${side}Hand.ringfinger3_link"/>
+    <xacro:gazebo_hand_link link="i01.${side}Hand.pinky0_link"/>
+    <xacro:gazebo_hand_link link="i01.${side}Hand.pinky_link"/>
+    <xacro:gazebo_hand_link link="i01.${side}Hand.pinky2_link"/>
+    <xacro:gazebo_hand_link link="i01.${side}Hand.pinky3_link"/>
+    <xacro:gazebo_hand_link link="i01.${side}Hand.thumb1_link"/>
+    <xacro:gazebo_hand_link link="i01.${side}Hand.thumb_link"/>
+    <xacro:gazebo_hand_link link="i01.${side}Hand.thumb3_link"/>
+  </xacro:macro>
+  <xacro:gazebo_hand_side side="left"/>
+  <xacro:gazebo_hand_side side="right"/>
   <gazebo>
     <plugin filename="gz_ros2_control-system" name="gz_ros2_control::GazeboSimROS2ControlPlugin">

File: description/ros2_control/inmoov_ros2_control.xacro (robot description, xacro)
@@ -294,25 +294,25 @@
           <state_interface name="position" />
       </joint>
+      <joint name="i01.torso.midStom_link_joint">
+          <param name="virtual_pin">2</param>
+          <param name="servo_type">180</param>
+          <param name="offset_deg">90</param>
+          <param name="direction">1</param>
+          <param name="scale">1</param>
+          <param name="servo_min_deg">0</param>
+          <param name="servo_max_deg">180</param>
+          <param name="servo_default_deg">90</param>
+          <command_interface name="position" />
+          <state_interface name="position" />
+      </joint>
       <joint name="i01.torso.topStom_link_joint">
-          <param name="virtual_pin">2</param>
-          <param name="servo_type">270</param>
-          <param name="offset_deg">0</param>
-          <param name="direction">1</param>
-          <param name="scale">1</param>
-          <param name="servo_min_deg">0</param>
-          <param name="servo_max_deg">270</param>
-          <param name="servo_default_deg">135</param>
-          <command_interface name="position" />
-          <state_interface name="position" />
-      </joint>
-      <joint name="i01.torso.midStom_link_joint">
           <param name="virtual_pin">3</param>
-          <param name="servo_type">270</param>
-          <param name="offset_deg">0</param>
-          <param name="direction">1</param>
-          <param name="scale">1</param>
-          <param name="servo_min_deg">0</param>
-          <param name="servo_max_deg">270</param>
-          <param name="servo_default_deg">135</param>
+          <param name="servo_type">180</param>
+          <param name="offset_deg">0</param>
+          <param name="direction">1</param>
+          <param name="scale">1</param>
+          <param name="servo_min_deg">0</param>
+          <param name="servo_max_deg">180</param>
+          <param name="servo_default_deg">90</param>
           <command_interface name="position" />
           <state_interface name="position" />

File: description/urdf/inmoov.urdf.xacro (robot description, xacro)
@@ -4,7 +4,10 @@
   <xacro:arg name="base_path" default="."/>
   <xacro:arg name="use_gazebo_sim" default="false"/>
+  <xacro:arg name="use_mock_hardware" default="false"/>
   <xacro:arg name="controller_config" default=""/>
   <xacro:property name="mesh_dir" value="file://$(arg base_path)/robot_description/meshes/dae"/>
   <xacro:property name="use_gazebo_sim" value="$(arg use_gazebo_sim)"/>
+  <!-- model_scale lives in properties.xacro; not a launch argument. -->
+  <xacro:include filename="../robot_description/urdf/properties.xacro"/>
   <!-- Import inmoov physical description (urdf) macro (uses use_gazebo_sim for heavy stand in sim) -->
   <xacro:include filename="../robot_description/urdf/robot_description.urdf.xacro"/>

Commit message: fix(gazebo): strip DAE line primitives and drop empty Texture.261/262 mesh refs

File: description/robot_description/urdf/robot_description.urdf.xacro (robot description, xacro)
@@ -724,16 +724,4 @@
       </geometry>
     </collision>
-    <collision name="i01..leftArm.shoulder.full.008_collision">
-      <origin rpy="0.06568 0.00000 0.00000" xyz="${model_scale * -1.46578} ${model_scale * 1.11459} ${model_scale * -13.51522}"/>
-      <geometry>
-        <mesh filename="${mesh_dir}/Texture.261.dae" scale="${model_scale * 1.00000} ${model_scale * 1.00000} ${model_scale * 1.00000}"/>
-      </geometry>
-    </collision>
-    <collision name="i01..leftArm.shoulder.full.009_collision">
-      <origin rpy="0.06568 0.00000 0.00000" xyz="${model_scale * -1.46578} ${model_scale * 1.11459} ${model_scale * -13.51522}"/>
-      <geometry>
-        <mesh filename="${mesh_dir}/Texture.262.dae" scale="${model_scale * 1.00000} ${model_scale * 1.00000} ${model_scale * 1.00000}"/>
-      </geometry>
-    </collision>
     <collision name="i01..leftArm.shoulder.full.010_collision">
       <origin rpy="0.06568 0.00000 0.00000" xyz="${model_scale * -1.46578} ${model_scale * 1.11459} ${model_scale * -13.51522}"/>
@@ -826,18 +814,4 @@
       <geometry>
         <mesh filename="${mesh_dir}/Texture.260.dae" scale="${model_scale * 1.00000} ${model_scale * 1.00000} ${model_scale * 1.00000}"/>
-      </geometry>
-    </visual>
-    <visual name="i01..leftArm.shoulder.full.008">
-      <material name="Material.390"/>
-      <origin rpy="0.06568 0.00000 0.00000" xyz="${model_scale * -1.46578} ${model_scale * 1.11459} ${model_scale * -13.51522}"/>
-      <geometry>
-        <mesh filename="${mesh_dir}/Texture.261.dae" scale="${model_scale * 1.00000} ${model_scale * 1.00000} ${model_scale * 1.00000}"/>
-      </geometry>
-    </visual>
-    <visual name="i01..leftArm.shoulder.full.009">
-      <material name="Material.390"/>
-      <origin rpy="0.06568 0.00000 0.00000" xyz="${model_scale * -1.46578} ${model_scale * 1.11459} ${model_scale * -13.51522}"/>
-      <geometry>
-        <mesh filename="${mesh_dir}/Texture.262.dae" scale="${model_scale * 1.00000} ${model_scale * 1.00000} ${model_scale * 1.00000}"/>
       </geometry>
     </visual>

File: description/urdf/inmoov.urdf (robot description, URDF)
Before this commit: robot r6bot, 59 links, 58 joints
Links:
- link left_shoulder_x_link: geometry visual mesh filename=meshes/dae/Texture.003.dae scale=1.00000 1.00000 1.00000; visual mesh filename=meshes/dae/Texture.254.dae scale=1.00000 1.00000 1.00000
