Commit message: feat(urdf): align hardware mapping, ros2_control xacro, and launch config
Centralize generated-artifact filenames via active.yaml generated_files keys
and consume them across launch and config. Refresh ros2_control xacro,
controllers, and hardware configs; clarify URDF position-limit clamp and
Gazebo limit behavior in docs.

File: description/robot_description/urdf/robot_description.urdf.xacro (robot description, xacro)
@@ -366,5 +366,5 @@
   </joint>
   <joint name="i01.head.rollNeck_link_joint" type="revolute">
-    <limit lower="0.00000" upper="0.00000" effort="100.00000" velocity="0.78540"/><!-- autocalibrated: 0.0 deg .. 0.0 deg (hit_lower=True, hit_upper=True) -->
+    <limit lower="-1.57080" upper="1.57080" effort="100.00000" velocity="0.78540"/><!-- hand-set: autocal sweep was degenerate (0 .. 0 deg) -->
     <dynamics damping="0.7" friction="0.5"/>
     <origin rpy="-0.00000 0.00000 -0.00000" xyz="${model_scale * 0.00000} ${model_scale * -0.00000} ${model_scale * 0.00435}"/>

File: description/ros2_control/inmoov_ros2_control.xacro (robot description, xacro)
@@ -10,9 +10,9 @@
           </xacro:if>
           <xacro:unless value="$(arg use_gazebo_sim)">
+            <plugin>lucy_ros2_control/LucySystemHardware</plugin>
             <xacro:if value="$(arg use_mock_hardware)">
-              <plugin>mock_components/GenericSystem</plugin>
+              <param name="publish_actuators">false</param>
             </xacro:if>
             <xacro:unless value="$(arg use_mock_hardware)">
-              <plugin>lucy_ros2_control/LucySystemHardware</plugin>
               <param name="publisher_topic">actuators/left_arm</param>
               <param name="node_name">lucy_hardware_interface_left_arm</param>
@@ -23,11 +23,14 @@
           <param name="virtual_pin">0</param>
           <param name="servo_type">270</param>
-          <param name="offset_deg">0</param>
-          <param name="direction">1</param>
-          <param name="scale">1</param>
-          <param name="servo_min_deg">0</param>
-          <param name="servo_max_deg">270</param>
-          <param name="servo_default_deg">135</param>
-          <command_interface name="position" />
+          <param name="offset_deg">90</param>
+          <param name="direction">1</param>
+          <param name="scale">1</param>
+          <param name="servo_min_deg">0</param>
+          <param name="servo_max_deg">180</param>
+          <param name="servo_default_deg">90</param>
+          <command_interface name="position">
+            <param name="min">-0.9163</param>
+            <param name="max">0.47124</param>
+          </command_interface>
           <state_interface name="position" />
       </joint>
@@ -39,7 +42,10 @@
           <param name="scale">1</param>
           <param name="servo_min_deg">0</param>
-          <param name="servo_max_deg">270</param>
-          <param name="servo_default_deg">135</param>
-          <command_interface name="position" />
+          <param name="servo_max_deg">180</param>
+          <param name="servo_default_deg">0</param>
+          <command_interface name="position">
+            <param name="min">-1.5708</param>
+            <param name="max">2.35619</param>
+          </command_interface>
           <state_interface name="position" />
       </joint>
@@ -51,7 +57,10 @@
           <param name="scale">1</param>
           <param name="servo_min_deg">0</param>
-          <param name="servo_max_deg">270</param>
-          <param name="servo_default_deg">90</param>
-          <command_interface name="position" />
+          <param name="servo_max_deg">180</param>
+          <param name="servo_default_deg">0</param>
+          <command_interface name="position">
+            <param name="min">0.0</param>
+            <param name="max">1.5708</param>
+          </command_interface>
           <state_interface name="position" />
       </joint>
@@ -59,11 +68,14 @@
           <param name="virtual_pin">3</param>
           <param name="servo_type">300</param>
-          <param name="offset_deg">0</param>
-          <param name="direction">1</param>
-          <param name="scale">1</param>
-          <param name="servo_min_deg">0</param>
-          <param name="servo_max_deg">150</param>
-          <param name="servo_default_deg">50</param>
-          <command_interface name="position" />
+          <param name="offset_deg">150</param>
+          <param name="direction">1</param>
+          <param name="scale">1</param>
+          <param name="servo_min_deg">0</param>
+          <param name="servo_max_deg">300</param>
+          <param name="servo_default_deg">150</param>
+          <command_interface name="position">
+            <param name="min">-1.5708</param>
+            <param name="max">1.5708</param>
+          </command_interface>
           <state_interface name="position" />
       </joint>
@@ -75,7 +87,10 @@
           <param name="scale">1</param>
           <param name="servo_min_deg">0</param>
-          <param name="servo_max_deg">150</param>
-          <param name="servo_default_deg">50</param>
-          <command_interface name="position" />
+          <param name="servo_max_deg">180</param>
+          <param name="servo_default_deg">0</param>
+          <command_interface name="position">
+            <param name="min">0.0</param>
+            <param name="max">1.5708</param>
+          </command_interface>
           <state_interface name="position" />
       </joint>
@@ -87,7 +102,10 @@
           <param name="scale">1</param>
           <param name="servo_min_deg">0</param>
-          <param name="servo_max_deg">150</param>
-          <param name="servo_default_deg">50</param>
-          <command_interface name="position" />
+          <param name="servo_max_deg">180</param>
+          <param name="servo_default_deg">0</param>
+          <command_interface name="position">
+            <param name="min">0.0</param>
+            <param name="max">1.5708</param>
+          </command_interface>
           <state_interface name="position" />
       </joint>
@@ -99,7 +117,10 @@
           <param name="scale">1</param>
           <param name="servo_min_deg">0</param>
-          <param name="servo_max_deg">150</param>
-          <param name="servo_default_deg">50</param>
-          <command_interface name="position" />
+          <param name="servo_max_deg">180</param>
+          <param name="servo_default_deg">0</param>
+          <command_interface name="position">
+            <param name="min">0.0</param>
+            <param name="max">1.5708</param>
+          </command_interface>
           <state_interface name="position" />
       </joint>
@@ -111,7 +132,10 @@
           <param name="scale">1</param>
           <param name="servo_min_deg">0</param>
-          <param name="servo_max_deg">150</param>
-          <param name="servo_default_deg">50</param>
-          <command_interface name="position" />
+          <param name="servo_max_deg">180</param>
+          <param name="servo_default_deg">0</param>
+          <command_interface name="position">
+            <param name="min">0.0</param>
+            <param name="max">1.5708</param>
+          </command_interface>
           <state_interface name="position" />
       </joint>
@@ -121,9 +145,12 @@
           <param name="offset_deg">0</param>
           <param name="direction">1</param>
-          <param name="scale">1</param>
-          <param name="servo_min_deg">0</param>
-          <param name="servo_max_deg">150</param>
-          <param name="servo_default_deg">50</param>
-          <command_interface name="position" />
+          <param name="scale">0.25</param>
+          <param name="servo_min_deg">0</param>
+          <param name="servo_max_deg">180</param>
+          <param name="servo_default_deg">0</param>
+          <command_interface name="position">
+            <param name="min">0.0</param>
+            <param name="max">1.5708</param>
+          </command_interface>
           <state_interface name="position" />
       </joint>
@@ -135,9 +162,9 @@
           </xacro:if>
           <xacro:unless value="$(arg use_gazebo_sim)">
+            <plugin>lucy_ros2_control/LucySystemHardware</plugin>
             <xacro:if value="$(arg use_mock_hardware)">
-              <plugin>mock_components/GenericSystem</plugin>
+              <param name="publish_actuators">false</param>
             </xacro:if>
             <xacro:unless value="$(arg use_mock_hardware)">
-              <plugin>lucy_ros2_control/LucySystemHardware</plugin>
               <param name="publisher_topic">actuators/right_arm</param>
               <param name="node_name">lucy_hardware_interface_right_arm</param>
@@ -148,11 +175,14 @@
           <param name="virtual_pin">0</param>
           <param name="servo_type">270</param>
-          <param name="offset_deg">0</param>
-          <param name="direction">1</param>
-          <param name="scale">1</param>
-          <param name="servo_min_deg">155</param>
-          <param name="servo_max_deg">165</param>
-          <param name="servo_default_deg">160</param>
-          <command_interface name="position" />
+          <param name="offset_deg">90</param>
+          <param name="direction">-1</param>
+          <param name="scale">1</param>
+          <param name="servo_min_deg">0</param>
+          <param name="servo_max_deg">180</param>
+          <param name="servo_default_deg">90</param>
+          <command_interface name="position">
+            <param name="min">-0.42761</param>
+            <param name="max">0.83776</param>
+          </command_interface>
           <state_interface name="position" />
       </joint>
@@ -163,8 +193,11 @@
           <param name="direction">1</param>
           <param name="scale">1</param>
-          <param name="servo_min_deg">140</param>
-          <param name="servo_max_deg">180</param>
-          <param name="servo_default_deg">180</param>
-          <command_interface name="position" />
+          <param name="servo_min_deg">0</param>
+          <param name="servo_max_deg">180</param>
+          <param name="servo_default_deg">0</param>
+          <command_interface name="position">
+            <param name="min">-1.5708</param>
+            <param name="max">2.35619</param>
+          </command_interface>
           <state_interface name="position" />
       </joint>
@@ -175,8 +208,11 @@
           <param name="direction">1</param>
           <param name="scale">1</param>
-          <param name="servo_min_deg">100</param>
-          <param name="servo_max_deg">110</param>
-          <param name="servo_default_deg">100</param>
-          <command_interface name="position" />
+          <param name="servo_min_deg">0</param>
+          <param name="servo_max_deg">180</param>
+          <param name="servo_default_deg">0</param>
+          <command_interface name="position">
+            <param name="min">0.0</param>
+            <param name="max">1.5708</param>
+          </command_interface>
           <state_interface name="position" />
       </joint>
@@ -184,11 +220,14 @@
           <param name="virtual_pin">3</param>
           <param name="servo_type">300</param>
-          <param name="offset_deg">0</param>
-          <param name="direction">1</param>
-          <param name="scale">1</param>
-          <param name="servo_min_deg">0</param>
-          <param name="servo_max_deg">230</param>
+          <param name="offset_deg">150</param>
+          <param name="direction">-1</param>
+          <param name="scale">1</param>
+          <param name="servo_min_deg">0</param>
+          <param name="servo_max_deg">300</param>
           <param name="servo_default_deg">150</param>
-          <command_interface name="position" />
+          <command_interface name="position">
+            <param name="min">-1.5708</param>
+            <param name="max">1.5708</param>
+          </command_interface>
           <state_interface name="position" />
       </joint>
@@ -199,8 +238,11 @@
           <param name="direction">1</param>
           <param name="scale">1</param>
-          <param name="servo_min_deg">36</param>
-          <param name="servo_max_deg">150</param>
-          <param name="servo_default_deg">36</param>
-          <command_interface name="position" />
+          <param name="servo_min_deg">0</param>
+          <param name="servo_max_deg">180</param>
+          <param name="servo_default_deg">0</param>
+          <command_interface name="position">
+            <param name="min">0.0</param>
+            <param name="max">1.5708</param>
+          </command_interface>
           <state_interface name="position" />
       </joint>
@@ -211,8 +253,11 @@
           <param name="direction">1</param>
           <param name="scale">1</param>
-          <param name="servo_min_deg">16</param>
-          <param name="servo_max_deg">150</param>
-          <param name="servo_default_deg">16</param>
-          <command_interface name="position" />
+          <param name="servo_min_deg">0</param>
+          <param name="servo_max_deg">180</param>
+          <param name="servo_default_deg">0</param>
+          <command_interface name="position">
+            <param name="min">0.0</param>
+            <param name="max">1.5708</param>
+          </command_interface>
           <state_interface name="position" />
       </joint>
@@ -223,8 +268,11 @@
           <param name="direction">1</param>
           <param name="scale">1</param>
-          <param name="servo_min_deg">21</param>
-          <param name="servo_max_deg">150</param>
-          <param name="servo_default_deg">21</param>
-          <command_interface name="position" />
+          <param name="servo_min_deg">0</param>
+          <param name="servo_max_deg">180</param>
+          <param name="servo_default_deg">0</param>
+          <command_interface name="position">
+            <param name="min">0.0</param>
+            <param name="max">1.5708</param>
+          </command_interface>
           <state_interface name="position" />
       </joint>
@@ -235,8 +283,11 @@
           <param name="direction">1</param>
           <param name="scale">1</param>
-          <param name="servo_min_deg">33</param>
-          <param name="servo_max_deg">150</param>
-          <param name="servo_default_deg">33</param>
-          <command_interface name="position" />
+          <param name="servo_min_deg">0</param>
+          <param name="servo_max_deg">180</param>
+          <param name="servo_default_deg">0</param>
+          <command_interface name="position">
+            <param name="min">0.0</param>
+            <param name="max">1.5708</param>
+          </command_interface>
           <state_interface name="position" />
       </joint>
@@ -247,8 +298,11 @@
           <param name="direction">1</param>
           <param name="scale">1</param>
-          <param name="servo_min_deg">30</param>
-          <param name="servo_max_deg">150</param>
-          <param name="servo_default_deg">30</param>
-          <command_interface name="position" />
+          <param name="servo_min_deg">0</param>
+          <param name="servo_max_deg">180</param>
+          <param name="servo_default_deg">0</param>
+          <command_interface name="position">
+            <param name="min">0.0</param>
+            <param name="max">1.5708</param>
+          </command_interface>
           <state_interface name="position" />
       </joint>
@@ -260,9 +314,9 @@
           </xacro:if>
           <xacro:unless value="$(arg use_gazebo_sim)">
+            <plugin>lucy_ros2_control/LucySystemHardware</plugin>
             <xacro:if value="$(arg use_mock_hardware)">
-              <plugin>mock_components/GenericSystem</plugin>
+              <param name="publish_actuators">false</param>
             </xacro:if>
             <xacro:unless value="$(arg use_mock_hardware)">
-              <plugin>lucy_ros2_control/LucySystemHardware</plugin>
               <param name="publisher_topic">actuators/torso</param>
               <param name="node_name">lucy_hardware_interface_torso_head</param>
@@ -277,7 +331,10 @@
           <param name="scale">1</param>
           <param name="servo_min_deg">0</param>
-          <param name="servo_max_deg">270</param>
-          <param name="servo_default_deg">0</param>
-          <command_interface name="position" />
+          <param name="servo_max_deg">180</param>
+          <param name="servo_default_deg">0</param>
+          <command_interface name="position">
+            <param name="min">0.0</param>
+            <param name="max">1.5708</param>
+          </command_interface>
           <state_interface name="position" />
       </joint>
@@ -289,31 +346,160 @@
           <param name="scale">1</param>
           <param name="servo_min_deg">0</param>
-          <param name="servo_max_deg">270</param>
-          <param name="servo_default_deg">0</param>
-          <command_interface name="position" />
+          <param name="servo_max_deg">180</param>
+          <param name="servo_default_deg">0</param>
+          <command_interface name="position">
+            <param name="min">0.0</param>
+            <param name="max">1.5708</param>
+          </command_interface>
           <state_interface name="position" />
       </joint>
       <joint name="i01.torso.midStom_link_joint">
           <param name="virtual_pin">2</param>
-          <param name="servo_type">180</param>
-          <param name="offset_deg">90</param>
-          <param name="direction">1</param>
-          <param name="scale">1</param>
-          <param name="servo_min_deg">0</param>
-          <param name="servo_max_deg">180</param>
-          <param name="servo_default_deg">90</param>
-          <command_interface name="position" />
+          <param name="servo_type">270</param>
+          <param name="offset_deg">135</param>
+          <param name="direction">1</param>
+          <param name="scale">1</param>
+          <param name="servo_min_deg">0</param>
+          <param name="servo_max_deg">270</param>
+          <param name="servo_default_deg">135</param>
+          <command_interface name="position">
+            <param name="min">-0.50615</param>
+            <param name="max">0.50615</param>
+          </command_interface>
           <state_interface name="position" />
       </joint>
       <joint name="i01.torso.topStom_link_joint">
           <param name="virtual_pin">3</param>
+          <param name="servo_type">270</param>
+          <param name="offset_deg">90</param>
+          <param name="direction">1</param>
+          <param name="scale">1</param>
+          <param name="servo_min_deg">0</param>
+          <param name="servo_max_deg">180</param>
+          <param name="servo_default_deg">90</param>
+          <command_interface name="position">
+            <param name="min">-0.12217</param>
+            <param name="max">0.12217</param>
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
File: description/urdf/inmoov.urdf.xacro (robot description, xacro)
@@ -6,4 +6,7 @@
   <xacro:arg name="use_mock_hardware" default="false"/>
   <xacro:arg name="controller_config" default=""/>
+  <!-- Generated ros2_control xacro basename (see generated_files in the hardware
+       mapping YAML). Directory is fixed at ../ros2_control/. -->
+  <xacro:arg name="ros2_control_file" default="inmoov_ros2_control.xacro"/>
   <xacro:property name="mesh_dir" value="file://$(arg base_path)/robot_description/meshes/dae"/>
   <xacro:property name="use_gazebo_sim" value="$(arg use_gazebo_sim)"/>
@@ -12,6 +15,7 @@
   <!-- Import inmoov physical description (urdf) macro (uses use_gazebo_sim for heavy stand in sim) -->
   <xacro:include filename="../robot_description/urdf/robot_description.urdf.xacro"/>
-  <!-- Import inmoov ros2_control description (use_gazebo_sim switches to gz_ros2_control in Gazebo launch) -->
-  <xacro:include filename="../ros2_control/inmoov_ros2_control.xacro" />
+  <!-- Import inmoov ros2_control description (use_gazebo_sim switches to gz_ros2_control in Gazebo launch).
+       Filename comes from the generated_files config so the generator, pipeline and launches agree. -->
+  <xacro:include filename="../ros2_control/$(arg ros2_control_file)" />
   <!-- Gazebo-only bits, gated on use_gazebo_sim:=true:
          - gazebo/inmoov_gazebo_physics.xacro    physics + surface tuning
