Commit message: feat(fork): update inmoov_urdf from thais_urdf and widen torso/head joint limits
Signed-off-by: Charles Madjeri <80175305+charlesmadjeri@users.noreply.github.com>

File: description/robot_description/urdf/robot_description.urdf.xacro (robot description, xacro)
@@ -102,5 +102,5 @@
   </joint>
   <joint name="i01.torso.midStom_link_joint" type="revolute">
-    <limit lower="-0.50615" upper="0.50615" effort="100.00000" velocity="0.78540"/><!-- autocalibrated: -29.0 deg .. 29.0 deg (hit_lower=False, hit_upper=False) -->
+    <limit lower="-1.57080" upper="1.57080" effort="100.00000" velocity="0.78540"/><!-- hand-set: -90.0 deg .. 90.0 deg -->
     <dynamics damping="0.7" friction="0.5"/>
     <origin rpy="0.00000 0.06589 1.57080" xyz="${model_scale * -0.00213} ${model_scale * 0.05565} ${model_scale * 1.13807}"/>
@@ -190,5 +190,5 @@
   </joint>
   <joint name="i01.torso.topStom_link_joint" type="revolute">
-    <limit lower="-0.12217" upper="0.12217" effort="100.00000" velocity="0.78540"/><!-- autocalibrated: -7.0 deg .. 7.0 deg (hit_lower=False, hit_upper=False) -->
+    <limit lower="-0.26180" upper="0.26180" effort="100.00000" velocity="0.78540"/><!-- hand-set: -15.0 deg .. 15.0 deg -->
     <dynamics damping="0.7" friction="0.5"/>
     <origin rpy="0.00000 0.00000 -1.57080" xyz="${model_scale * -0.06317} ${model_scale * 0.00033} ${model_scale * 1.01916}"/>
@@ -278,5 +278,5 @@
   </joint>
   <joint name="i01.head.neck.001_link_joint" type="revolute">
-    <limit lower="-0.34907" upper="0.00000" effort="100.00000" velocity="0.78540"/><!-- autocalibrated: -20.0 deg .. 0.0 deg (hit_lower=False, hit_upper=False) -->
+    <limit lower="-0.34907" upper="0.34907" effort="100.00000" velocity="0.78540"/><!-- hand-set: -20.0 deg .. 20.0 deg -->
     <dynamics damping="0.7" friction="0.5"/>
     <origin rpy="0.06589 -0.00000 -0.00000" xyz="${model_scale * 0.00390} ${model_scale * 0.29817} ${model_scale * 4.29073}"/>
@@ -366,5 +366,5 @@
   </joint>
   <joint name="i01.head.rollNeck_link_joint" type="revolute">
-    <limit lower="-1.57080" upper="1.57080" effort="100.00000" velocity="0.78540"/><!-- hand-set: autocal sweep was degenerate (0 .. 0 deg) -->
+    <limit lower="-0.34907" upper="0.34907" effort="100.00000" velocity="0.78540"/><!-- hand-set: -20.0 deg .. 20.0 deg -->
     <dynamics damping="0.7" friction="0.5"/>
     <origin rpy="-0.00000 0.00000 -0.00000" xyz="${model_scale * 0.00000} ${model_scale * -0.00000} ${model_scale * 0.00435}"/>
@@ -438,5 +438,5 @@
   </joint>
   <joint name="i01.head.rothead_link_joint" type="revolute">
-    <limit lower="-0.08727" upper="0.04363" effort="100.00000" velocity="0.78540"/><!-- autocalibrated: -5.0 deg .. 2.5 deg (hit_lower=False, hit_upper=False) -->
+    <limit lower="-1.57080" upper="1.57080" effort="100.00000" velocity="0.78540"/><!-- hand-set: -90.0 deg .. 90.0 deg -->
     <dynamics damping="0.7" friction="0.5"/>
     <origin rpy="0.00000 -0.00000 1.57080" xyz="${model_scale * 0.00246} ${model_scale * 0.01503} ${model_scale * 0.24911}"/>

File: description/ros2_control/inmoov_ros2_control.xacro (robot description, xacro)
@@ -364,6 +364,6 @@
           <param name="servo_default_deg">135</param>
           <command_interface name="position">
-            <param name="min">-0.50615</param>
-            <param name="max">0.50615</param>
+            <param name="min">-1.5708</param>
+            <param name="max">1.5708</param>
           </command_interface>
           <state_interface name="position" />
@@ -379,6 +379,6 @@
           <param name="servo_default_deg">90</param>
           <command_interface name="position">
-            <param name="min">-0.12217</param>
-            <param name="max">0.12217</param>
+            <param name="min">-0.2618</param>
+            <param name="max">0.2618</param>
           </command_interface>
           <state_interface name="position" />
@@ -394,6 +394,6 @@
           <param name="servo_default_deg">90</param>
           <command_interface name="position">
-            <param name="min">-0.08727</param>
-            <param name="max">0.04363</param>
+            <param name="min">-1.5708</param>
+            <param name="max">1.5708</param>
           </command_interface>
           <state_interface name="position" />
@@ -409,6 +409,6 @@
           <param name="servo_default_deg">90</param>
           <command_interface name="position">
-            <param name="min">-1.5708</param>
-            <param name="max">1.5708</param>
+            <param name="min">-0.34907</param>
+            <param name="max">0.34907</param>
           </command_interface>
           <state_interface name="position" />
@@ -425,5 +425,5 @@
           <command_interface name="position">
             <param name="min">-0.34907</param>
-            <param name="max">0.0</param>
+            <param name="max">0.34907</param>
           </command_interface>
           <state_interface name="position" />
@@ -432,10 +432,10 @@
           <param name="virtual_pin">7</param>
           <param name="servo_type">300</param>
-          <param name="offset_deg">90</param>
-          <param name="direction">1</param>
-          <param name="scale">1</param>
-          <param name="servo_min_deg">0</param>
-          <param name="servo_max_deg">180</param>
-          <param name="servo_default_deg">90</param>
+          <param name="offset_deg">0</param>
+          <param name="direction">1</param>
+          <param name="scale">1</param>
+          <param name="servo_min_deg">0</param>
+          <param name="servo_max_deg">180</param>
+          <param name="servo_default_deg">0</param>
           <command_interface name="position">
             <param name="min">0.0</param>
