Commit message: fix(color): add unique white color
Signed-off-by: m-brl <103381146+m-brl@users.noreply.github.com>

File: description/robot_description/urdf/robot_description.urdf.xacro (robot description, xacro)
@@ -531,5 +531,5 @@
     </collision>
     <visual name="i01.head.eyeRight.full">
-      <material name="Material.038"/>
+      <material name="Material.White"/>
       <origin rpy="-0.00000 0.00000 0.00000" xyz="${model_scale * 0.29460} ${model_scale * 0.89123} ${model_scale * -16.02297}"/>
       <geometry>
@@ -559,5 +559,5 @@
     </collision>
     <visual name="i01.head.mouth">
-      <material name="Material.046"/>
+      <material name="Material.White"/>
       <origin rpy="0.00000 0.00000 -0.00000" xyz="${model_scale * 0.00732} ${model_scale * 0.15065} ${model_scale * -15.97164}"/>
       <geometry>
@@ -566,5 +566,5 @@
     </visual>
     <visual name="i01.head.mouth.001">
-      <material name="Material.046"/>
+      <material name="Material.White"/>
       <origin rpy="0.00000 0.00000 -0.00000" xyz="${model_scale * 0.00732} ${model_scale * 0.15065} ${model_scale * -15.97164}"/>
       <geometry>
@@ -573,5 +573,5 @@
     </visual>
     <visual name="i01.head.mouth.002">
-      <material name="Material.046"/>
+      <material name="Material.White"/>
       <origin rpy="0.00000 0.00000 -0.00000" xyz="${model_scale * 0.00732} ${model_scale * 0.15065} ${model_scale * -15.97164}"/>
       <geometry>
@@ -625,5 +625,5 @@
     </collision>
     <visual name="i01.leftArm.omoplate.full">
-      <material name="Material.254"/>
+      <material name="Material.White"/>
       <origin rpy="0.06568 0.00000 0.00000" xyz="${model_scale * -1.35226} ${model_scale * 1.11649} ${model_scale * -13.89027}"/>
       <geometry>
@@ -632,5 +632,5 @@
     </visual>
     <visual name="i01.leftArm.omoplate.full.001">
-      <material name="Material.254"/>
+      <material name="Material.White"/>
       <origin rpy="0.06568 0.00000 0.00000" xyz="${model_scale * -1.35226} ${model_scale * 1.11649} ${model_scale * -13.89027}"/>
       <geometry>
@@ -639,5 +639,5 @@
     </visual>
     <visual name="i01.leftArm.omoplate.full.002">
-      <material name="Material.254"/>
+      <material name="Material.White"/>
       <origin rpy="0.06568 0.00000 0.00000" xyz="${model_scale * -1.35226} ${model_scale * 1.11649} ${model_scale * -13.89027}"/>
       <geometry>
@@ -646,5 +646,5 @@
     </visual>
     <visual name="i01.leftArm.omoplate.full.003">
-      <material name="Material.254"/>
+      <material name="Material.White"/>
       <origin rpy="0.06568 0.00000 0.00000" xyz="${model_scale * -1.35226} ${model_scale * 1.11649} ${model_scale * -13.89027}"/>
       <geometry>
@@ -653,5 +653,5 @@
     </visual>
     <visual name="i01.leftArm.omoplate.full.004">
-      <material name="Material.254"/>
+      <material name="Material.White"/>
       <origin rpy="0.06568 0.00000 0.00000" xyz="${model_scale * -1.35226} ${model_scale * 1.11649} ${model_scale * -13.89027}"/>
       <geometry>
@@ -660,5 +660,5 @@
     </visual>
     <visual name="i01.leftArm.omoplate.full.005">
-      <material name="Material.254"/>
+      <material name="Material.White"/>
       <origin rpy="0.06568 0.00000 0.00000" xyz="${model_scale * -1.35226} ${model_scale * 1.11649} ${model_scale * -13.89027}"/>
       <geometry>
@@ -667,5 +667,5 @@
     </visual>
     <visual name="i01.leftArm.omoplate.full.006">
-      <material name="Material.254"/>
+      <material name="Material.White"/>
       <origin rpy="0.06568 0.00000 0.00000" xyz="${model_scale * -1.35226} ${model_scale * 1.11649} ${model_scale * -13.89027}"/>
       <geometry>
@@ -761,5 +761,5 @@
     </collision>
     <visual name="i01..leftArm.shoulder.full">
-      <material name="Material.239"/>
+      <material name="Material.White"/>
       <origin rpy="0.06568 0.00000 0.00000" xyz="${model_scale * -1.46578} ${model_scale * 1.11459} ${model_scale * -13.51522}"/>
       <geometry>
@@ -768,5 +768,5 @@
     </visual>
     <visual name="i01..leftArm.shoulder.full.001">
-      <material name="Material.390"/>
+      <material name="Material.White"/>
       <origin rpy="0.06568 0.00000 0.00000" xyz="${model_scale * -1.46578} ${model_scale * 1.11459} ${model_scale * -13.51522}"/>
       <geometry>
@@ -775,5 +775,5 @@
     </visual>
     <visual name="i01..leftArm.shoulder.full.002">
-      <material name="Material.390"/>
+      <material name="Material.White"/>
       <origin rpy="0.06568 0.00000 0.00000" xyz="${model_scale * -1.46578} ${model_scale * 1.11459} ${model_scale * -13.51522}"/>
       <geometry>
@@ -782,5 +782,5 @@
     </visual>
     <visual name="i01..leftArm.shoulder.full.003">
-      <material name="Material.390"/>
+      <material name="Material.White"/>
       <origin rpy="0.06568 0.00000 0.00000" xyz="${model_scale * -1.46578} ${model_scale * 1.11459} ${model_scale * -13.51522}"/>
       <geometry>
@@ -789,5 +789,5 @@
     </visual>
     <visual name="i01..leftArm.shoulder.full.004">
-      <material name="Material.390"/>
+      <material name="Material.White"/>
       <origin rpy="0.06568 0.00000 0.00000" xyz="${model_scale * -1.46578} ${model_scale * 1.11459} ${model_scale * -13.51522}"/>
       <geometry>
@@ -796,5 +796,5 @@
     </visual>
     <visual name="i01..leftArm.shoulder.full.005">
-      <material name="Material.390"/>
+      <material name="Material.White"/>
       <origin rpy="0.06568 0.00000 0.00000" xyz="${model_scale * -1.46578} ${model_scale * 1.11459} ${model_scale * -13.51522}"/>
       <geometry>
@@ -803,5 +803,5 @@
     </visual>
     <visual name="i01..leftArm.shoulder.full.006">
-      <material name="Material.390"/>
+      <material name="Material.White"/>
       <origin rpy="0.06568 0.00000 0.00000" xyz="${model_scale * -1.46578} ${model_scale * 1.11459} ${model_scale * -13.51522}"/>
       <geometry>
@@ -810,5 +810,5 @@
     </visual>
     <visual name="i01..leftArm.shoulder.full.007">
-      <material name="Material.390"/>
+      <material name="Material.White"/>
       <origin rpy="0.06568 0.00000 0.00000" xyz="${model_scale * -1.46578} ${model_scale * 1.11459} ${model_scale * -13.51522}"/>
       <geometry>
@@ -817,5 +817,5 @@
     </visual>
     <visual name="i01..leftArm.shoulder.full.010">
-      <material name="Material.390"/>
+      <material name="Material.White"/>
       <origin rpy="0.06568 0.00000 0.00000" xyz="${model_scale * -1.46578} ${model_scale * 1.11459} ${model_scale * -13.51522}"/>
       <geometry>
@@ -824,5 +824,5 @@
     </visual>
     <visual name="i01..leftArm.shoulder.full.011">
-      <material name="Material.390"/>
+      <material name="Material.White"/>
       <origin rpy="0.06568 0.00000 0.00000" xyz="${model_scale * -1.46578} ${model_scale * 1.11459} ${model_scale * -13.51522}"/>
       <geometry>
@@ -831,5 +831,5 @@
     </visual>
     <visual name="i01..leftArm.shoulder.full.014">
-      <material name="Material.390"/>
+      <material name="Material.White"/>
       <origin rpy="0.06568 0.00000 0.00000" xyz="${model_scale * -1.46578} ${model_scale * 1.11459} ${model_scale * -13.51522}"/>
       <geometry>
@@ -838,5 +838,5 @@
     </visual>
     <visual name="i01..leftArm.shoulder.full.015">
-      <material name="Material.390"/>
+      <material name="Material.White"/>
       <origin rpy="0.06568 0.00000 0.00000" xyz="${model_scale * -1.46578} ${model_scale * 1.11459} ${model_scale * -13.51522}"/>
       <geometry>
@@ -845,5 +845,5 @@
     </visual>
     <visual name="i01..leftArm.shoulder.full.016">
-      <material name="Material.390"/>
+      <material name="Material.White"/>
       <origin rpy="0.06568 0.00000 0.00000" xyz="${model_scale * -1.46578} ${model_scale * 1.11459} ${model_scale * -13.51522}"/>
       <geometry>
@@ -852,5 +852,5 @@
     </visual>
     <visual name="i01..leftArm.shoulder.full.017">
-      <material name="Material.390"/>
+      <material name="Material.White"/>
       <origin rpy="0.06568 0.00000 0.00000" xyz="${model_scale * -1.46578} ${model_scale * 1.11459} ${model_scale * -13.51522}"/>
       <geometry>
@@ -988,5 +988,5 @@
     </collision>
     <visual name="i01.leftArm.rotate.full">
-      <material name="[0131_Silver].001"/>
+      <material name="Material.White"/>
       <origin rpy="-0.00792 -0.00000 -0.00000" xyz="${model_scale * -2.08983} ${model_scale * 1.12391} ${model_scale * -12.92101}"/>
       <geometry>
@@ -995,5 +995,5 @@
     </visual>
     <visual name="i01.leftArm.rotate.full.001">
-      <material name="[0131_Silver].001"/>
+      <material name="Material.White"/>
       <origin rpy="-0.00792 -0.00000 -0.00000" xyz="${model_scale * -2.08983} ${model_scale * 1.12391} ${model_scale * -12.92101}"/>
       <geometry>
@@ -1002,5 +1002,5 @@
     </visual>
     <visual name="i01.leftArm.rotate.full.002">
-      <material name="[0131_Silver].001"/>
+      <material name="Material.White"/>
       <origin rpy="-0.00792 -0.00000 -0.00000" xyz="${model_scale * -2.08983} ${model_scale * 1.12391} ${model_scale * -12.92101}"/>
       <geometry>
@@ -1009,5 +1009,5 @@
     </visual>
     <visual name="i01.leftArm.rotate.full.003">
-      <material name="[0131_Silver].001"/>
+      <material name="Material.White"/>
       <origin rpy="-0.00792 -0.00000 -0.00000" xyz="${model_scale * -2.08983} ${model_scale * 1.12391} ${model_scale * -12.92101}"/>
       <geometry>
@@ -1016,5 +1016,5 @@
     </visual>
     <visual name="i01.leftArm.rotate.full.004">
-      <material name="[0131_Silver].001"/>
+      <material name="Material.White"/>
       <origin rpy="-0.00792 -0.00000 -0.00000" xyz="${model_scale * -2.08983} ${model_scale * 1.12391} ${model_scale * -12.92101}"/>
       <geometry>
@@ -1023,5 +1023,5 @@
     </visual>
     <visual name="i01.leftArm.rotate.full.005">
-      <material name="[0131_Silver].001"/>
+      <material name="Material.White"/>
       <origin rpy="-0.00792 -0.00000 -0.00000" xyz="${model_scale * -2.08983} ${model_scale * 1.12391} ${model_scale * -12.92101}"/>
       <geometry>
@@ -1030,5 +1030,5 @@
     </visual>
     <visual name="i01.leftArm.rotate.full.006">
-      <material name="[0131_Silver].001"/>
+      <material name="Material.White"/>
       <origin rpy="-0.00792 -0.00000 -0.00000" xyz="${model_scale * -2.08983} ${model_scale * 1.12391} ${model_scale * -12.92101}"/>
       <geometry>
@@ -1037,5 +1037,5 @@
     </visual>
     <visual name="i01.leftArm.rotate.full.007">
-      <material name="[0131_Silver].001"/>
+      <material name="Material.White"/>
       <origin rpy="-0.00792 -0.00000 -0.00000" xyz="${model_scale * -2.08983} ${model_scale * 1.12391} ${model_scale * -12.92101}"/>
       <geometry>
@@ -1044,5 +1044,5 @@
     </visual>
     <visual name="i01.leftArm.rotate.full.008">
-      <material name="[0131_Silver].001"/>
+      <material name="Material.White"/>
       <origin rpy="-0.00792 -0.00000 -0.00000" xyz="${model_scale * -2.08983} ${model_scale * 1.12391} ${model_scale * -12.92101}"/>
       <geometry>
@@ -1051,5 +1051,5 @@
     </visual>
     <visual name="i01.leftArm.rotate.full.009">
-      <material name="[0131_Silver].001"/>
+      <material name="Material.White"/>
       <origin rpy="-0.00792 -0.00000 -0.00000" xyz="${model_scale * -2.08983} ${model_scale * 1.12391} ${model_scale * -12.92101}"/>
       <geometry>
@@ -1058,5 +1058,5 @@
     </visual>
     <visual name="i01.leftArm.rotate.full.010">
-      <material name="[0131_Silver].001"/>
+      <material name="Material.White"/>
       <origin rpy="-0.00792 -0.00000 -0.00000" xyz="${model_scale * -2.08983} ${model_scale * 1.12391} ${model_scale * -12.92101}"/>
       <geometry>
@@ -1065,5 +1065,5 @@
     </visual>
     <visual name="i01.leftArm.rotate.full.011">
-      <material name="[0131_Silver].001"/>
+      <material name="Material.White"/>
       <origin rpy="-0.00792 -0.00000 -0.00000" xyz="${model_scale * -2.08983} ${model_scale * 1.12391} ${model_scale * -12.92101}"/>
       <geometry>
@@ -1072,5 +1072,5 @@
     </visual>
     <visual name="i01.leftArm.rotate.full.012">
-      <material name="[0131_Silver].001"/>
+      <material name="Material.White"/>
       <origin rpy="-0.00792 -0.00000 -0.00000" xyz="${model_scale * -2.08983} ${model_scale * 1.12391} ${model_scale * -12.92101}"/>
       <geometry>
@@ -1079,5 +1079,5 @@
     </visual>
     <visual name="i01.leftArm.rotate.full.013">
-      <material name="[0131_Silver].001"/>
+      <material name="Material.White"/>
       <origin rpy="-0.00792 -0.00000 -0.00000" xyz="${model_scale * -2.08983} ${model_scale * 1.12391} ${model_scale * -12.92101}"/>
       <geometry>
@@ -1086,5 +1086,5 @@
     </visual>
     <visual name="i01.leftArm.rotate.full.014">
-      <material name="[0131_Silver].001"/>
+      <material name="Material.White"/>
       <origin rpy="-0.00792 -0.00000 -0.00000" xyz="${model_scale * -2.08983} ${model_scale * 1.12391} ${model_scale * -12.92101}"/>
       <geometry>
@@ -1093,5 +1093,5 @@
     </visual>
     <visual name="i01.leftArm.rotate.full.015">
-      <material name="[0131_Silver].001"/>
+      <material name="Material.White"/>
       <origin rpy="-0.00792 -0.00000 -0.00000" xyz="${model_scale * -2.08983} ${model_scale * 1.12391} ${model_scale * -12.92101}"/>
       <geometry>
@@ -1100,5 +1100,5 @@
     </visual>
     <visual name="i01.leftArm.rotate.full.016">
-      <material name="[0131_Silver].001"/>
+      <material name="Material.White"/>
       <origin rpy="-0.00792 -0.00000 -0.00000" xyz="${model_scale * -2.08983} ${model_scale * 1.12391} ${model_scale * -12.92101}"/>
       <geometry>
@@ -1107,5 +1107,5 @@
     </visual>
     <visual name="i01.leftArm.rotate.full.017">
-      <material name="[0131_Silver].001"/>
+      <material name="Material.White"/>
       <origin rpy="-0.00792 -0.00000 -0.00000" xyz="${model_scale * -2.08983} ${model_scale * 1.12391} ${model_scale * -12.92101}"/>
       <geometry>
@@ -1114,5 +1114,5 @@
     </visual>
     <visual name="i01.leftArm.rotate.full.018">
-      <material name="[0131_Silver].001"/>
+      <material name="Material.White"/>
       <origin rpy="-0.00792 -0.00000 -0.00000" xyz="${model_scale * -2.08983} ${model_scale * 1.12391} ${model_scale * -12.92101}"/>
       <geometry>
@@ -1121,5 +1121,5 @@
     </visual>
     <visual name="i01.leftArm.rotate.full.019">
-      <material name="[0131_Silver].001"/>
+      <material name="Material.White"/>
       <origin rpy="-0.00792 -0.00000 -0.00000" xyz="${model_scale * -2.08983} ${model_scale * 1.12391} ${model_scale * -12.92101}"/>
       <geometry>
@@ -1128,5 +1128,5 @@
     </visual>
     <visual name="i01.leftArm.rotate.full.020">
-      <material name="[0131_Silver].001"/>
+      <material name="Material.White"/>
       <origin rpy="-0.00792 -0.00000 -0.00000" xyz="${model_scale * -2.08983} ${model_scale * 1.12391} ${model_scale * -12.92101}"/>
       <geometry>
@@ -1216,5 +1216,5 @@
     </collision>
     <visual name="i01.left.bicep.full">
-      <material name="Material.022"/>
+      <material name="Material.White"/>
       <origin rpy="-0.00000 0.00000 0.00000" xyz="${model_scale * -2.07702} ${model_scale * 0.12073} ${model_scale * -10.83652}"/>
       <geometry>
@@ -1223,5 +1223,5 @@
     </visual>
     <visual name="i01.left.bicep.full.001">
-      <material name="Material.022"/>
+      <material name="Material.White"/>
       <origin rpy="-0.00000 0.00000 0.00000" xyz="${model_scale * -2.07702} ${model_scale * 0.12073} ${model_scale * -10.83652}"/>
       <geometry>
@@ -1230,5 +1230,5 @@
     </visual>
     <visual name="i01.left.bicep.full.002">
-      <material name="Material.022"/>
+      <material name="Material.White"/>
       <origin rpy="-0.00000 0.00000 0.00000" xyz="${model_scale * -2.07702} ${model_scale * 0.12073} ${model_scale * -10.83652}"/>
       <geometry>
@@ -1237,5 +1237,5 @@
     </visual>
     <visual name="i01.left.bicep.full.003">
-      <material name="Material.022"/>
+      <material name="Material.White"/>
       <origin rpy="-0.00000 0.00000 0.00000" xyz="${model_scale * -2.07702} ${model_scale * 0.12073} ${model_scale * -10.83652}"/>
       <geometry>
@@ -1244,5 +1244,5 @@
     </visual>
     <visual name="i01.left.bicep.full.004">
-      <material name="Material.022"/>
+      <material name="Material.White"/>
       <origin rpy="-0.00000 0.00000 0.00000" xyz="${model_scale * -2.07702} ${model_scale * 0.12073} ${model_scale * -10.83652}"/>
       <geometry>
@@ -1251,5 +1251,5 @@
     </visual>
     <visual name="i01.left.bicep.full.005">
-      <material name="Material.022"/>
+      <material name="Material.White"/>
       <origin rpy="-0.00000 0.00000 0.00000" xyz="${model_scale * -2.07702} ${model_scale * 0.12073} ${model_scale * -10.83652}"/>
       <geometry>
@@ -1258,5 +1258,5 @@
     </visual>
     <visual name="i01.left.bicep.full.006">
-      <material name="Material.022"/>
+      <material name="Material.White"/>
       <origin rpy="-0.00000 0.00000 0.00000" xyz="${model_scale * -2.07702} ${model_scale * 0.12073} ${model_scale * -10.83652}"/>
       <geometry>
@@ -1265,5 +1265,5 @@
     </visual>
     <visual name="i01.left.bicep.full.007">
-      <material name="Material.022"/>
+      <material name="Material.White"/>
       <origin rpy="-0.00000 0.00000 0.00000" xyz="${model_scale * -2.07702} ${model_scale * 0.12073} ${model_scale * -10.83652}"/>
       <geometry>
@@ -1272,5 +1272,5 @@
     </visual>
     <visual name="i01.left.bicep.full.008">
-      <material name="Material.022"/>
+      <material name="Material.White"/>
       <origin rpy="-0.00000 0.00000 0.00000" xyz="${model_scale * -2.07702} ${model_scale * 0.12073} ${model_scale * -10.83652}"/>
       <geometry>
@@ -1279,5 +1279,5 @@
     </visual>
     <visual name="i01.left.bicep.full.009">
-      <material name="Material.022"/>
+      <material name="Material.White"/>
       <origin rpy="-0.00000 0.00000 0.00000" xyz="${model_scale * -2.07702} ${model_scale * 0.12073} ${model_scale * -10.83652}"/>
       <geometry>
@@ -1286,5 +1286,5 @@
     </visual>
     <visual name="i01.left.bicep.full.010">
-      <material name="Material.022"/>
+      <material name="Material.White"/>
       <origin rpy="-0.00000 0.00000 0.00000" xyz="${model_scale * -2.07702} ${model_scale * 0.12073} ${model_scale * -10.83652}"/>
       <geometry>
@@ -1293,5 +1293,5 @@
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