Commit message: fix: mimic joints for fingers

File: description/robot_description/urdf/properties.xacro (robot description, xacro)
@@ -14,3 +14,12 @@
 <robot xmlns:xacro="http://www.ros.org/wiki/xacro">
   <xacro:property name="model_scale" value="0.1196"/>
+  <!--
+  Tendon coupling for the fingers. Each finger is driven by one servo pulling a
+  single string through all its phalanges, so the middle and distal joints are
+  <mimic> joints following the proximal joint (index/majeure/ringFinger/pinky,
+  and thumb3 following thumb). 1.0 = every phalanx curls by the same angle.
+  Lower the distal ratio if the modelled fist curls tighter than the hardware.
+  -->
+  <xacro:property name="finger_mid_ratio" value="1.0"/>
+  <xacro:property name="finger_distal_ratio" value="1.0"/>
 </robot>

File: description/robot_description/urdf/robot_description.urdf.xacro (robot description, xacro)
@@ -100,4 +100,5 @@
     <child link="i01.leftHand.index2_link"/>
     <axis xyz="-0.99994 0.00000 0.01111"/>
+    <mimic joint="i01.leftHand.index_link_joint" multiplier="${finger_mid_ratio}" offset="0.0"/><!-- tendon-coupled phalanx -->
   </joint>
   <joint name="i01.torso.midStom_link_joint" type="revolute">
@@ -116,4 +117,5 @@
     <child link="i01.leftHand.index3_link"/>
     <axis xyz="-0.99994 0.00000 0.01111"/>
+    <mimic joint="i01.leftHand.index_link_joint" multiplier="${finger_distal_ratio}" offset="0.0"/><!-- tendon-coupled phalanx -->
   </joint>
   <joint name="i01.leftHand.majeure_link_joint" type="revolute">
@@ -132,4 +134,5 @@
     <child link="i01.leftHand.majeure2_link"/>
     <axis xyz="-0.99994 0.00000 0.01111"/>
+    <mimic joint="i01.leftHand.majeure_link_joint" multiplier="${finger_mid_ratio}" offset="0.0"/><!-- tendon-coupled phalanx -->
   </joint>
   <joint name="i01.leftHand.majeure3_link_joint" type="revolute">
@@ -140,4 +143,5 @@
     <child link="i01.leftHand.majeure3_link"/>
     <axis xyz="-0.99994 0.00000 0.01111"/>
+    <mimic joint="i01.leftHand.majeure_link_joint" multiplier="${finger_distal_ratio}" offset="0.0"/><!-- tendon-coupled phalanx -->
   </joint>
   <joint name="i01.leftHand.pinky0_link_joint" type="revolute">
@@ -164,4 +168,5 @@
     <child link="i01.leftHand.pinky2_link"/>
     <axis xyz="-0.99994 0.00000 0.01111"/>
+    <mimic joint="i01.leftHand.pinky_link_joint" multiplier="${finger_mid_ratio}" offset="0.0"/><!-- tendon-coupled phalanx -->
   </joint>
   <joint name="i01.leftHand.pinky3_link_joint" type="revolute">
@@ -172,4 +177,5 @@
     <child link="i01.leftHand.pinky3_link"/>
     <axis xyz="-0.99994 0.00000 0.01111"/>
+    <mimic joint="i01.leftHand.pinky_link_joint" multiplier="${finger_distal_ratio}" offset="0.0"/><!-- tendon-coupled phalanx -->
   </joint>
   <joint name="i01.leftHand.ringfinger0_link_joint" type="revolute">
@@ -204,4 +210,5 @@
     <child link="i01.leftHand.ringfinger2_link"/>
     <axis xyz="-0.99994 0.00000 0.01111"/>
+    <mimic joint="i01.leftHand.ringFinger_link_joint" multiplier="${finger_mid_ratio}" offset="0.0"/><!-- tendon-coupled phalanx -->
   </joint>
   <joint name="i01.leftHand.ringfinger3_link_joint" type="revolute">
@@ -212,4 +219,5 @@
     <child link="i01.leftHand.ringfinger3_link"/>
     <axis xyz="-0.99994 0.00000 0.01111"/>
+    <mimic joint="i01.leftHand.ringFinger_link_joint" multiplier="${finger_distal_ratio}" offset="0.0"/><!-- tendon-coupled phalanx -->
   </joint>
   <joint name="i01.leftHand.thumb1_link_joint" type="revolute">
@@ -236,4 +244,5 @@
     <child link="i01.leftHand.thumb3_link"/>
     <axis xyz="-0.99994 0.00000 0.01111"/>
+    <mimic joint="i01.leftHand.thumb_link_joint" multiplier="${finger_distal_ratio}" offset="0.0"/><!-- tendon-coupled phalanx -->
   </joint>
   <joint name="right_shoulder_y_link_joint" type="revolute">
@@ -308,4 +317,5 @@
     <child link="i01.rightHand.index2_link"/>
     <axis xyz="-0.99994 0.00000 0.01111"/>
+    <mimic joint="i01.rightHand.index_link_joint" multiplier="${finger_mid_ratio}" offset="0.0"/><!-- tendon-coupled phalanx -->
   </joint>
   <joint name="i01.rightHand.index3_link_joint" type="revolute">
@@ -316,4 +326,5 @@
     <child link="i01.rightHand.index3_link"/>
     <axis xyz="-0.99994 0.00000 0.01111"/>
+    <mimic joint="i01.rightHand.index_link_joint" multiplier="${finger_distal_ratio}" offset="0.0"/><!-- tendon-coupled phalanx -->
   </joint>
   <joint name="i01.rightHand.majeure_link_joint" type="revolute">
@@ -332,4 +343,5 @@
     <child link="i01.rightHand.majeure2_link"/>
     <axis xyz="-0.99994 0.00000 0.01111"/>
+    <mimic joint="i01.rightHand.majeure_link_joint" multiplier="${finger_mid_ratio}" offset="0.0"/><!-- tendon-coupled phalanx -->
   </joint>
   <joint name="i01.rightHand.majeure3_link_joint" type="revolute">
@@ -340,4 +352,5 @@
     <child link="i01.rightHand.majeure3_link"/>
     <axis xyz="-0.99994 0.00000 0.01111"/>
+    <mimic joint="i01.rightHand.majeure_link_joint" multiplier="${finger_distal_ratio}" offset="0.0"/><!-- tendon-coupled phalanx -->
   </joint>
   <joint name="i01.rightHand.pinky0_link_joint" type="revolute">
@@ -364,4 +377,5 @@
     <child link="i01.rightHand.pinky2_link"/>
     <axis xyz="-0.99994 0.00000 0.01111"/>
+    <mimic joint="i01.rightHand.pinky_link_joint" multiplier="${finger_mid_ratio}" offset="0.0"/><!-- tendon-coupled phalanx -->
   </joint>
   <joint name="i01.head.rollNeck_link_joint" type="revolute">
@@ -380,4 +394,5 @@
     <child link="i01.rightHand.pinky3_link"/>
     <axis xyz="-0.99994 0.00000 0.01111"/>
+    <mimic joint="i01.rightHand.pinky_link_joint" multiplier="${finger_distal_ratio}" offset="0.0"/><!-- tendon-coupled phalanx -->
   </joint>
   <joint name="i01.rightHand.ringfinger0_link_joint" type="revolute">
@@ -404,4 +419,5 @@
     <child link="i01.rightHand.ringfinger2_link"/>
     <axis xyz="-0.99994 0.00000 0.01111"/>
+    <mimic joint="i01.rightHand.ringFinger_link_joint" multiplier="${finger_mid_ratio}" offset="0.0"/><!-- tendon-coupled phalanx -->
   </joint>
   <joint name="i01.rightHand.ringfinger3_link_joint" type="revolute">
@@ -412,4 +428,5 @@
     <child link="i01.rightHand.ringfinger3_link"/>
     <axis xyz="-0.99994 0.00000 0.01111"/>
+    <mimic joint="i01.rightHand.ringFinger_link_joint" multiplier="${finger_distal_ratio}" offset="0.0"/><!-- tendon-coupled phalanx -->
   </joint>
   <joint name="i01.rightHand.thumb1_link_joint" type="revolute">
@@ -436,4 +453,5 @@
     <child link="i01.rightHand.thumb3_link"/>
     <axis xyz="-0.99994 0.00000 0.01111"/>
+    <mimic joint="i01.rightHand.thumb_link_joint" multiplier="${finger_distal_ratio}" offset="0.0"/><!-- tendon-coupled phalanx -->
   </joint>
   <joint name="i01.head.rothead_link_joint" type="revolute">

Commit message: clean(urdf): drop the repeated mimic comments
The per-line "tendon-coupled phalanx" note repeated on all 18 mimic tags said
nothing the multiplier name did not, and the block in properties.xacro listed
joint names the URDF already spells out.

File: description/robot_description/urdf/properties.xacro (robot description, xacro)
@@ -15,9 +15,7 @@
   <xacro:property name="model_scale" value="0.1196"/>
   <!--
-  Tendon coupling for the fingers. Each finger is driven by one servo pulling a
-  single string through all its phalanges, so the middle and distal joints are
-  <mimic> joints following the proximal joint (index/majeure/ringFinger/pinky,
-  and thumb3 following thumb). 1.0 = every phalanx curls by the same angle.
-  Lower the distal ratio if the modelled fist curls tighter than the hardware.
+  One servo pulls a single tendon through each finger, so the middle and distal
+  phalanges mimic the proximal joint. 1.0 curls every phalanx by the same angle;
+  lower the distal ratio if the model curls tighter than the hardware.
   -->
   <xacro:property name="finger_mid_ratio" value="1.0"/>

File: description/robot_description/urdf/robot_description.urdf.xacro (robot description, xacro)
@@ -100,5 +100,5 @@
     <child link="i01.leftHand.index2_link"/>
     <axis xyz="-0.99994 0.00000 0.01111"/>
-    <mimic joint="i01.leftHand.index_link_joint" multiplier="${finger_mid_ratio}" offset="0.0"/><!-- tendon-coupled phalanx -->
+    <mimic joint="i01.leftHand.index_link_joint" multiplier="${finger_mid_ratio}" offset="0.0"/>
   </joint>
   <joint name="i01.torso.midStom_link_joint" type="revolute">
@@ -117,5 +117,5 @@
     <child link="i01.leftHand.index3_link"/>
     <axis xyz="-0.99994 0.00000 0.01111"/>
-    <mimic joint="i01.leftHand.index_link_joint" multiplier="${finger_distal_ratio}" offset="0.0"/><!-- tendon-coupled phalanx -->
+    <mimic joint="i01.leftHand.index_link_joint" multiplier="${finger_distal_ratio}" offset="0.0"/>
   </joint>
   <joint name="i01.leftHand.majeure_link_joint" type="revolute">
@@ -134,5 +134,5 @@
     <child link="i01.leftHand.majeure2_link"/>
     <axis xyz="-0.99994 0.00000 0.01111"/>
-    <mimic joint="i01.leftHand.majeure_link_joint" multiplier="${finger_mid_ratio}" offset="0.0"/><!-- tendon-coupled phalanx -->
+    <mimic joint="i01.leftHand.majeure_link_joint" multiplier="${finger_mid_ratio}" offset="0.0"/>
   </joint>
   <joint name="i01.leftHand.majeure3_link_joint" type="revolute">
@@ -143,5 +143,5 @@
     <child link="i01.leftHand.majeure3_link"/>
     <axis xyz="-0.99994 0.00000 0.01111"/>
-    <mimic joint="i01.leftHand.majeure_link_joint" multiplier="${finger_distal_ratio}" offset="0.0"/><!-- tendon-coupled phalanx -->
+    <mimic joint="i01.leftHand.majeure_link_joint" multiplier="${finger_distal_ratio}" offset="0.0"/>
   </joint>
   <joint name="i01.leftHand.pinky0_link_joint" type="revolute">
@@ -168,5 +168,5 @@
     <child link="i01.leftHand.pinky2_link"/>
     <axis xyz="-0.99994 0.00000 0.01111"/>
-    <mimic joint="i01.leftHand.pinky_link_joint" multiplier="${finger_mid_ratio}" offset="0.0"/><!-- tendon-coupled phalanx -->
+    <mimic joint="i01.leftHand.pinky_link_joint" multiplier="${finger_mid_ratio}" offset="0.0"/>
   </joint>
   <joint name="i01.leftHand.pinky3_link_joint" type="revolute">
@@ -177,5 +177,5 @@
     <child link="i01.leftHand.pinky3_link"/>
     <axis xyz="-0.99994 0.00000 0.01111"/>
-    <mimic joint="i01.leftHand.pinky_link_joint" multiplier="${finger_distal_ratio}" offset="0.0"/><!-- tendon-coupled phalanx -->
+    <mimic joint="i01.leftHand.pinky_link_joint" multiplier="${finger_distal_ratio}" offset="0.0"/>
   </joint>
   <joint name="i01.leftHand.ringfinger0_link_joint" type="revolute">
@@ -210,5 +210,5 @@
     <child link="i01.leftHand.ringfinger2_link"/>
     <axis xyz="-0.99994 0.00000 0.01111"/>
-    <mimic joint="i01.leftHand.ringFinger_link_joint" multiplier="${finger_mid_ratio}" offset="0.0"/><!-- tendon-coupled phalanx -->
+    <mimic joint="i01.leftHand.ringFinger_link_joint" multiplier="${finger_mid_ratio}" offset="0.0"/>
   </joint>
   <joint name="i01.leftHand.ringfinger3_link_joint" type="revolute">
@@ -219,5 +219,5 @@
     <child link="i01.leftHand.ringfinger3_link"/>
     <axis xyz="-0.99994 0.00000 0.01111"/>
-    <mimic joint="i01.leftHand.ringFinger_link_joint" multiplier="${finger_distal_ratio}" offset="0.0"/><!-- tendon-coupled phalanx -->
+    <mimic joint="i01.leftHand.ringFinger_link_joint" multiplier="${finger_distal_ratio}" offset="0.0"/>
   </joint>
   <joint name="i01.leftHand.thumb1_link_joint" type="revolute">
@@ -244,5 +244,5 @@
     <child link="i01.leftHand.thumb3_link"/>
     <axis xyz="-0.99994 0.00000 0.01111"/>
-    <mimic joint="i01.leftHand.thumb_link_joint" multiplier="${finger_distal_ratio}" offset="0.0"/><!-- tendon-coupled phalanx -->
+    <mimic joint="i01.leftHand.thumb_link_joint" multiplier="${finger_distal_ratio}" offset="0.0"/>
   </joint>
   <joint name="right_shoulder_y_link_joint" type="revolute">
@@ -317,5 +317,5 @@
     <child link="i01.rightHand.index2_link"/>
     <axis xyz="-0.99994 0.00000 0.01111"/>
-    <mimic joint="i01.rightHand.index_link_joint" multiplier="${finger_mid_ratio}" offset="0.0"/><!-- tendon-coupled phalanx -->
+    <mimic joint="i01.rightHand.index_link_joint" multiplier="${finger_mid_ratio}" offset="0.0"/>
   </joint>
   <joint name="i01.rightHand.index3_link_joint" type="revolute">
@@ -326,5 +326,5 @@
     <child link="i01.rightHand.index3_link"/>
     <axis xyz="-0.99994 0.00000 0.01111"/>
-    <mimic joint="i01.rightHand.index_link_joint" multiplier="${finger_distal_ratio}" offset="0.0"/><!-- tendon-coupled phalanx -->
+    <mimic joint="i01.rightHand.index_link_joint" multiplier="${finger_distal_ratio}" offset="0.0"/>
   </joint>
   <joint name="i01.rightHand.majeure_link_joint" type="revolute">
@@ -343,5 +343,5 @@
     <child link="i01.rightHand.majeure2_link"/>
     <axis xyz="-0.99994 0.00000 0.01111"/>
-    <mimic joint="i01.rightHand.majeure_link_joint" multiplier="${finger_mid_ratio}" offset="0.0"/><!-- tendon-coupled phalanx -->
+    <mimic joint="i01.rightHand.majeure_link_joint" multiplier="${finger_mid_ratio}" offset="0.0"/>
   </joint>
   <joint name="i01.rightHand.majeure3_link_joint" type="revolute">
@@ -352,5 +352,5 @@
     <child link="i01.rightHand.majeure3_link"/>
     <axis xyz="-0.99994 0.00000 0.01111"/>
-    <mimic joint="i01.rightHand.majeure_link_joint" multiplier="${finger_distal_ratio}" offset="0.0"/><!-- tendon-coupled phalanx -->
+    <mimic joint="i01.rightHand.majeure_link_joint" multiplier="${finger_distal_ratio}" offset="0.0"/>
   </joint>
   <joint name="i01.rightHand.pinky0_link_joint" type="revolute">
@@ -377,5 +377,5 @@
     <child link="i01.rightHand.pinky2_link"/>
     <axis xyz="-0.99994 0.00000 0.01111"/>
-    <mimic joint="i01.rightHand.pinky_link_joint" multiplier="${finger_mid_ratio}" offset="0.0"/><!-- tendon-coupled phalanx -->
+    <mimic joint="i01.rightHand.pinky_link_joint" multiplier="${finger_mid_ratio}" offset="0.0"/>
   </joint>
   <joint name="i01.head.rollNeck_link_joint" type="revolute">
@@ -394,5 +394,5 @@
     <child link="i01.rightHand.pinky3_link"/>
     <axis xyz="-0.99994 0.00000 0.01111"/>
-    <mimic joint="i01.rightHand.pinky_link_joint" multiplier="${finger_distal_ratio}" offset="0.0"/><!-- tendon-coupled phalanx -->
+    <mimic joint="i01.rightHand.pinky_link_joint" multiplier="${finger_distal_ratio}" offset="0.0"/>
   </joint>
   <joint name="i01.rightHand.ringfinger0_link_joint" type="revolute">
@@ -419,5 +419,5 @@
     <child link="i01.rightHand.ringfinger2_link"/>
     <axis xyz="-0.99994 0.00000 0.01111"/>
-    <mimic joint="i01.rightHand.ringFinger_link_joint" multiplier="${finger_mid_ratio}" offset="0.0"/><!-- tendon-coupled phalanx -->
+    <mimic joint="i01.rightHand.ringFinger_link_joint" multiplier="${finger_mid_ratio}" offset="0.0"/>
   </joint>
   <joint name="i01.rightHand.ringfinger3_link_joint" type="revolute">
@@ -428,5 +428,5 @@
     <child link="i01.rightHand.ringfinger3_link"/>
     <axis xyz="-0.99994 0.00000 0.01111"/>
-    <mimic joint="i01.rightHand.ringFinger_link_joint" multiplier="${finger_distal_ratio}" offset="0.0"/><!-- tendon-coupled phalanx -->
+    <mimic joint="i01.rightHand.ringFinger_link_joint" multiplier="${finger_distal_ratio}" offset="0.0"/>
   </joint>
   <joint name="i01.rightHand.thumb1_link_joint" type="revolute">
@@ -453,5 +453,5 @@
     <child link="i01.rightHand.thumb3_link"/>
     <axis xyz="-0.99994 0.00000 0.01111"/>
-    <mimic joint="i01.rightHand.thumb_link_joint" multiplier="${finger_distal_ratio}" offset="0.0"/><!-- tendon-coupled phalanx -->
+    <mimic joint="i01.rightHand.thumb_link_joint" multiplier="${finger_distal_ratio}" offset="0.0"/>
   </joint>
   <joint name="i01.head.rothead_link_joint" type="revolute">
